File: Main_PCB_001/Main_PCB_001.kicad_pcb (KiCad board)
At the start: 2 copper layers, 72 parts, among them IC1 FDN8601, IC2 FDN8601, IC3 TPS40211QDGQRQ1, IC4 PAM2863ECR, IC5 SI3440ADV-T1-GE3, IC6 FDN8601, IC7 ZXTR2105FQ-7, U1 ATtiny25-20S

Commit message: PCB. Working 001
Parts:
- removed D16: WireHole_1p5, Connector_Wire_User_001:WireHole_1p5
- removed IC7: ZXTR2105FQ-7, libraries:SOT96P240X110-3N
- added D20: WireHole_1p5, libraries:WireHole_1p5, F.Cu at (221.7, 118.5)
- added U2: Mounting_Hole_M2, mount_holes:Hole_screw_M2, F.Cu at (153.0, 111.0)
- added U3: Mounting_Hole_M2, mount_holes:Hole_screw_M2, F.Cu at (102.0, 102.0)
- added U4: Mounting_Hole_M2, mount_holes:Hole_screw_M2, F.Cu at (153.0, 102.0)
- added U5: Mounting_Hole_M2, mount_holes:Hole_screw_M2, F.Cu at (102.0, 111.0)
- D1, D2, D3: footprint Connector_Wire_User_001:WireHole_1p5 -> libraries:WireHole_1p5
- D11, D13, D14, D15, D4, D5, D6, D7, D8, D9: footprint Connector_Wire_User_001:Wire_Pad_01 -> libraries:Wire_Pad_01
- IC5: value SI3440ADV-T1-GE3 -> FDN8601; footprint libraries:SOT95P284X110-6N -> libraries:SOT95P251X112-3N
- IC6: value FDN8601 -> ZXTR2105FQ-7; footprint libraries:SOT95P251X112-3N -> libraries:SOT96P240X110-3N
- moved R2 110.7 mm to (223.8, 109.6)
- moved C3 107.7 mm to (214.3, 105.0)
- moved D14 104.0 mm to (232.5, 104.9)
- moved R9 103.9 mm to (213.9, 114.6)
- moved C7 100.3 mm to (228.8, 104.5)
- moved C20 99.7 mm to (224.5, 104.5)
- moved Z3 99.1 mm to (196.6, 117.1)
- moved R7 97.5 mm to (210.0, 120.5)
- moved C17 97.5 mm to (203.8, 111.5)
- moved R11 97.4 mm to (219.4, 112.5)
- moved C8 97.4 mm to (214.4, 119.6)
- moved D15 97.3 mm to (202.5, 133.9)
- moved R8 95.2 mm to (200.2, 131.0)
- moved Z2 94.6 mm to (207.7, 105.6)
- moved IC1 94.2 mm to (219.8, 105.6)
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Connections:
- D1 pad 1: (no net) -> Net-(C21-Pad1)
- D11 pad 1: (no net) -> Net-(D11-Pad1)
- D13 pad 1: (no net) -> Net-(D13-Pad1)
- D14 pad 1: (no net) -> Net-(D13-Pad1)
- D15 pad 1: (no net) -> Net-(D15-Pad1)
- D2 pad 1: (no net) -> Net-(C1-Pad1)
- D3 pad 1: (no net) -> Net-(D3-Pad1)
- D4 pad 1: (no net) -> Net-(D4-Pad1)
- D5 pad 1: (no net) -> Net-(D5-Pad1)
- D6 pad 1: (no net) -> Net-(D5-Pad1)
- D7 pad 1: (no net) -> Net-(D7-Pad1)
- D8 pad 1: (no net) -> Net-(D7-Pad1)
- D9 pad 1: (no net) -> Net-(D9-Pad1)
- IC1 pad 3: Net-(D3-Pad) -> Net-(D3-Pad1)
- IC2 pad 3: Net-(D3-Pad) -> Net-(D3-Pad1)
- IC4 pad 2: Net-(D11-Pad) -> Net-(D11-Pad1)
- IC5 pad 1: Net-(D12-Pad2) -> Net-(IC5-Pad1)
- IC5 pad 2: Net-(D12-Pad2) -> Net-(IC5-Pad2)
- IC5 pad 3: Net-(IC5-Pad3) -> Net-(D12-Pad2)
- IC6 pad 1: unconnected-(IC6-Pad1) -> GND
- IC6 pad 2: unconnected-(IC6-Pad2) -> Net-(C22-Pad1)
- IC6 pad 3: unconnected-(IC6-Pad3) -> Net-(C23-Pad1)
- L5 pad 1: Net-(D9-Pad) -> Net-(D9-Pad1)
- L9 pad 2: Net-(D15-Pad) -> Net-(D15-Pad1)
- R10 pad 1: Net-(IC5-Pad4) -> Net-(IC5-Pad2)
- R3 pad 2: Net-(D4-Pad) -> Net-(D4-Pad1)
- R4 pad 1: Net-(D4-Pad) -> Net-(D4-Pad1)
- R6 pad 1: Net-(D11-Pad) -> Net-(D11-Pad1)
- R8 pad 2: Net-(IC5-Pad3) -> Net-(IC5-Pad1)
- R9 pad 2: Net-(IC5-Pad4) -> Net-(IC5-Pad2)
Other:
- board outline added: 55 x 13 mm

Commit message: PCB working 003
Parts:
- R4, R5: footprint Resistor_SMD:R_0201_0603Metric_Pad0.64x0.40mm_HandSolder -> Resistor_SMD:R_0603_1608Metric_Pad0.98x0.95mm_HandSolder
- moved R4 172.7 mm to (39.6, 145.8)
- moved C4 170.3 mm to (40.3, 154.9)
- moved C8 163.8 mm to (51.8, 139.2)
- moved C6 162.2 mm to (43.8, 152.9)
- moved C15 162.1 mm to (61.6, 154.4)
- moved R5 161.5 mm to (40.2, 152.9)
- moved L6 160.1 mm to (62.5, 160.5), turned to 180 degrees
- moved R9 157.0 mm to (61.6, 152.4)
- moved C17 156.9 mm to (55.4, 162.5), turned to -90 degrees
- moved R7 153.4 mm to (58.0, 141.2)
- moved C19 152.4 mm to (58.9, 162.1), turned to -90 degrees
- moved D5 151.6 mm to (89.4, 160.5)
- moved C16 149.7 mm to (68.2, 148.8)
- moved D6 149.2 mm to (85.9, 160.5)
- moved D7 147.7 mm to (81.8, 160.5)
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
Commit message: Pcb working 004
Parts:
- removed C19: C, Capacitor_SMD:C_1206_3216Metric_Pad1.33x1.80mm_HandSolder
- removed L5: TFM201610ALC-R47MTAA, libraries:INDC2016X80N
- D10, D12: footprint libraries:DIOM7959X262N -> libraries:SODFL4626X120N
- moved R4 102.7 mm to (142.0, 137.0), turned to 180 degrees
- moved L4 101.7 mm to (133.2, 142.2), turned to 180 degrees
- moved R5 100.7 mm to (139.4, 135.4)
- moved C4 98.8 mm to (136.9, 134.5), turned to -90 degrees
- moved C6 97.5 mm to (139.4, 133.6), turned to 180 degrees
- moved C9 85.7 mm to (137.9, 138.4), turned to 90 degrees
- moved C8 82.9 mm to (134.7, 138.4), turned to 180 degrees
- moved L2 80.8 mm to (138.8, 144.0), turned to 180 degrees
- moved C3 76.2 mm to (139.7, 141.5), turned to 180 degrees
- moved IC3 75.2 mm to (132.8, 135.8), turned to 180 degrees
- moved R7 73.3 mm to (131.3, 138.4), turned to 180 degrees
- moved C13 71.8 mm to (132.3, 126.2)
- moved C15 70.6 mm to (123.2, 120.0)
- moved R9 70.6 mm to (123.2, 118.0)
- moved C18 68.7 mm to (117.0, 140.8), turned to 0 degrees
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Connections:
- D9 pad 1: Net-(D9-Pad1) -> Net-(C14-Pad1)
Other:
- board size 55 x 13 mm -> 55 x 45.3 mm
- copper layers 2 -> 4

Commit message: PCB working
Parts:
- removed C18: C, Capacitor_SMD:C_1206_3216Metric_Pad1.33x1.80mm_HandSolder
- C13: footprint Capacitor_SMD:C_1206_3216Metric_Pad1.33x1.80mm_HandSolder -> Capacitor_SMD:C_0805_2012Metric_Pad1.18x1.45mm_HandSolder
- R10: footprint Resistor_SMD:R_0805_2012Metric_Pad1.20x1.40mm_HandSolder -> Resistor_SMD:R_0603_1608Metric_Pad0.98x0.95mm_HandSolder
- moved D11 155.3 mm to (85.3, 68.3)
- moved D13 155.3 mm to (88.9, 68.3)
- moved D14 155.3 mm to (92.5, 68.3)
- moved D15 155.3 mm to (96.0, 68.3)
- moved C10 143.4 mm to (108.2, 96.9), turned to 180 degrees
- moved C12 124.2 mm to (115.6, 142.7), turned to 90 degrees
- moved C20 120.2 mm to (119.1, 87.9), turned to 90 degrees
- moved C7 118.4 mm to (112.0, 85.6)
- moved L9 117.1 mm to (118.6, 96.0), turned to 180 degrees
- moved L8 115.0 mm to (117.2, 92.2)
- moved L1 114.6 mm to (112.0, 88.5), turned to 180 degrees
- moved C1 112.4 mm to (115.1, 87.2), turned to 90 degrees
- moved IC4 110.8 mm to (110.1, 92.6)
- moved R6 106.3 mm to (104.9, 92.3), turned to 90 degrees
- moved C2 105.9 mm to (117.3, 87.9), turned to 90 degrees
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Other:
- outline, holes or cut-outs redrawn

Commit message: PCB on work
Parts:
- removed C13: C, Capacitor_SMD:C_0805_2012Metric_Pad1.18x1.45mm_HandSolder
- removed C3: C, Capacitor_SMD:C_1206_3216Metric_Pad1.33x1.80mm_HandSolder
- C20: footprint Capacitor_SMD:C_0603_1608Metric_Pad1.08x0.95mm_HandSolder -> Capacitor_SMD:C_1206_3216Metric_Pad1.33x1.80mm_HandSolder
- moved D5 88.7 mm to (170.2, 123.8)
- moved D7 88.7 mm to (162.6, 123.8)
- moved D4 88.7 mm to (173.7, 123.8)
- moved D6 88.7 mm to (166.6, 123.8)
- moved D8 88.7 mm to (159.0, 123.8)
- moved D9 88.7 mm to (156.0, 123.8)
- moved C20 4.45 mm to (123.4, 87.0)
- moved C4 3.88 mm to (133.3, 133.0), turned to 0 degrees
- moved R3 3.12 mm to (138.3, 140.1), turned to 90 degrees
- moved C9 2.85 mm to (136.9, 135.8), turned to -90 degrees
- moved C6 2.62 mm to (136.9, 133.0)
- moved R4 2.53 mm to (139.4, 136.8), turned to 0 degrees
- moved R5 1.53 mm to (139.6, 133.9), turned to 90 degrees
- moved L9 0.57 mm to (119.0, 96.4)
Connections:
- C2 pad 1: Net-(C1-Pad1) -> Net-(C2-Pad1)
- D2 pad 1: Net-(C1-Pad1) -> Net-(C2-Pad1)
- L1 pad 1: Net-(C1-Pad1) -> Net-(C2-Pad1)
- R2 pad 1: Net-(C1-Pad1) -> Net-(C2-Pad1)

Commit message: PCB underwork
Parts:
- removed C1: C, Capacitor_SMD:C_1206_3216Metric
- removed C5: C, Capacitor_SMD:C_0603_1608Metric
- removed L2: TFM201610ALC-R47MTAA, libraries:INDC2016X80N
- C15, C4, C6, C8, C9: footprint Capacitor_SMD:C_0603_1608Metric_Pad1.08x0.95mm_HandSolder -> Capacitor_SMD:C_0402_1005Metric_Pad0.74x0.62mm_HandSolder
- L4: footprint libraries:INDPM5752X300N -> libraries:INDPM4441X200N
- L7: footprint libraries:INDPM7366X500N -> libraries:INDPM5752X300N
- R10, R11, R4, R5, R7, R8, R9: footprint Resistor_SMD:R_0603_1608Metric_Pad0.98x0.95mm_HandSolder -> Resistor_SMD:R_0402_1005Metric_Pad0.72x0.64mm_HandSolder
- R3: footprint Resistor_SMD:R_1206_3216Metric_Pad1.30x1.75mm_HandSolder -> Resistor_SMD:R_0805_2012Metric_Pad1.20x1.40mm_HandSolder
- moved C14 34.9 mm to (145.9, 121.0), turned to 180 degrees
- moved L6 30.7 mm to (145.9, 123.1)
- moved Z3 30.1 mm to (145.9, 127.0), turned to -90 degrees
- moved C12 28.2 mm to (135.4, 122.7), turned to -90 degrees
- moved D12 27.7 mm to (144.8, 131.6), turned to 180 degrees
- moved L7 24.0 mm to (140.3, 123.2), turned to 0 degrees
- moved IC5 21.5 mm to (142.1, 127.9), turned to 0 degrees
- moved C11 20.0 mm to (129.0, 127.4), turned to -90 degrees
- moved L4 19.7 mm to (130.9, 122.7), turned to 0 degrees
- moved C17 17.6 mm to (139.2, 132.0), turned to 180 degrees
- moved R8 16.4 mm to (138.9, 126.7), turned to 0 degrees
- moved R10 13.8 mm to (138.9, 130.2), turned to 180 degrees
- moved R9 13.8 mm to (138.9, 127.9), turned to 0 degrees
- moved R7 12.9 mm to (136.5, 126.6), turned to 0 degrees
- moved C8 12.8 mm to (135.4, 125.6), turned to 0 degrees
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Connections:
- C11 pad 1: Net-(C11-Pad1) -> Net-(C21-Pad1)
- L4 pad 1: Net-(C11-Pad1) -> Net-(C21-Pad1)
Other:
- board size 55 x 45.3 mm -> 55 x 33.3 mm

Commit message: PCB working on
Parts:
- removed C2: C, Capacitor_SMD:C_0603_1608Metric_Pad1.08x0.95mm_HandSolder
- removed L1: TFM201610ALC-R47MTAA, libraries:INDC2016X80N
- C10, C20: footprint Capacitor_SMD:C_1206_3216Metric_Pad1.33x1.80mm_HandSolder -> Capacitor_SMD:C_0805_2012Metric_Pad1.18x1.45mm_HandSolder
- C21, C22, C23, IC1, IC2, IC6, L10, R1, R12, R2, U1, Z1, Z2: moved to B.Cu
- L3: footprint libraries:INDPM4441X200N -> libraries:INDC2016X80N
- R10: footprint Resistor_SMD:R_0402_1005Metric_Pad0.72x0.64mm_HandSolder -> Resistor_SMD:R_0603_1608Metric_Pad0.98x0.95mm_HandSolder
- R11: footprint Resistor_SMD:R_0402_1005Metric_Pad0.72x0.64mm_HandSolder -> Resistor_SMD:R_0603_1608Metric_Pad0.98x0.95mm_HandSolder; moved to B.Cu
- U2, U3, U4, U5: footprint mount_holes:Hole_screw_M2 -> mount_holes:Hole_screw_M1p2
- moved C21 115.2 mm to (104.6, 94.1), turned to -90 degrees
- moved L10 92.9 mm to (141.9, 88.0), turned to 90 degrees
- moved R11 91.8 mm to (139.3, 92.2), turned to -90 degrees
- moved R12 87.6 mm to (138.6, 95.3), turned to 180 degrees
- moved IC6 87.2 mm to (148.7, 88.0), turned to 90 degrees
- moved R2 82.4 mm to (117.1, 96.2), turned to 90 degrees
- moved Z2 82.0 mm to (115.4, 92.5)
- moved C23 81.9 mm to (145.0, 86.9), turned to 180 degrees
- moved IC2 80.5 mm to (114.1, 96.4), turned to -90 degrees
- moved C22 79.6 mm to (145.0, 89.1), turned to 180 degrees
- moved D11 78.2 mm to (153.1, 107.5), turned to 90 degrees
- moved U1 76.7 mm to (145.7, 93.2), turned to 180 degrees
- moved D4 75.0 mm to (101.3, 104.4)
- moved D13 74.1 mm to (153.1, 105.3), turned to 90 degrees
- moved D5 69.8 mm to (103.1, 104.4)
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Connections:
- C7 pad 1: Net-(C7-Pad1) -> Net-(D2-Pad1)
- D2 pad 1: Net-(C2-Pad1) -> Net-(D2-Pad1)
- L3 pad 1: Net-(C7-Pad1) -> Net-(D2-Pad1)
- R2 pad 1: Net-(C2-Pad1) -> Net-(D2-Pad1)
Routing:
- net Net-(C17-Pad1): track 0.00 -> 13.9 mm
- net Net-(D12-Pad2): track 0.00 -> 9.06 mm
- net Net-(C12-Pad1): track 0.00 -> 6.97 mm
- net Net-(C4-Pad1): track 0.00 -> 6.60 mm
- net Net-(C16-Pad1): track 0.00 -> 6.15 mm
- net Net-(C15-Pad1): track 0.00 -> 5.50 mm
- net Net-(IC5-Pad2): track 0.00 -> 4.91 mm
- net Net-(C14-Pad1): track 0.00 -> 4.41 mm
- net Net-(C4-Pad2): track 0.00 -> 4.19 mm
- net Net-(IC3-Pad8): track 0.00 -> 3.54 mm
- net Net-(C8-Pad2): track 0.00 -> 2.82 mm
- net Net-(C9-Pad2): track 0.00 -> 2.13 mm
- net Net-(D4-Pad1): track 0.00 -> 1.84 mm
- net Net-(IC5-Pad1): track 0.00 -> 1.69 mm
- net Net-(C6-Pad1): track 0.00 -> 1.03 mm
Other:
- board size 55 x 33.3 mm -> 55 x 15 mm

Commit message: PCB working on
Parts:
- moved C21 3.06 mm to (107.1, 95.9), turned to 180 degrees
- moved R11 2.99 mm to (138.4, 95.0), turned to 0 degrees
- moved R12 2.70 mm to (138.4, 92.6)
- moved D6 0.15 mm to (150.0, 111.8)
- moved D9 0.15 mm to (150.0, 101.1)
Connections:
- U1 pad 5: Net-(R12-Pad1) -> unconnected-(U1-Pad5)
- U1 pad 7: unconnected-(U1-Pad7) -> Net-(R12-Pad1)
Routing:
- net Net-(D10-Pad2): track 0.00 -> 12.4 mm
- net Net-(C10-Pad1): track 0.00 -> 9.25 mm
- net Net-(C23-Pad1): track 0.00 -> 8.82 mm
- net Net-(IC1-Pad1): track 0.00 -> 8.28 mm
- net Net-(IC2-Pad1): track 0.00 -> 7.99 mm
- net Net-(C22-Pad1): track 0.00 -> 7.33 mm
- net Net-(C20-Pad1): track 0.00 -> 4.54 mm
- net Net-(D11-Pad1): track 0.00 -> 3.45 mm, vias 0 -> 1
- net Net-(R11-Pad2): track 0.00 -> 3.32 mm
- net Net-(R12-Pad1): track 0.00 -> 2.84 mm
- net Net-(C7-Pad1): track 0.00 -> 2.20 mm
- net Net-(IC3-Pad3): vias 0 -> 1
- net Net-(D7-Pad1): vias 0 -> 2
- net Net-(D5-Pad1): vias 0 -> 2
- net Net-(D4-Pad1): vias 0 -> 2
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