File: Main_PCB_001/Main_PCB_001.kicad_pcb (KiCad board)
At the start: 4 copper layers, 55 x 15 mm, 65 parts, among them IC1 FDN8601, IC2 FDN8601, IC3 TPS40211QDGQRQ1, IC4 PAM2863ECR, IC5 FDN8601, IC6 ZXTR2105FQ-7, U1 ATtiny25-20S, U2 Mounting_Hole_M2, U3 Mounting_Hole_M2, U4 Mounting_Hole_M2, U5 Mounting_Hole_M2

Commit message: PCB working
Parts:
- moved L9 14.2 mm to (106.4, 102.7), turned to 90 degrees
- moved C7 13.8 mm to (119.2, 107.1), turned to -90 degrees
- moved C10 13.6 mm to (117.5, 102.0), turned to 0 degrees
- moved L3 11.8 mm to (117.9, 104.3), turned to 180 degrees
- moved C20 10.5 mm to (108.7, 102.7), turned to 90 degrees
- moved L8 10.4 mm to (107.3, 107.8), turned to 90 degrees
- moved D10 9.74 mm to (116.9, 108.3), turned to -90 degrees
- moved R6 8.80 mm to (113.0, 102.1), turned to 0 degrees
- moved D15 5.61 mm to (103.2, 103.7), turned to 180 degrees
- moved D14 5.58 mm to (101.4, 103.7), turned to 180 degrees
- moved D4 4.67 mm to (101.4, 109.1)
- moved D5 4.67 mm to (103.2, 109.1)
- moved IC4 1.41 mm to (112.6, 107.1), turned to -90 degrees
Routing:
- net Net-(D13-Pad1): track 0.00 -> 58.3 mm
- net Net-(D5-Pad1): track 0.00 -> 51.7 mm
- net Net-(D11-Pad1): track 3.45 -> 54.8 mm, vias 1 -> 2
- net Net-(D4-Pad1): track 1.84 -> 34.9 mm
- net Net-(C14-Pad1): track 4.41 -> 16.7 mm
- net Net-(D7-Pad1): track 0.00 -> 11.5 mm
- net Net-(D15-Pad1): track 0.00 -> 8.58 mm, vias 1 -> 2

Commit message: PCB+Solidworks
Parts:
- D1, D2, D20, D3: footprint libraries:WireHole_1p5 -> libraries:WireHole_1p2
- moved C22 16.5 mm to (139.8, 104.8)
- moved U1 16.5 mm to (140.6, 108.8)
- moved L10 16.5 mm to (136.7, 103.7)
- moved C23 16.5 mm to (139.9, 102.6)
- moved IC6 16.5 mm to (143.5, 103.7)
- moved R11 16.5 mm to (133.2, 110.7)
- moved R12 16.5 mm to (133.2, 108.3)
- moved Z1 13.1 mm to (130.2, 105.3), turned to -90 degrees
- moved Z2 12.5 mm to (114.0, 104.9), turned to 90 degrees
- moved R1 11.2 mm to (126.3, 107.0), turned to 0 degrees
- moved IC2 10.5 mm to (117.9, 106.2), turned to 0 degrees
- moved C21 10.5 mm to (107.2, 106.3), turned to -90 degrees
- moved IC1 7.63 mm to (126.2, 104.0), turned to 180 degrees
- moved R2 6.94 mm to (117.8, 103.1), turned to 180 degrees
- moved D13 3.04 mm to (153.4, 108.3)
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Routing:
- net Net-(C11-Pad1): track 0.00 -> 46.7 mm, vias 0 -> 1
- net Net-(IC3-Pad3): track 0.00 -> 17.2 mm
- net Net-(D20-Pad1): track 0.00 -> 11.4 mm
- net Net-(C7-Pad1): track 2.20 -> 13.0 mm, vias 0 -> 1
- net Net-(D3-Pad1): track 0.00 -> 6.93 mm
- net Net-(D13-Pad1): track 58.3 -> 63.0 mm
- net Net-(D11-Pad1): track 54.8 -> 57.0 mm
- net Net-(C14-Pad1): track 16.7 -> 15.5 mm
- net GND: vias 0 -> 38
- added copper zone on B.Cu, net GND
- added copper zone on F.Cu, net GND
- added copper zone on In1.Cu, net GND
- added copper zone on In2.Cu, net GND
