File: Main_PCB_001/Main_PCB_001.kicad_sch (KiCad schematic)
At the start: 72 parts

Commit message: PCB. Working 001
Parts:
- removed D16: (no value), symbol Connectors_for_Wire:WireHole_1p5
- removed IC5: (no value), symbol SI3440ADV-T1-GE3:SI3440ADV-T1-GE3
- added D20: (no value), symbol Connectors_for_Wire:WireHole_1p5
- added U2, U3: (no value), symbol Mounting_Holes:Mounting_Hole_M2
- added U4, U5: Mounting_Hole_M2, symbol Mounting_Holes:Mounting_Hole_M2
- U1: footprint (none) -> Package_SO:SOIC-8W_5.3x5.3mm_P1.27mm
- renumbered IC6 to IC5, IC7 to IC6
Connections:
- net GND: now also U2.1 (Mnt), U3.1 (Mnt), U4.1 (Mnt), U5.1 (Mnt)
- net at R3.2, R4.1: now also D4.1 (Conn); no longer D4.
- net at R8.2: now also IC5.1 (G)
- net at R10.1, R9.2: now also IC5.2 (S)
- net at D12.2, L7.2: now also IC5.3 (D)
- net at L5.1: now also D9.1 (Conn); no longer D9.
- net at C1.1, C2.1, L1.1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: now also D2.1 (Conn); no longer D2.
- net at C21.1, C3.1, C5.1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: now also D1.1 (Conn); no longer D1.
- net at IC4.2 (ISENSE), R6.1: now also D11.1 (Conn); no longer D11.
- net at L9.2: now also D15.1 (Conn); no longer D15.
- net at IC1.3 (D), IC2.3 (D): now also D3.1 (Conn); no longer D3.
- net at R12.2: now also D20.1 (Conn)
- new net: D13.1 (Conn), D14.1 (Conn)
- new net: D7.1 (Conn), D8.1 (Conn)
- new net: D5.1 (Conn), D6.1 (Conn)
Other:
- moved on the sheet: IC5

Commit message: PCB working 003
Parts:
- C1: value (none) -> C; footprint (none) -> Capacitor_SMD:C_1206_3216Metric
- C10, C12, C13, C17, C18, C19, C3: value (none) -> C; footprint (none) -> Capacitor_SMD:C_1206_3216Metric_Pad1.33x1.80mm_HandSolder
- C11, C14, C15, C16, C2, C20, C22, C23, C4, C6, C7, C8, C9: value (none) -> C; footprint (none) -> Capacitor_SMD:C_0603_1608Metric_Pad1.08x0.95mm_HandSolder
- C21: value (none) -> C; footprint (none) -> Capacitor_SMD:C_1812_4532Metric_Pad1.57x3.40mm_HandSolder
- C5: value (none) -> C; footprint (none) -> Capacitor_SMD:C_0603_1608Metric
- D1, D2, D20, D3: value (none) -> WireHole_1p5; footprint (none) -> libraries:WireHole_1p5
- D10, D12: value (none) -> SS36; footprint (none) -> libraries:DIOM7959X262N
- D11, D13, D14, D15, D4, D5, D6, D7, D8, D9: value (none) -> Wire_Pad_01; footprint (none) -> libraries:Wire_Pad_01
- IC1, IC2, IC5: value (none) -> FDN8601; footprint (none) -> libraries:SOT95P251X112-3N
- IC3: value (none) -> TPS40211QDGQRQ1; footprint (none) -> libraries:SOP50P490X110-11N
- IC4: value (none) -> PAM2863ECR; footprint (none) -> libraries:SOIC127P600X175-9N
- IC6: value (none) -> ZXTR2105FQ-7; footprint (none) -> libraries:SOT96P240X110-3N
- L1, L10, L2, L5, L6, L9: value (none) -> TFM201610ALC-R47MTAA; footprint (none) -> libraries:INDC2016X80N
- L3, L8: value (none) -> SRP4020TA-100M; footprint (none) -> libraries:INDPM4441X200N
- L4: value (none) -> SRP5030T-100M; footprint (none) -> libraries:INDPM5752X300N
- L7: value (none) -> SRP7050AA-220M; footprint (none) -> libraries:INDPM7366X500N
- R1, R11, R12, R2, R7, R8, R9: value (none) -> R; footprint (none) -> Resistor_SMD:R_0603_1608Metric_Pad0.98x0.95mm_HandSolder
- R10: value (none) -> R; footprint (none) -> Resistor_SMD:R_0805_2012Metric_Pad1.20x1.40mm_HandSolder
- R3, R6: value (none) -> R; footprint (none) -> Resistor_SMD:R_1206_3216Metric_Pad1.30x1.75mm_HandSolder
- R4, R5: value (none) -> R
- U1: value (none) -> ATtiny25-20S
- U2, U3: value (none) -> Mounting_Hole_M2; footprint (none) -> mount_holes:Hole_screw_M2
- U4, U5: footprint (none) -> mount_holes:Hole_screw_M2
- Z1, Z2: value (none) -> BZT52-C12J; footprint (none) -> libraries:BZT52C12J
- Z3: value (none) -> BZT52-C5V1J; footprint (none) -> libraries:SOD3616X130N

Commit message: Pcb working 004
Parts:
- removed C19: C, Capacitor_SMD:C_1206_3216Metric_Pad1.33x1.80mm_HandSolder, symbol Device:C
- removed L5: TFM201610ALC-R47MTAA, libraries:INDC2016X80N, symbol TFM201610ALC-R47MTAA:TFM201610ALC-R47MTAA
- D10, D12: footprint libraries:DIOM7959X262N -> (none)
- R4, R5: footprint (none) -> Resistor_SMD:R_0603_1608Metric_Pad0.98x0.95mm_HandSolder
Connections:
- net at C14.1, L6.1: now also D9.1 (Conn)
Changed lines of the file:
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@@
   (junction (at 186.69 250.19) (diameter 0) (color 0 0 0 0)
   )
-  (junction (at 264.16 33.02) (diameter 0) (color 0 0 0 0)
-  )
   (junction (at 180.34 83.82) (diameter 0) (color 0 0 0 0)
   )
@@
     (stroke (width 0) (type default) (color 0 0 0 0))
   )
-  (wire (pts (xy 220.98 33.02) (xy 223.52 33.02))
+  (wire (pts (xy 195.58 33.02) (xy 223.52 33.02))
     (stroke (width 0) (type default) (color 0 0 0 0))
   )
@@
     (stroke (width 0) (type default) (color 0 0 0 0))
   )
-  (wire (pts (xy 256.54 33.02) (xy 264.16 33.02))
-    (stroke (width 0) (type default) (color 0 0 0 0))
-  )
   (wire (pts (xy 140.97 148.59) (xy 138.43 148.59))
     (stroke (width 0) (type default) (color 0 0 0 0))
@@
     (stroke (width 0) (type default) (color 0 0 0 0))
   )
-  (wire (pts (xy 264.16 33.02) (xy 270.51 33.02))
+  (wire (pts (xy 256.54 33.02) (xy 270.51 33.02))
     (stroke (width 0) (type default) (color 0 0 0 0))
   )
@@
     (stroke (width 0) (type default) (color 0 0 0 0))
   )
-  (wire (pts (xy 264.16 40.64) (xy 264.16 43.18))
-    (stroke (width 0) (type default) (color 0 0 0 0))
-  )
   (wire (pts (xy 152.4 33.02) (xy 156.21 33.02))
     (stroke (width 0) (type default) (color 0 0 0 0))
@@
   )
   (wire (pts (xy 283.21 162.56) (xy 283.21 78.74))
-    (stroke (width 0) (type default) (color 0 0 0 0))
-  )
-  (wire (pts (xy 195.58 33.02) (xy 200.66 33.02))
     (stroke (width 0) (type default) (color 0 0 0 0))
   )
@@
       (effects (font (size 1.27 1.27)) (justify left))
     )
-    (property "Footprint" "" (id 2) (at 107.442 115.57 90)
+    (property "Footprint" "Resistor_SMD:R_0603_1608Metric_Pad0.98x0.95mm_HandSolder" (id 2) (at 107.442 115.57 90)
       (effects (font (size 1.27 1.27)) hide)
     )
@@
       (effects (font (size 1.27 1.27)) (justify left))
     )
-    (property "Footprint" "" (id 2) (at 134.62 150.368 90)
+    (property "Footprint" "Resistor_SMD:R_0603_1608Metric_Pad0.98x0.95mm_HandSolder" (id 2) (at 134.62 150.368 90)
       (effects (font (size 1.27 1.27)) hide)
     )
@@
     )
     (property "Datasheet" "~" (id 3) (at 162.56 123.19 0)
-      (effects (font (size 1.27 1.27)) hide)
-    )
-    (pin "1")
-    (pin "2")
-  )
-  (symbol (lib_id "Device:C") (at 264.16 36.83 0) (unit 1)
-    (in_bom yes) (on_board yes)
-    (property "Reference" "C19" (id 0) (at 267.081 35.6616 0)
-      (effects (font (size 1.27 1.27)) (justify left))
-    )
-    (property "Value" "C" (id 1) (at 267.081 37.973 0)
-      (effects (font (size 1.27 1.27)) (justify left))
-    )
-    (property "Footprint" "Capacitor_SMD:C_1206_3216Metric_Pad1.33x1.80mm_HandSolder" (id 2) (at 265.1252 40.64 0)
-      (effects (font (size 1.27 1.27)) hide)
-    )
-    (property "Datasheet" "~" (id 3) (at 264.16 36.83 0)
       (effects (font (size 1.27 1.27)) hide)
     )
@@
     (pin "1")
   )
-  (symbol (lib_id "power:GND") (at 264.16 43.18 0) (unit 1)
-    (in_bom yes) (on_board yes)
-    (property "Reference" "#PWR027" (id 0) (at 264.16 49.53 0)
-      (effects (font (size 1.27 1.27)) hide)
-    )
-    (property "Value" "GND" (id 1) (at 264.287 47.5742 0))
-    (property "Footprint" "" (id 2) (at 264.16 43.18 0)
-      (effects (font (size 1.27 1.27)) hide)
-    )
-    (property "Datasheet" "" (id 3) (at 264.16 43.18 0)
-      (effects (font (size 1.27 1.27)) hide)
-    )
-    (pin "1")
-  )
   (symbol (lib_id "power:GND") (at 96.52 96.52 0) (unit 1)
     (in_bom yes) (on_board yes)
@@
       (effects (font (size 1.27 1.27)) (justify left))
     )
-    (property "Footprint" "libraries:DIOM7959X262N" (id 2) (at 274.32 73.66 0)
+    (property "Footprint" "" (id 2) (at 274.32 73.66 0)
       (effects (font (size 1.27 1.27)) (justify left) hide)
     )
@@
     (property "Datasheet" "~" (id 3) (at 223.52 36.83 0)
       (effects (font (size 1.27 1.27)) hide)
-    )
-    (pin "1")
-    (pin "2")
-  )
-  (symbol (lib_id "TFM201610ALC-R47MTAA:TFM201610ALC-R47MTAA") (at 200.66 33.02 0) (unit 1)
-    (in_bom yes) (on_board yes) (fields_autoplaced)
-    (property "Reference" "L5" (id 0) (at 210.82 26.67 0))
-    (property "Value" "TFM201610ALC-R47MTAA" (id 1) (at 210.82 29.21 0))
-    (property "Footprint" "libraries:INDC2016X80N" (id 2) (at 217.17 31.75 0)
-      (effects (font (size 1.27 1.27)) (justify left) hide)
-    )
-    (property "Datasheet" "https://datasheet.datasheetarchive.com/originals/distributors/DKDS41/DSANUWW0039576.pdf" (id 3) (at 217.17 34.29 0)
-      (effects (font (size 1.27 1.27)) (justify left) hide)
-    )
-    (property "Description" "Inductors for Power Circuits, for Consumer, Thin Film Metal, TFM201610ALC ,-40 to +125" (id 4) (at 217.17 36.83 0)
-      (effects (font (size 1.27 1.27)) (justify left) hide)
-    )
-    (property "Height" "0.8" (id 5) (at 217.17 39.37 0)
-      (effects (font (size 1.27 1.27)) (justify left) hide)
-    )
-    (property "Manufacturer_Name" "TDK" (id 6) (at 217.17 41.91 0)
-      (effects (font (size 1.27 1.27)) (justify left) hide)
-    )
-    (property "Manufacturer_Part_Number" "TFM201610ALC-R47MTAA" (id 7) (at 217.17 44.45 0)
-      (effects (font (size 1.27 1.27)) (justify left) hide)
-    )
-    (property "Mouser Part Number" "810-TFM201610ALCR47M" (id 8) (at 217.17 46.99 0)
-      (effects (font (size 1.27 1.27)) (justify left) hide)
-    )
-    (property "Mouser Price/Stock" "https://www.mouser.co.uk/ProductDetail/TDK/TFM201610ALC-R47MTAA?qs=MLItCLRbWsy9rkE7tyNMeg%3D%3D" (id 9) (at 217.17 49.53 0)
-      (effects (font (size 1.27 1.27)) (justify left) hide)
-    )
-    (property "Arrow Part Number" "TFM201610ALC-R47MTAA" (id 10) (at 217.17 52.07 0)
-      (effects (font (size 1.27 1.27)) (justify left) hide)
-    )
-    (property "Arrow Price/Stock" "https://www.arrow.com/en/products/tfm201610alc-r47mtaa/tdk" (id 11) (at 217.17 54.61 0)
-      (effects (font (size 1.27 1.27)) (justify left) hide)
     )
     (pin "1")
@@
     (property "Reference" "D10" (id 0) (at 215.9 222.25 0))
     (property "Value" "SS36" (id 1) (at 215.9 224.79 0))
-    (property "Footprint" "libraries:DIOM7959X262N" (id 2) (at 218.44 226.06 0)
+    (property "Footprint" "" (id 2) (at 218.44 226.06 0)
       (effects (font (size 1.27 1.27)) (justify left) hide)
     )
@@
       (reference "#PWR026") (unit 1) (value "GND") (footprint "")
     )
-    (path "/00000000-0000-0000-0000-0000624a317e"
-      (reference "#PWR027") (unit 1) (value "GND") (footprint "")
-    )
     (path "/00000000-0000-0000-0000-0000624a2c8d"
       (reference "#PWR028") (unit 1) (value "GND") (footprint "")
@@
       (reference "C18") (unit 1) (value "C") (footprint "Capacitor_SMD:C_1206_3216Metric_Pad1.33x1.80mm_HandSolder")
     )
-    (path "/00000000-0000-0000-0000-00006248f4c1"
-      (reference "C19") (unit 1) (value "C") (footprint "Capacitor_SMD:C_1206_3216Metric_Pad1.33x1.80mm_HandSolder")
-    )
     (path "/55ec37cf-15cf-4b36-b24a-60d153216a17"
       (reference "C20") (unit 1) (value "C") (footprint "Capacitor_SMD:C_0603_1608Metric_Pad1.08x0.95mm_HandSolder")
@@
     )
     (path "/eb3c41f5-e593-4739-b28b-d6a356df9427"
-      (reference "D10") (unit 1) (value "SS36") (footprint "libraries:DIOM7959X262N")
+      (reference "D10") (unit 1) (value "SS36") (footprint "libraries:SODFL4626X120N")
     )
     (path "/96adca15-5b91-449f-87e3-15c5f9491b32"
@@
     )
     (path "/00000000-0000-0000-0000-0000624b854d"
-      (reference "D12") (unit 1) (value "SS36") (footprint "libraries:DIOM7959X262N")
+      (reference "D12") (unit 1) (value "SS36") (footprint "libraries:SODFL4626X120N")
     )
     (path "/73cf8535-cf48-4953-9103-28ae6c565156"
@@
       (reference "L4") (unit 1) (value "SRP5030T-100M") (footprint "libraries:INDPM5752X300N")
     )
-    (path "/043395fa-6652-4fe3-a89e-9fec57550fac"
-      (reference "L5") (unit 1) (value "TFM201610ALC-R47MTAA") (footprint "libraries:INDC2016X80N")
-    )
     (path "/bad926e6-0260-4e9a-aa4d-2eb3bd5bd948"

Commit message: PCB working
Parts:
- removed C18: C, Capacitor_SMD:C_1206_3216Metric_Pad1.33x1.80mm_HandSolder, symbol Device:C
- C13: footprint Capacitor_SMD:C_1206_3216Metric_Pad1.33x1.80mm_HandSolder -> (none)
- D10, D12: footprint (none) -> libraries:SODFL4626X120N
- R10: footprint Resistor_SMD:R_0805_2012Metric_Pad1.20x1.40mm_HandSolder -> (none)
Changed lines of the file:
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@@
   (junction (at 406.4 274.32) (diameter 0) (color 0 0 0 0)
   )
-  (junction (at 256.54 33.02) (diameter 0) (color 0 0 0 0)
-  )
   (junction (at 148.59 140.97) (diameter 0) (color 0 0 0 0)
   )
@@
     (stroke (width 0) (type default) (color 0 0 0 0))
   )
-  (wire (pts (xy 248.92 33.02) (xy 256.54 33.02))
-    (stroke (width 0) (type default) (color 0 0 0 0))
-  )
-  (wire (pts (xy 256.54 40.64) (xy 256.54 43.18))
-    (stroke (width 0) (type default) (color 0 0 0 0))
-  )
   (wire (pts (xy 166.37 250.19) (xy 163.83 250.19))
     (stroke (width 0) (type default) (color 0 0 0 0))
@@
     (stroke (width 0) (type default) (color 0 0 0 0))
   )
-  (wire (pts (xy 256.54 33.02) (xy 270.51 33.02))
+  (wire (pts (xy 248.92 33.02) (xy 270.51 33.02))
     (stroke (width 0) (type default) (color 0 0 0 0))
   )
@@
       (effects (font (size 1.27 1.27)) (justify left))
     )
-    (property "Footprint" "Resistor_SMD:R_0805_2012Metric_Pad1.20x1.40mm_HandSolder" (id 2) (at 268.732 148.59 90)
+    (property "Footprint" "" (id 2) (at 268.732 148.59 90)
       (effects (font (size 1.27 1.27)) hide)
     )
@@
       (effects (font (size 1.27 1.27)) (justify left))
     )
-    (property "Footprint" "Capacitor_SMD:C_1206_3216Metric_Pad1.33x1.80mm_HandSolder" (id 2) (at 223.2152 115.57 0)
+    (property "Footprint" "" (id 2) (at 223.2152 115.57 0)
       (effects (font (size 1.27 1.27)) hide)
     )
@@
       (effects (font (size 1.27 1.27)) (justify left))
     )
-    (property "Footprint" "" (id 2) (at 274.32 73.66 0)
+    (property "Footprint" "libraries:SODFL4626X120N" (id 2) (at 274.32 73.66 0)
       (effects (font (size 1.27 1.27)) (justify left) hide)
     )
@@
     (property "Reference" "D10" (id 0) (at 215.9 222.25 0))
     (property "Value" "SS36" (id 1) (at 215.9 224.79 0))
-    (property "Footprint" "" (id 2) (at 218.44 226.06 0)
+    (property "Footprint" "libraries:SODFL4626X120N" (id 2) (at 218.44 226.06 0)
       (effects (font (size 1.27 1.27)) (justify left) hide)
     )
@@
     (property "Arrow Price/Stock" "" (id 11) (at 218.44 248.92 0)
       (effects (font (size 1.27 1.27)) (justify left) hide)
-    )
-    (pin "1")
-    (pin "2")
-  )
-  (symbol (lib_id "power:GND") (at 256.54 43.18 0) (unit 1)
-    (in_bom yes) (on_board yes)
-    (property "Reference" "#PWR026" (id 0) (at 256.54 49.53 0)
-      (effects (font (size 1.27 1.27)) hide)
-    )
-    (property "Value" "GND" (id 1) (at 256.667 47.5742 0))
-    (property "Footprint" "" (id 2) (at 256.54 43.18 0)
-      (effects (font (size 1.27 1.27)) hide)
-    )
-    (property "Datasheet" "" (id 3) (at 256.54 43.18 0)
-      (effects (font (size 1.27 1.27)) hide)
-    )
-    (pin "1")
-  )
-  (symbol (lib_id "Device:C") (at 256.54 36.83 0) (unit 1)
-    (in_bom yes) (on_board yes)
-    (property "Reference" "C18" (id 0) (at 259.461 35.6616 0)
-      (effects (font (size 1.27 1.27)) (justify left))
-    )
-    (property "Value" "C" (id 1) (at 259.461 37.973 0)
-      (effects (font (size 1.27 1.27)) (justify left))
-    )
-    (property "Footprint" "Capacitor_SMD:C_1206_3216Metric_Pad1.33x1.80mm_HandSolder" (id 2) (at 257.5052 40.64 0)
-      (effects (font (size 1.27 1.27)) hide)
-    )
-    (property "Datasheet" "~" (id 3) (at 256.54 36.83 0)
-      (effects (font (size 1.27 1.27)) hide)
     )
     (pin "1")
@@
       (reference "#PWR025") (unit 1) (value "GND") (footprint "")
     )
-    (path "/f299e2a9-9c77-40ba-8d3a-4a4a5eeedaa8"
-      (reference "#PWR026") (unit 1) (value "GND") (footprint "")
-    )
     (path "/00000000-0000-0000-0000-0000624a2c8d"
       (reference "#PWR028") (unit 1) (value "GND") (footprint "")
@@
     )
     (path "/00000000-0000-0000-0000-00006248dce7"
-      (reference "C13") (unit 1) (value "C") (footprint "Capacitor_SMD:C_1206_3216Metric_Pad1.33x1.80mm_HandSolder")
+      (reference "C13") (unit 1) (value "C") (footprint "Capacitor_SMD:C_0805_2012Metric_Pad1.18x1.45mm_HandSolder")
     )
     (path "/03a53aed-e8a1-4f4a-9d56-d39951d6f91c"
@@
       (reference "C17") (unit 1) (value "C") (footprint "Capacitor_SMD:C_1206_3216Metric_Pad1.33x1.80mm_HandSolder")
     )
-    (path "/f578b530-5ba9-4c02-bd0d-6b9808b7fc70"
-      (reference "C18") (unit 1) (value "C") (footprint "Capacitor_SMD:C_1206_3216Metric_Pad1.33x1.80mm_HandSolder")
-    )
     (path "/55ec37cf-15cf-4b36-b24a-60d153216a17"
       (reference "C20") (unit 1) (value "C") (footprint "Capacitor_SMD:C_0603_1608Metric_Pad1.08x0.95mm_HandSolder")
@@
     )
     (path "/00000000-0000-0000-0000-00006248ba16"
-      (reference "R10") (unit 1) (value "R") (footprint "Resistor_SMD:R_0805_2012Metric_Pad1.20x1.40mm_HandSolder")
+      (reference "R10") (unit 1) (value "R") (footprint "Resistor_SMD:R_0603_1608Metric_Pad0.98x0.95mm_HandSolder")
     )
     (path "/6729f72e-30e4-4ec0-b909-52baa463595b"

Commit message: PCB on work
Parts:
- removed C1: C, Capacitor_SMD:C_1206_3216Metric, symbol Device:C
- removed C13: C, symbol Device:C
- removed C3: C, Capacitor_SMD:C_1206_3216Metric_Pad1.33x1.80mm_HandSolder, symbol Device:C
- C20: footprint Capacitor_SMD:C_0603_1608Metric_Pad1.08x0.95mm_HandSolder -> (none)
- R10: footprint (none) -> Resistor_SMD:R_0603_1608Metric_Pad0.98x0.95mm_HandSolder

Commit message: PCB underwork
Parts:
- removed C5: C, Capacitor_SMD:C_0603_1608Metric, symbol Device:C
- removed L2: TFM201610ALC-R47MTAA, libraries:INDC2016X80N, symbol TFM201610ALC-R47MTAA:TFM201610ALC-R47MTAA
- C15, C4, C6, C8, C9: footprint Capacitor_SMD:C_0603_1608Metric_Pad1.08x0.95mm_HandSolder -> (none)
- C20: footprint (none) -> Capacitor_SMD:C_1206_3216Metric_Pad1.33x1.80mm_HandSolder
- L4: footprint libraries:INDPM5752X300N -> (none)
- L7: footprint libraries:INDPM7366X500N -> (none)
- R10, R11, R4, R5, R7, R8, R9: footprint Resistor_SMD:R_0603_1608Metric_Pad0.98x0.95mm_HandSolder -> (none)
- R3: footprint Resistor_SMD:R_1206_3216Metric_Pad1.30x1.75mm_HandSolder -> (none)
Connections:
- net at C21.1, D1.1 (Conn), L10.1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: now also C11.1, L4.1

Commit message: PCB working on
Parts:
- removed C2: C, Capacitor_SMD:C_0603_1608Metric_Pad1.08x0.95mm_HandSolder, symbol Device:C
- removed L1: TFM201610ALC-R47MTAA, libraries:INDC2016X80N, symbol TFM201610ALC-R47MTAA:TFM201610ALC-R47MTAA
- C10, C20: footprint Capacitor_SMD:C_1206_3216Metric_Pad1.33x1.80mm_HandSolder -> (none)
- C15, C4, C6, C8, C9: footprint (none) -> Capacitor_SMD:C_0402_1005Metric_Pad0.74x0.62mm_HandSolder
- L3: footprint libraries:INDPM4441X200N -> (none)
- L4: footprint (none) -> libraries:INDPM4441X200N
- L7: footprint (none) -> libraries:INDPM5752X300N
- R10: footprint (none) -> Resistor_SMD:R_0603_1608Metric_Pad0.98x0.95mm_HandSolder
- R3: footprint (none) -> Resistor_SMD:R_0805_2012Metric_Pad1.20x1.40mm_HandSolder
- R4, R5, R7, R8, R9: footprint (none) -> Resistor_SMD:R_0402_1005Metric_Pad0.72x0.64mm_HandSolder
- U2, U3, U4, U5: footprint mount_holes:Hole_screw_M2 -> (none)
Connections:
- net at D2.1 (Conn), R2.1: now also C7.1, L3.1

Commit message: PCB working on
Parts:
- C10, C20: footprint (none) -> Capacitor_SMD:C_0805_2012Metric_Pad1.18x1.45mm_HandSolder
- L3: footprint (none) -> libraries:INDC2016X80N
- R11: footprint (none) -> Resistor_SMD:R_0603_1608Metric_Pad0.98x0.95mm_HandSolder
- U2, U3, U4, U5: footprint (none) -> mount_holes:Hole_screw_M1p2
Connections:
- net at R12.1: now also U1.7 (PB2); no longer U1.5 (AREF/PB0)
Changed lines of the file:
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@@
+    (stroke (width 0) (type default) (color 0 0 0 0))
+  )
+  (wire (pts (xy 412.75 105.41) (xy 412.75 100.33))
     (stroke (width 0) (type default) (color 0 0 0 0))
   )
@@
     (stroke (width 0) (type default) (color 0 0 0 0))
   )
+  (wire (pts (xy 412.75 100.33) (xy 422.91 100.33))
+    (stroke (width 0) (type default) (color 0 0 0 0))
+  )
+  (wire (pts (xy 406.4 105.41) (xy 412.75 105.41))
+    (stroke (width 0) (type default) (color 0 0 0 0))
+  )
   (wire (pts (xy 173.99 250.19) (xy 186.69 250.19))
     (stroke (width 0) (type default) (color 0 0 0 0))
@@
   )
   (wire (pts (xy 222.25 250.19) (xy 233.68 250.19))
-    (stroke (width 0) (type default) (color 0 0 0 0))
-  )
-  (wire (pts (xy 406.4 100.33) (xy 422.91 100.33))
     (stroke (width 0) (type default) (color 0 0 0 0))
   )
@@
       (effects (font (size 1.27 1.27)) (justify left))
     )
-    (property "Footprint" "" (id 2) (at 414.02 259.08 0)
+    (property "Footprint" "mount_holes:Hole_screw_M1p2" (id 2) (at 414.02 259.08 0)
       (effects (font (size 1.27 1.27)) hide)
     )
@@
     (property "Reference" "L3" (id 0) (at 161.29 223.52 0))
     (property "Value" "SRP4020TA-100M" (id 1) (at 161.29 226.06 0))
-    (property "Footprint" "" (id 2) (at 167.64 228.6 0)
+    (property "Footprint" "libraries:INDC2016X80N" (id 2) (at 167.64 228.6 0)
       (effects (font (size 1.27 1.27)) (justify left) hide)
     )
@@
       (effects (font (size 1.27 1.27)) (justify left))
     )
-    (property "Footprint" "" (id 2) (at 414.02 274.32 0)
+    (property "Footprint" "mount_holes:Hole_screw_M1p2" (id 2) (at 414.02 274.32 0)
       (effects (font (size 1.27 1.27)) hide)
     )
@@
       (effects (font (size 1.27 1.27)) (justify left))
     )
-    (property "Footprint" "" (id 2) (at 284.1752 265.43 0)
+    (property "Footprint" "Capacitor_SMD:C_0805_2012Metric_Pad1.18x1.45mm_HandSolder" (id 2) (at 284.1752 265.43 0)
       (effects (font (size 1.27 1.27)) hide)
     )
@@
       (effects (font (size 1.27 1.27)) (justify left))
     )
-    (property "Footprint" "" (id 2) (at 414.02 251.46 0)
+    (property "Footprint" "mount_holes:Hole_screw_M1p2" (id 2) (at 414.02 251.46 0)
       (effects (font (size 1.27 1.27)) hide)
     )
@@
       (effects (font (size 1.27 1.27)) (justify left))
     )
-    (property "Footprint" "" (id 2) (at 418.338 123.19 90)
+    (property "Footprint" "Resistor_SMD:R_0603_1608Metric_Pad0.98x0.95mm_HandSolder" (id 2) (at 418.338 123.19 90)
       (effects (font (size 1.27 1.27)) hide)
     )
@@
       (effects (font (size 1.27 1.27)) (justify left))
     )
-    (property "Footprint" "" (id 2) (at 414.02 266.7 0)
+    (property "Footprint" "mount_holes:Hole_screw_M1p2" (id 2) (at 414.02 266.7 0)
       (effects (font (size 1.27 1.27)) hide)
     )
@@
       (effects (font (size 1.27 1.27)) (justify left))
     )
-    (property "Footprint" "" (id 2) (at 177.4952 237.49 0)
-      (effects (font (size 1.27 1.27)) hide)
-    )
+    (property "Footprint" "Capacitor_SMD:C_0805_2012Metric_Pad1.18x1.45mm_HandSolder" (id 2) (at 177.4952 237.49 0)
+      (effects (font (size 1.27 1.27)) hide)
+    )
