File: Main_PCB_001/Main_PCB_001.kicad_sch (KiCad schematic)
At the start: 65 parts, among them IC1 FDN8601, IC2 FDN8601, IC3 TPS40211QDGQRQ1, IC4 PAM2863ECR, IC5 FDN8601, IC6 ZXTR2105FQ-7, U1 ATtiny25-20S, U2 Mounting_Hole_M2, U3 Mounting_Hole_M2, U4 Mounting_Hole_M2, U5 Mounting_Hole_M2

Commit message: PCB+Solidworks
Parts:
- D1, D2, D20, D3: footprint libraries:WireHole_1p5 -> (none)
Changed lines of the file:
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@@
       (effects (font (size 1.27 1.27)) (justify left))
     )
-    (property "Footprint" "libraries:WireHole_1p5" (id 2) (at 44.45 82.55 0)
+    (property "Footprint" "" (id 2) (at 44.45 82.55 0)
       (effects (font (size 1.27 1.27)) hide)
     )
@@
       (effects (font (size 1.27 1.27)) (justify left))
     )
-    (property "Footprint" "libraries:WireHole_1p5" (id 2) (at 453.39 101.6 0)
+    (property "Footprint" "" (id 2) (at 453.39 101.6 0)
       (effects (font (size 1.27 1.27)) hide)
     )
@@
       (effects (font (size 1.27 1.27)) (justify left))
     )
-    (property "Footprint" "libraries:WireHole_1p5" (id 2) (at 44.45 260.35 0)
+    (property "Footprint" "" (id 2) (at 44.45 260.35 0)
       (effects (font (size 1.27 1.27)) hide)
     )
@@
       (effects (font (size 1.27 1.27)) (justify left))
     )
-    (property "Footprint" "libraries:WireHole_1p5" (id 2) (at 44.45 228.6 0)
+    (property "Footprint" "" (id 2) (at 44.45 228.6 0)
       (effects (font (size 1.27 1.27)) hide)
     )
@@
     )
     (path "/5737afb7-2ca9-42d3-818e-4a8d58f1bfb1"
-      (reference "D1") (unit 1) (value "WireHole_1p5") (footprint "libraries:WireHole_1p5")
+      (reference "D1") (unit 1) (value "WireHole_1p5") (footprint "libraries:WireHole_1p2")
     )
     (path "/fdcf5a0b-5cc4-4a64-a579-df5462e72f5e"
-      (reference "D2") (unit 1) (value "WireHole_1p5") (footprint "libraries:WireHole_1p5")
+      (reference "D2") (unit 1) (value "WireHole_1p5") (footprint "libraries:WireHole_1p2")
     )
     (path "/a5704062-c423-49cd-af3a-ff4be8d176cc"
-      (reference "D3") (unit 1) (value "WireHole_1p5") (footprint "libraries:WireHole_1p5")
+      (reference "D3") (unit 1) (value "WireHole_1p5") (footprint "libraries:WireHole_1p2")
     )
     (path "/df9f7caa-4e64-4153-b6e2-37c443369569"
@@
     )
     (path "/7ffaf412-974d-4eab-86fd-7eec7991b7d2"
-      (reference "D20") (unit 1) (value "WireHole_1p5") (footprint "libraries:WireHole_1p5")
+      (reference "D20") (unit 1) (value "WireHole_1p5") (footprint "libraries:WireHole_1p2")
     )
     (path "/2c2af9fe-d6ab-4cfa-802b-05c089d70c5d"

Commit message: Corrections 001
Parts:
- removed IC5: FDN8601, libraries:SOT95P251X112-3N, symbol FDN8601:FDN8601
- added C1: C, Capacitor_SMD:C_0402_1005Metric_Pad0.74x0.62mm_HandSolder, symbol Device:C
- added Q1: (no value), symbol AON7407:AON7407
- C8: footprint Capacitor_SMD:C_0402_1005Metric_Pad0.74x0.62mm_HandSolder -> (none)
- D1, D2, D20, D3: footprint (none) -> libraries:WireHole_1p2
- R8, R9: footprint Resistor_SMD:R_0402_1005Metric_Pad0.72x0.64mm_HandSolder -> (none)
- Z3: value BZT52-C5V1J -> (none); footprint libraries:SOD3616X130N -> Diode_SMD:D_SOD-323F; symbol Main_PCB_001-rescue:BZT52-C5V1J-BZT52-C5V1J -> Diode:MM3Zxx
Connections:
- net GND: now also C1.2
- net at IC3.9 (BP): now also C1.1
- net at R8.2: now also Q1.4 (G)
- net at R10.1, R9.2: now also Q1.1 (S_1), Q1.2 (S_2), Q1.3 (S_3)
- net at D12.2, L7.2: now also Q1.5 (D_1), Q1.6 (D_2), Q1.7 (D_3), Q1.8 (D_4)
