File: Main_PCB_002/Main_PCB_001.kicad_sch (KiCad schematic)
At the start: 66 parts, among them IC1 FDN8601, IC2 FDN8601, IC3 TPS40211QDGQRQ1, IC4 PAM2863ECR, IC6 ZXTR2105FQ-7, U1 ATtiny25-20S, U2 Mounting_Hole_M2, U3 Mounting_Hole_M2, U4 Mounting_Hole_M2, U5 Mounting_Hole_M2

Commit message: Start 2nd version
Parts:
- added IC?: (no value), symbol LM5164QDDATQ1:LM5164QDDATQ1
- added U?: (no value), symbol Amplifier_Current:INA138
- C8: footprint (none) -> Capacitor_SMD:C_0402_1005Metric_Pad0.74x0.62mm_HandSolder
- Q1: value (none) -> AON7407; footprint (none) -> libraries:DFN_3X3_EP
- R8: footprint (none) -> Resistor_SMD:R_0402_1005Metric_Pad0.72x0.64mm_HandSolder
- R9: footprint (none) -> Resistor_SMD:R_0603_1608Metric_Pad0.98x0.95mm_HandSolder
- Z3: value (none) -> BZT52-C5V1J

Commit message: Underwork 001
Parts:
- removed D10: SS36, libraries:SODFL4626X120N, symbol SS36:SS36
- removed IC1, IC2: FDN8601, libraries:SOT95P251X112-3N, symbol FDN8601:FDN8601
- removed IC4: PAM2863ECR, libraries:SOIC127P600X175-9N, symbol PAM2863ECR:PAM2863ECR
- removed R1, R2: R, Resistor_SMD:R_0603_1608Metric_Pad0.98x0.95mm_HandSolder, symbol Device:R
- removed R6: R, Resistor_SMD:R_1206_3216Metric_Pad1.30x1.75mm_HandSolder, symbol Device:R
- removed Z1, Z2: BZT52-C12J, libraries:BZT52C12J, symbol BZT52-C12J:BZT52-C12J
- added C? (x2): C, Capacitor_SMD:C_0805_2012Metric_Pad1.18x1.45mm_HandSolder, symbol Device:C
- added R? (x2): (no value), symbol Device:R
- added R?: R, symbol Device:R
- IC?: value (none) -> LM5164QDDATQ1; footprint (none) -> SOIC127P600X170-9N
- U?: value (none) -> INA138; footprint (none) -> Package_TO_SOT_SMD:SOT-23-5
Connections:
- net GND: now also D15.1 (Conn), D3.1 (Conn), IC?.1 (GND), IC?.9 (EP), U?.2 (GND), C?.2, R?.1, R?.2
- net at C10.1, L3.2: now also IC?.2 (VIN), IC?.3 (EN/UVLO), U?.5 (V+)
- net at D11.1 (Conn): now also L9.2
- net at L8.1: now also IC?.8 (SW), C?.1
- net at C20.1, L8.2: now also U?.3 (+), R?.1; no longer L9.1
- net at IC?.4 (RON): now also R?.1
- net at IC?.5 (FB): now also U?.1, R?.2
- net at IC?.7 (BST): now also C?.2
- net at U?.4 (-): now also L9.1, C?.1, R?.2
Other:
- moved on the sheet: C20, D11, D13, D14, D15, IC?, L8, L9, U2, U3, U4, U5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
