File: Main_PCB_002/Module_of_protections_and_control/Protections_and_Control_module/_autosave-Protections_and_Control_module.kicad_sch (KiCad schematic)
At the start: 52 parts

Commit message: Modeling of ... . Modeling.
Parts:
- gave numbers to parts that had none: 52
Connections:
- net at C2.2, C3.2, C4.2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: no longer D4.1 (Conn), Q1.5 (D_1), Q1.6 (D_2), Q1.7 (D_3), Q1.8 (D_4)
- new net: D4.1 (Conn), Q1.5 (D_1), Q1.6 (D_2), Q1.7 (D_3), Q1.8 (D_4)
