File: Main_PCB_003/Main_PCB_001.kicad_pcb (KiCad board)
At the start: 4 copper layers, 55 x 15 mm, 55 parts, among them IC3 TPS40211QDGQRQ1, Q1 AON7407, U1 INA138, U2 Mounting_Hole_M2, U3 Mounting_Hole_M2, U4 Mounting_Hole_M2, U5 Mounting_Hole_M2

Commit message: Layering 002
Parts:
- added IC1: LM5164QDDATQ1, libraries:SOIC127P600X170-9N, F.Cu at (93.6, 139.7)
- moved R1 73.2 mm to (89.3, 141.3), turned to 90 degrees
- moved D2 71.9 mm to (84.6, 142.5)
- moved R6 62.7 mm to (97.9, 141.0), turned to -90 degrees
- moved R2 62.4 mm to (99.3, 137.6), turned to -90 degrees
- moved C2 58.9 mm to (98.0, 138.4), turned to -90 degrees
- moved U1 57.8 mm to (101.1, 140.8), turned to 180 degrees
- moved C20 56.1 mm to (99.6, 133.9), turned to 90 degrees
- moved C3 54.9 mm to (102.2, 133.9), turned to 90 degrees
- moved L8 54.3 mm to (95.2, 133.5)
- moved C7 47.2 mm to (89.1, 138.4), turned to -90 degrees
- moved L9 44.9 mm to (101.6, 137.7)
- moved C10 44.7 mm to (90.2, 133.9), turned to 90 degrees
- moved R8 23.1 mm to (80.1, 83.7)
- moved D4 0.33 mm to (101.6, 109.4)
- moved D5 0.33 mm to (103.0, 109.4)
Routing:
- net Net-(C10-Pad1): track 0.00 -> 16.5 mm
- net Net-(C20-Pad1): track 0.00 -> 13.6 mm
- net Net-(C2-Pad1): track 0.00 -> 8.28 mm
- net Net-(IC1-Pad5): track 0.00 -> 6.20 mm
- net Net-(C3-Pad1): track 0.00 -> 6.14 mm
- net Net-(C2-Pad2): track 0.00 -> 2.10 mm
- net Net-(IC1-Pad4): track 0.00 -> 2.02 mm
- net Net-(C10-Pad2): track 0.00 -> 1.37 mm

Commit message: Prototyping
Parts:
- removed IC3: TPS40211QDGQRQ1, libraries:SOP50P490X110-11N
- removed L8: SRP4020TA-100M, libraries:INDPM4441X200N
- removed L9: TFM201610ALC-R47MTAA, libraries:INDC2016X80N
- removed Z3: BZT52-C5V1J, Diode_SMD:D_SOD-323F
- added C13: C, Capacitor_SMD:C_1206_3216Metric_Pad1.33x1.80mm_HandSolder, F.Cu at (102.6, 68.9)
- added C18: C, Capacitor_SMD:C_1206_3216Metric_Pad1.33x1.80mm_HandSolder, F.Cu at (254.3, 108.0)
- added C19: C, Capacitor_SMD:C_0805_2012Metric_Pad1.18x1.45mm_HandSolder, F.Cu at (235.9, 76.0)
- added C21: C, Capacitor_SMD:C_1206_3216Metric_Pad1.33x1.80mm_HandSolder, F.Cu at (246.1, 120.9)
- added C5: C, Capacitor_SMD:C_0603_1608Metric_Pad1.08x0.95mm_HandSolder, F.Cu at (58.8, 55.4)
- added D17: WireHole_1p5, libraries:WireHole_1p2, F.Cu at (103.6, 91.5)
- added D18: WireHole_1p5, libraries:WireHole_1p2, F.Cu at (260.0, 111.0)
- added D19: WireHole_1p5, libraries:WireHole_1p2, F.Cu at (263.1, 107.5)
- added D21: SS36, libraries:SODFL4626X120N, F.Cu at (226.8, 115.4)
- added D22: WireHole_1p5, libraries:WireHole_1p2, F.Cu at (257.4, 111.0)
- added D23: WireHole_1p5, libraries:WireHole_1p2, F.Cu at (255.6, 113.9)
- added D24: LED_Cree_XHP50_6V, LED_SMD:LED_Cree-XHP50_6V, F.Cu at (233.4, 116.6)
- added D25: LED_Cree_XHP50_6V, LED_SMD:LED_Cree-XHP50_6V, F.Cu at (248.9, 103.1)
- added D26: LED_Cree_XHP50_6V, LED_SMD:LED_Cree-XHP50_6V, F.Cu at (239.8, 122.4)
- added D27: LED_Cree_XHP50_6V, LED_SMD:LED_Cree-XHP50_6V, F.Cu at (241.7, 109.5)
- added D28: LED_Cree_XHP50_6V, LED_SMD:LED_Cree-XHP50_6V, F.Cu at (255.4, 103.1)
- added D29: LED_Cree_XHP50_6V, LED_SMD:LED_Cree-XHP50_6V, F.Cu at (233.2, 123.0)
- added D30: LED_Cree_XHP50_6V, LED_SMD:LED_Cree-XHP50_6V, F.Cu at (226.7, 120.6)
- added D31: LED_Cree_XHP50_6V, LED_SMD:LED_Cree-XHP50_6V, F.Cu at (248.1, 109.5)
- added D32: LED_Cree_XHP50_6V, LED_SMD:LED_Cree-XHP50_6V, F.Cu at (246.3, 116.0)
- added D33: LED_Cree_XHP50_6V, LED_SMD:LED_Cree-XHP50_6V, F.Cu at (235.2, 108.9)
- added D34: LED_Cree_XHP50_6V, LED_SMD:LED_Cree-XHP50_6V, F.Cu at (242.5, 103.1)
- added D35: LED_Cree_XHP50_6V, LED_SMD:LED_Cree-XHP50_6V, F.Cu at (239.8, 116.0)
- added IC2: LM5164QDDATQ1, libraries:SOIC127P600X170-9N, F.Cu at (95.8, 147.7)
- added L1: TFM201610ALC-R47MTAA, libraries:INDC2016X80N, F.Cu at (99.2, 44.5)
- added L2: SRP7050AA-220M, libraries:INDPM5752X300N, F.Cu at (88.0, 62.1)
- added L3: SRP4020TA-100M, libraries:INDPM4441X200N, F.Cu at (109.7, 154.5)
- added L4: TFM201610ALC-R47MTAA, libraries:INDC2016X80N, F.Cu at (125.1, 139.5)
- added L5: TFM201610ALC-R47MTAA, libraries:INDC2016X80N, F.Cu at (259.6, 108.0)
- added Q2: AON7407, libraries:DFN_3X3_EP, F.Cu at (237.5, 65.2)
- added R11: R, Resistor_SMD:R_0805_2012Metric_Pad1.20x1.40mm_HandSolder, F.Cu at (251.9, 114.2)
- added R12: R, Resistor_SMD:R_0805_2012Metric_Pad1.20x1.40mm_HandSolder, F.Cu at (253.7, 111.1)
- added R13: R, Resistor_SMD:R_0805_2012Metric_Pad1.20x1.40mm_HandSolder, F.Cu at (261.0, 104.7)
- added Z1: BZT52-C5V1J, Diode_SMD:D_SOD-323F, F.Cu at (95.9, 77.3)
- added Z2: BZT52-C5V1J, Diode_SMD:D_SOD-323F, F.Cu at (251.2, 120.7)
- C1, C2, C4, C9: footprint Capacitor_SMD:C_0402_1005Metric_Pad0.74x0.62mm_HandSolder -> Capacitor_SMD:C_0805_2012Metric_Pad1.18x1.45mm_HandSolder
- C10, C12: footprint Capacitor_SMD:C_1206_3216Metric_Pad1.33x1.80mm_HandSolder -> Capacitor_SMD:C_0603_1608Metric_Pad1.08x0.95mm_HandSolder
- C11: footprint Capacitor_SMD:C_0603_1608Metric_Pad1.08x0.95mm_HandSolder -> Capacitor_SMD:C_0805_2012Metric_Pad1.18x1.45mm_HandSolder
- C14: footprint Capacitor_SMD:C_0603_1608Metric_Pad1.08x0.95mm_HandSolder -> Capacitor_SMD:C_0402_1005Metric_Pad0.74x0.62mm_HandSolder
- C15, C8: footprint Capacitor_SMD:C_0402_1005Metric_Pad0.74x0.62mm_HandSolder -> Capacitor_SMD:C_1206_3216Metric_Pad1.33x1.80mm_HandSolder
- C16, C7: footprint Capacitor_SMD:C_0603_1608Metric_Pad1.08x0.95mm_HandSolder -> Capacitor_SMD:C_1206_3216Metric_Pad1.33x1.80mm_HandSolder
- C17, C20, C3: footprint Capacitor_SMD:C_1206_3216Metric_Pad1.33x1.80mm_HandSolder -> Capacitor_SMD:C_0805_2012Metric_Pad1.18x1.45mm_HandSolder
- C6: footprint Capacitor_SMD:C_0402_1005Metric_Pad0.74x0.62mm_HandSolder -> Capacitor_SMD:C_0603_1608Metric_Pad1.08x0.95mm_HandSolder
- D10, D16: value WireHole_1p5 -> Wire_Pad_01; footprint libraries:WireHole_1p2 -> Flat_Wires_Pads:Wire_Hole_1mm
- D20: value WireHole_1p5 -> TX6211; footprint libraries:WireHole_1p2 -> XDS_Semi:TX6211
- D4, D5: value Wire_Pad_01 -> WireHole_1p5; footprint Flat_Wires_Pads:Wire_Hole_1mm -> libraries:WireHole_1p2
- IC1: value LM5164QDDATQ1 -> TPS40211QDGQRQ1; footprint libraries:SOIC127P600X170-9N -> libraries:SOP50P490X110-11N
- L6: footprint libraries:INDC2016X80N -> libraries:INDPM5752X300N
- L7: value SRP7050AA-220M -> TFM201610ALC-R47MTAA; footprint libraries:INDPM5752X300N -> libraries:INDC2016X80N
- R1, R2, R4, R6, R7, R8: footprint Resistor_SMD:R_0402_1005Metric_Pad0.72x0.64mm_HandSolder -> Resistor_SMD:R_0805_2012Metric_Pad1.20x1.40mm_HandSolder
- R10, R9: footprint Resistor_SMD:R_0603_1608Metric_Pad0.98x0.95mm_HandSolder -> Resistor_SMD:R_0402_1005Metric_Pad0.72x0.64mm_HandSolder
- moved L7 151.6 mm to (241.0, 52.5)
- moved U3 129.9 mm to (220.0, 47.2)
- moved L6 126.6 mm to (225.6, 59.2)
- moved C17 126.1 mm to (214.4, 70.1)
- moved C20 123.0 mm to (209.5, 78.5)
- moved D6 121.4 mm to (40.8, 58.0)
- moved U5 120.0 mm to (209.9, 60.9)
- moved D20 117.3 mm to (224.7, 69.9)
- moved D3 95.8 mm to (210.3, 74.4)
- moved R2 85.7 mm to (47.2, 69.5)
- moved U2 84.0 mm to (212.4, 52.7)
- moved D11 83.9 mm to (69.7, 104.3), turned to 0 degrees
- moved D14 82.4 mm to (150.3, 37.2), turned to 0 degrees
- moved D15 82.0 mm to (145.6, 33.6), turned to 0 degrees
- moved R1 80.4 mm to (54.6, 68.7)
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Connections:
- C11 pad 2: Net-(C1-Pad2) -> Net-(C10-Pad2)
- C12 pad 1: Net-(C11-Pad1) -> Net-(C12-Pad1)
- C12 pad 2: Net-(C1-Pad2) -> Net-(C10-Pad2)
- C14 pad 2: Net-(C1-Pad2) -> Net-(C14-Pad2)
- C15 pad 2: Net-(C1-Pad2) -> Net-(C15-Pad2)
- C16 pad 2: Net-(C1-Pad2) -> Net-(C15-Pad2)
- C17 pad 2: Net-(C1-Pad2) -> GND
- C2 pad 2: Net-(C2-Pad2) -> Net-(C1-Pad2)
- C20 pad 2: Net-(C10-Pad2) -> GND
- C3 pad 1: Net-(C3-Pad1) -> Net-(C10-Pad2)
- C3 pad 2: Net-(C10-Pad2) -> Net-(C3-Pad2)
- C4 pad 1: Net-(C4-Pad1) -> Net-(C10-Pad2)
- C6 pad 2: Net-(C4-Pad2) -> Net-(C15-Pad2)
- C7 pad 1: Net-(C10-Pad1) -> Net-(C6-Pad1)
- C7 pad 2: Net-(C10-Pad2) -> Net-(C15-Pad2)
- C8 pad 1: Net-(C1-Pad2) -> Net-(C5-Pad1)
- C8 pad 2: Net-(C8-Pad2) -> Net-(C10-Pad2)
- C9 pad 1: Net-(C1-Pad2) -> Net-(C9-Pad1)
- C9 pad 2: Net-(C9-Pad2) -> Net-(C10-Pad2)
- D1 pad 1: Net-(C11-Pad1) -> Net-(C10-Pad2)
- D10 pad 1: Net-(C1-Pad2) -> Net-(D10-Pad1)
- D11 pad 1: Net-(D11-Pad1) -> Net-(C10-Pad1)
- D12 pad 1: Net-(C17-Pad1) -> Net-(C13-Pad1)
- D14 pad 1: Net-(D13-Pad1) -> Net-(D14-Pad1)
- D15 pad 1: Net-(C10-Pad2) -> Net-(D14-Pad1)
- D16 pad 1: Net-(C10-Pad2) -> Net-(C15-Pad2)
- D2 pad 1: Net-(C10-Pad1) -> Net-(C15-Pad2)
- D20 pad 1: Net-(D20-Pad1) -> GND
- D4 pad 1: Net-(D4-Pad1) -> Net-(C5-Pad1)
- D5 pad 1: Net-(D5-Pad1) -> Net-(C6-Pad1)
- D6 pad 1: Net-(D5-Pad1) -> Net-(D6-Pad1)
- D9 pad 1: Net-(C14-Pad1) -> Net-(D10-Pad1)
- IC1 pad 1: Net-(C10-Pad2) -> Net-(C3-Pad2)
- IC1 pad 2: Net-(C10-Pad1) -> Net-(C4-Pad2)
- IC1 pad 3: Net-(C10-Pad1) -> Net-(D17-Pad1)
- IC1 pad 4: Net-(IC1-Pad4) -> Net-(C1-Pad2)
- IC1 pad 5: Net-(IC1-Pad5) -> Net-(C1-Pad1)
- IC1 pad 6: unconnected-(IC1-Pad6) -> Net-(C10-Pad2)
- IC1 pad 7: Net-(C2-Pad2) -> Net-(C11-Pad1)
- IC1 pad 8: Net-(C2-Pad1) -> Net-(IC1-Pad8)
- IC1 pad 9: Net-(C10-Pad2) -> Net-(C9-Pad1)
- L6 pad 1: Net-(C14-Pad1) -> Net-(C18-Pad1)
- L6 pad 2: Net-(C17-Pad1) -> Net-(D21-Pad2)
- L7 pad 1: Net-(C11-Pad1) -> Net-(C21-Pad1)
- L7 pad 2: Net-(D12-Pad2) -> Net-(D23-Pad1)
- R1 pad 1: Net-(IC1-Pad4) -> Net-(C10-Pad2)
- R1 pad 2: Net-(C10-Pad2) -> Net-(D6-Pad1)
- R10 pad 1: Net-(Q1-Pad1) -> Net-(C15-Pad2)
- R10 pad 2: Net-(C1-Pad2) -> Net-(IC2-Pad5)
- R2 pad 1: Net-(C20-Pad1) -> Net-(D6-Pad1)
- R2 pad 2: Net-(C3-Pad1) -> Net-(C1-Pad1)
- R3 pad 1: Net-(C1-Pad2) -> Net-(C1-Pad1)
- R3 pad 2: Net-(D4-Pad1) -> Net-(C2-Pad1)
- R4 pad 1: Net-(D4-Pad1) -> Net-(C3-Pad2)
- R4 pad 2: Net-(C4-Pad1) -> Net-(C12-Pad1)
- R5 pad 1: Net-(C4-Pad1) -> Net-(IC2-Pad4)
- R5 pad 2: Net-(C6-Pad1) -> Net-(C15-Pad2)
- R6 pad 1: Net-(C10-Pad2) -> Net-(IC1-Pad8)
- R6 pad 2: Net-(IC1-Pad5) -> Net-(Q1-Pad4)
- R7 pad 1: Net-(C8-Pad2) -> Net-(C11-Pad1)
- R7 pad 2: Net-(C16-Pad1) -> Net-(Q1-Pad1)
- R8 pad 1: Net-(IC3-Pad8) -> Net-(Q1-Pad1)
- R8 pad 2: Net-(Q1-Pad4) -> Net-(C10-Pad2)
- R9 pad 2: Net-(Q1-Pad1) -> Net-(C16-Pad1)
- U1 pad 1: Net-(IC1-Pad5) -> Net-(IC2-Pad5)
- U1 pad 2: Net-(C10-Pad2) -> Net-(C15-Pad2)
- U1 pad 3: Net-(C20-Pad1) -> Net-(C15-Pad1)
- U1 pad 4: Net-(C3-Pad1) -> Net-(C16-Pad1)
- U1 pad 5: Net-(C10-Pad1) -> Net-(C6-Pad1)
Routing:
- net Net-(D13-Pad1): track 113.5 -> 0.00 mm, vias 4 -> 0
- net Net-(C10-Pad1): track 16.5 -> 0.00 mm
- net Net-(C20-Pad1): track 13.6 -> 0.00 mm
- net Net-(D5-Pad1): track 12.5 -> 0.00 mm, vias 3 -> 0
- net Net-(D7-Pad1): track 11.3 -> 0.00 mm, vias 2 -> 0
- net Net-(C2-Pad1): track 8.28 -> 0.00 mm
- net Net-(IC1-Pad5): track 6.20 -> 0.00 mm
- net Net-(C3-Pad1): track 6.14 -> 0.00 mm
- net Net-(C2-Pad2): track 2.10 -> 0.00 mm
- net Net-(IC1-Pad4): track 2.02 -> 0.00 mm
- net Net-(C14-Pad1): track 1.38 -> 0.00 mm, vias 1 -> 0
- net Net-(C10-Pad2): track 1.37 -> 0.00 mm
- net GND: vias 3 -> 0
Other:
- board outline removed

Commit message: Prototyping
Parts:
- moved D13 46.3 mm to (108.3, 157.9)
- moved D5 33.4 mm to (110.1, 142.1)
- moved D2 32.4 mm to (116.8, 146.2)
- moved D16 25.7 mm to (113.4, 152.0)
- moved L4 24.1 mm to (106.1, 154.4)
- moved C7 23.0 mm to (104.4, 146.6), turned to 0 degrees
- moved R9 17.7 mm to (101.2, 154.7)
- moved C6 15.7 mm to (102.8, 149.4)
- moved L3 15.6 mm to (95.3, 148.3), turned to 180 degrees
- moved C16 13.5 mm to (105.9, 150.7), turned to 90 degrees
- moved C15 11.9 mm to (90.9, 148.3), turned to -90 degrees
- moved U1 11.8 mm to (102.1, 152.1), turned to 0 degrees
- moved R5 11.7 mm to (100.6, 146.2), turned to -90 degrees
- moved R10 11.3 mm to (100.5, 149.0), turned to -90 degrees
- moved C14 7.34 mm to (97.9, 152.0), turned to -90 degrees
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Connections:
- C20 pad 1: Net-(C20-Pad1) -> Net-(C18-Pad1)
- C5 pad 1: Net-(C5-Pad1) -> Net-(C12-Pad1)
- C8 pad 1: Net-(C5-Pad1) -> Net-(C12-Pad1)
- D20 pad 2: Net-(C20-Pad1) -> Net-(C18-Pad1)
- D20 pad 8: Net-(C20-Pad1) -> Net-(C18-Pad1)
- D4 pad 1: Net-(C5-Pad1) -> Net-(C12-Pad1)
- L2 pad 1: Net-(C5-Pad1) -> Net-(C12-Pad1)
