File: Main_PCB_003/Main_PCB_001.kicad_sch (KiCad schematic)
At the start: 56 parts, among them IC1 LM5164QDDATQ1, IC3 TPS40211QDGQRQ1, Q1 AON7407, U1 INA138, U2 Mounting_Hole_M2, U3 Mounting_Hole_M2, U4 Mounting_Hole_M2, U5 Mounting_Hole_M2

Commit message: Layering 002
Parts:
- C10, C20, C3: footprint (none) -> Capacitor_SMD:C_1206_3216Metric_Pad1.33x1.80mm_HandSolder
- C2: footprint (none) -> Capacitor_SMD:C_0402_1005Metric_Pad0.74x0.62mm_HandSolder
- D11, D13, D14, D15, D4, D5, D6, D7, D8, D9: footprint (none) -> Flat_Wires_Pads:Wire_Hole_1mm
- IC1: footprint SOIC127P600X170-9N -> libraries:SOIC127P600X170-9N
- R1, R2, R6: footprint (none) -> Resistor_SMD:R_0402_1005Metric_Pad0.72x0.64mm_HandSolder
Connections:
- net GND: no longer IC1.1 (GND)
- net at C10.2, C20.2, C3.2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: now also IC1.1 (GND)
Other:
- moved on the sheet: C10, C7

Commit message: Prototyping
Parts:
- added C13, C21: C, Capacitor_SMD:C_1206_3216Metric_Pad1.33x1.80mm_HandSolder, symbol Device:C
- added C18: (no value), symbol Device:C
- added C19, C5: C, symbol Device:C
- added D17, D18, D22, D23: WireHole_1p5, libraries:WireHole_1p2, symbol Connectors_for_Wire:WireHole_1p5
- added D19: (no value), symbol XDS_Semi:TX6211
- added D21: SS36, libraries:SODFL4626X120N, symbol SS36:SS36
- added D24: (no value), symbol LED:LED_Cree_XHP50_6V
- added D25, D26, D27, D28, D29, D30, D31, D32, D33, D34, D35: LED_Cree_XHP50_6V, LED_SMD:LED_Cree-XHP50_6V, symbol LED:LED_Cree_XHP50_6V
- added L1, L2: TFM201610ALC-R47MTAA, libraries:INDC2016X80N, symbol TFM201610ALC-R47MTAA:TFM201610ALC-R47MTAA
- added Q2: AON7407, libraries:DFN_3X3_EP, symbol AON7407:AON7407
- added R11, R12: R, symbol Device:R
- added R13: (no value), symbol Device:R
- added Z1: BZT52-C5V1J, Diode_SMD:D_SOD-323F, symbol Diode:MM3Zxx
Connections:
- net GND: now also C13.2, C18.2, C19.2, C21.2, C5.2, D18.1 (Conn), D19.1 (GND), R11.2, R13.2
- new net: D23.1 (Conn), D35.1 (K), R12.2, R13.1
- new net: D33.1 (K), D34.2 (A)
- new net: D32.1 (K), D33.2 (A)
- new net: D34.1 (K), D35.2 (A)
- new net: D30.1 (K), D31.2 (A)
- new net: D29.1 (K), D30.2 (A)
- new net: C13.1, L1.2, L2.1
- new net: D21.2, L2.2, Q2.5 (D_1), Q2.6 (D_2), Q2.7 (D_3), Q2.8 (D_4)
- new net: D24.1 (K), D25.2 (A)
- new net: C21.1, D21.1, D22.1 (Conn), D24.2 (A), Z1.1 (K)
- new net: D25.1 (K), D26.2 (A)
- new net: D28.1 (K), D29.2 (A)
- new net: C19.1, D19.2 (En), D19.8 (Vdd)
- new net: C5.1, D19.3 (Comp)
- new net: D19.4 (VFB), R12.1, Z1.2 (A)
- new net: D19.5 (DRV), Q2.4 (G)
- new net: D19.6 (ICS), Q2.1 (S_1), Q2.2 (S_2), Q2.3 (S_3), R11.1
- new net: C18.1, D19.7 (TOFF)
- new net: D31.1 (K), D32.2 (A)
- new net: D26.1 (K), D27.2 (A)
- new net: D17.1 (Conn), L1.1
- new net: D27.1 (K), D28.2 (A)

Commit message: Prototyping
Parts:
- added L7: TFM201610ALC-R47MTAA, libraries:INDC2016X80N, symbol TFM201610ALC-R47MTAA:TFM201610ALC-R47MTAA
- C1: renamed from C4; footprint Capacitor_SMD:C_0402_1005Metric_Pad0.74x0.62mm_HandSolder -> Capacitor_SMD:C_0805_2012Metric_Pad1.18x1.45mm_HandSolder
- C11: renamed from C15; footprint Capacitor_SMD:C_0402_1005Metric_Pad0.74x0.62mm_HandSolder -> Capacitor_SMD:C_0805_2012Metric_Pad1.18x1.45mm_HandSolder
- C17: renamed from C5; footprint (none) -> Capacitor_SMD:C_0805_2012Metric_Pad1.18x1.45mm_HandSolder
- C19: renamed from C18; value (none) -> C; footprint (none) -> Capacitor_SMD:C_0805_2012Metric_Pad1.18x1.45mm_HandSolder
- C2: renamed from C6; footprint Capacitor_SMD:C_0402_1005Metric_Pad0.74x0.62mm_HandSolder -> Capacitor_SMD:C_0805_2012Metric_Pad1.18x1.45mm_HandSolder
- C20: renamed from C19; footprint (none) -> Capacitor_SMD:C_0805_2012Metric_Pad1.18x1.45mm_HandSolder
- C3: renamed from C8; footprint Capacitor_SMD:C_0402_1005Metric_Pad0.74x0.62mm_HandSolder -> Capacitor_SMD:C_0805_2012Metric_Pad1.18x1.45mm_HandSolder
- C4: renamed from C9; footprint Capacitor_SMD:C_0402_1005Metric_Pad0.74x0.62mm_HandSolder -> Capacitor_SMD:C_0805_2012Metric_Pad1.18x1.45mm_HandSolder
- C9: renamed from C1; footprint Capacitor_SMD:C_0402_1005Metric_Pad0.74x0.62mm_HandSolder -> Capacitor_SMD:C_0805_2012Metric_Pad1.18x1.45mm_HandSolder
- D20: renamed from D19; value (none) -> TX6211; footprint (none) -> XDS_Semi:TX6211
- D24: value (none) -> LED_Cree_XHP50_6V; footprint (none) -> LED_SMD:LED_Cree-XHP50_6V
- L6: renamed from L2; footprint libraries:INDC2016X80N -> libraries:INDPM5752X300N
- R11, R12: footprint (none) -> Resistor_SMD:R_0805_2012Metric_Pad1.20x1.40mm_HandSolder
- R13: value (none) -> R; footprint (none) -> Resistor_SMD:R_0805_2012Metric_Pad1.20x1.40mm_HandSolder
- R2: renamed from R4; footprint Resistor_SMD:R_0402_1005Metric_Pad0.72x0.64mm_HandSolder -> Resistor_SMD:R_0805_2012Metric_Pad1.20x1.40mm_HandSolder
- R3: renamed from R5; footprint Resistor_SMD:R_0402_1005Metric_Pad0.72x0.64mm_HandSolder -> Resistor_SMD:R_0805_2012Metric_Pad1.20x1.40mm_HandSolder
- R4: renamed from R7; footprint Resistor_SMD:R_0402_1005Metric_Pad0.72x0.64mm_HandSolder -> Resistor_SMD:R_0805_2012Metric_Pad1.20x1.40mm_HandSolder
- R6: renamed from R8; footprint Resistor_SMD:R_0402_1005Metric_Pad0.72x0.64mm_HandSolder -> Resistor_SMD:R_0805_2012Metric_Pad1.20x1.40mm_HandSolder
- R7: renamed from R9; footprint Resistor_SMD:R_0603_1608Metric_Pad0.98x0.95mm_HandSolder -> Resistor_SMD:R_0805_2012Metric_Pad1.20x1.40mm_HandSolder
- R8: renamed from R10; footprint Resistor_SMD:R_0603_1608Metric_Pad0.98x0.95mm_HandSolder -> Resistor_SMD:R_0805_2012Metric_Pad1.20x1.40mm_HandSolder
- renumbered C14 to C10, C16 to C12, C17 to C13, C2 to C14, C20 to C15, C3 to C16, C13 to C18, C11 to C5, C7 to C6, C10 to C7, C12 to C8, D10 to D1, D8 to D10, D9 to D11, D11 to D13, D13 to D14, D14 to D15, D15 to D16, D20 to D17, D17 to D18, D18 to D19, D16 to D2, D23 to D22, D22 to D23, D1 to D4, D2 to D5, D4 to D6, D5 to D7, D6 to D8, D7 to D9, IC3 to IC1, IC1 to IC2, L6 to L1, L7 to L2, L8 to L3, L9 to L4, L1 to L5, R3 to R1, R6 to R10, R1 to R5, R2 to R9, Z3 to Z1, Z1 to Z2
Connections:
- net at C21.1, D21.1, Z2.1 (K): now also L7.1; no longer D23.1 (Conn), D24.2 (A)
- new net: D23.1 (Conn), D24.2 (A), L7.2
Other:
- moved on the sheet: D23

Commit message: Prototyping
Connections:
- net at C12.1, IC1.10 (VDD), R4.2: now also C5.1, C8.1, D4.1 (Conn), L2.1
- net at C18.1, L5.2, L6.1: now also C20.1, D20.2 (En), D20.8 (Vdd)
Other:
- moved on the sheet: C10, C13, C8, D1, D10, D11, D17, D4, D6, D7, D8, D9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

Commit message: Prototyping
Parts:
- added C22: C, symbol Device:C
- L4: footprint libraries:INDC2016X80N -> (none)
- R10, R5, R9: footprint Resistor_SMD:R_0402_1005Metric_Pad0.72x0.64mm_HandSolder -> (none)
Connections:
- net at C15.2, C16.2, C6.2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: now also C22.2
- net at C6.1, C7.1, D5.1 (Conn)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: now also C22.1
Changed lines of the file:
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@@
   (junction (at 224.79 184.15) (diameter 0) (color 0 0 0 0)
   )
+  (junction (at 285.75 284.48) (diameter 0) (color 0 0 0 0)
+  )
   (junction (at 148.59 140.97) (diameter 0) (color 0 0 0 0)
   )
@@
   (junction (at 525.78 31.75) (diameter 0) (color 0 0 0 0)
   )
+  (junction (at 288.29 251.46) (diameter 0) (color 0 0 0 0)
+  )
   (junction (at 495.3 289.56) (diameter 0) (color 0 0 0 0)
   )
@@
     (stroke (width 0) (type default) (color 0 0 0 0))
   )
-  (wire (pts (xy 276.86 284.48) (xy 295.91 284.48))
+  (wire (pts (xy 276.86 284.48) (xy 285.75 284.48))
     (stroke (width 0) (type default) (color 0 0 0 0))
   )
@@
     (stroke (width 0) (type default) (color 0 0 0 0))
   )
+  (wire (pts (xy 285.75 276.86) (xy 285.75 284.48))
+    (stroke (width 0) (type default) (color 0 0 0 0))
+  )
   (wire (pts (xy 525.78 120.65) (xy 523.24 120.65))
     (stroke (width 0) (type default) (color 0 0 0 0))
@@
     (stroke (width 0) (type default) (color 0 0 0 0))
   )
+  (wire (pts (xy 285.75 269.24) (xy 285.75 251.46))
+    (stroke (width 0) (type default) (color 0 0 0 0))
+  )
   (wire (pts (xy 604.52 99.06) (xy 604.52 125.73))
     (stroke (width 0) (type default) (color 0 0 0 0))
@@
     (stroke (width 0) (type default) (color 0 0 0 0))
   )
+  (wire (pts (xy 285.75 251.46) (xy 288.29 251.46))
+    (stroke (width 0) (type default) (color 0 0 0 0))
+  )
   (wire (pts (xy 171.45 137.16) (xy 179.07 137.16))
     (stroke (width 0) (type default) (color 0 0 0 0))
@@
     (stroke (width 0) (type default) (color 0 0 0 0))
   )
+  (wire (pts (xy 285.75 284.48) (xy 295.91 284.48))
+    (stroke (width 0) (type default) (color 0 0 0 0))
+  )
   (wire (pts (xy 504.19 124.46) (xy 501.65 124.46))
     (stroke (width 0) (type default) (color 0 0 0 0))
@@
     (property "Reference" "R9" (id 0) (at 295.91 237.49 90))
     (property "Value" "R" (id 1) (at 295.91 240.03 90))
-    (property "Footprint" "Resistor_SMD:R_0402_1005Metric_Pad0.72x0.64mm_HandSolder" (id 2) (at 295.91 245.618 90)
+    (property "Footprint" "" (id 2) (at 295.91 245.618 90)
       (effects (font (size 1.27 1.27)) hide)
     )
@@
     (property "Reference" "L4" (id 0) (at 335.28 237.49 0))
     (property "Value" "TFM201610ALC-R47MTAA" (id 1) (at 335.28 240.03 0))
-    (property "Footprint" "libraries:INDC2016X80N" (id 2) (at 341.63 242.57 0)
+    (property "Footprint" "" (id 2) (at 341.63 242.57 0)
       (effects (font (size 1.27 1.27)) (justify left) hide)
     )
@@
     (pin "1")
   )
+  (symbol (lib_id "Device:C") (at 285.75 273.05 0) (unit 1)
+    (in_bom yes) (on_board yes)
+    (property "Reference" "C22" (id 0) (at 288.671 271.8816 0)
+      (effects (font (size 1.27 1.27)) (justify left))
+    )
+    (property "Value" "C" (id 1) (at 288.671 274.193 0)
+      (effects (font (size 1.27 1.27)) (justify left))
+    )
+    (property "Footprint" "" (id 2) (at 286.7152 276.86 0)
+      (effects (font (size 1.27 1.27)) hide)
+    )
+    (property "Datasheet" "~" (id 3) (at 285.75 273.05 0)
+      (effects (font (size 1.27 1.27)) hide)
+    )
+    (pin "1")
+    (pin "2")
+  )
   (symbol (lib_id "Device:R") (at 618.49 125.73 90) (unit 1)
     (in_bom yes) (on_board yes) (fields_autoplaced)
@@
       (effects (font (size 1.27 1.27)) (justify right))
     )
-    (property "Footprint" "Resistor_SMD:R_0402_1005Metric_Pad0.72x0.64mm_HandSolder" (id 2) (at 297.688 270.51 90)
+    (property "Footprint" "" (id 2) (at 297.688 270.51 90)
       (effects (font (size 1.27 1.27)) hide)
     )
@@
       (effects (font (size 1.27 1.27)) (justify left))
     )
-    (property "Footprint" "Resistor_SMD:R_0402_1005Metric_Pad0.72x0.64mm_HandSolder" (id 2) (at 207.772 265.43 90)
+    (property "Footprint" "" (id 2) (at 207.772 265.43 90)
       (effects (font (size 1.27 1.27)) hide)
     )
@@
       (reference "C21") (unit 1) (value "C") (footprint "Capacitor_SMD:C_1206_3216Metric_Pad1.33x1.80mm_HandSolder")
     )
+    (path "/789d3f5b-3534-4e8a-89c9-ca398e75eeeb"
+      (reference "C22") (unit 1) (value "C") (footprint "Capacitor_SMD:C_0402_1005Metric_Pad0.74x0.62mm_HandSolder")
+    )
     (path "/0c3aa802-ed3b-4a37-847a-7535c56a8e9b"
       (reference "D1") (unit 1) (value "WireHole_1p5") (footprint "libraries:WireHole_1p2")
@@
     )
     (path "/5195d6f0-e9e1-4174-bc28-ceaf9e3afdfe"
-      (reference "L4") (unit 1) (value "TFM201610ALC-R47MTAA") (footprint "libraries:INDC2016X80N")
+      (reference "L4") (unit 1) (value "TFM201610ALC-R47MTAA") (footprint "libraries:WPN252010UR47MT")
     )
     (path "/95cfb089-c199-4836-9ffe-c3c7057df2f8"
@@
     )
     (path "/f8349e20-f50b-409d-b70f-d46b045c76a3"
-      (reference "R5") (unit 1) (value "R") (footprint "Resistor_SMD:R_0402_1005Metric_Pad0.72x0.64mm_HandSolder")
+      (reference "R5") (unit 1) (value "R") (footprint "Resistor_SMD:R_0805_2012Metric_Pad1.20x1.40mm_HandSolder")
     )
     (path "/00000000-0000-0000-0000-00006248b6d6"
@@
     )
     (path "/4741c2f9-3aad-4ec5-93d7-cfe712a42a5a"
-      (reference "R9") (unit 1) (value "R") (footprint "Resistor_SMD:R_0402_1005Metric_Pad0.72x0.64mm_HandSolder")
+      (reference "R9") (unit 1) (value "R") (footprint "Resistor_SMD:R_0805_2012Metric_Pad1.20x1.40mm_HandSolder")
     )
     (path "/a82ed511-da4c-4b63-9d60-585267c54cae"
-      (reference "R10") (unit 1) (value "R") (footprint "Resistor_SMD:R_0402_1005Metric_Pad0.72x0.64mm_HandSolder")
+      (reference "R10") (unit 1) (value "R") (footprint "Resistor_SMD:R_0805_2012Metric_Pad1.20x1.40mm_HandSolder")
     )
     (path "/deb57808-2041-4e7e-ac2d-51b09e0e2aad"
