File: Main_PCB_003/Main_PCB_002.kicad_pcb (KiCad board)
At the start: 4 copper layers, 88 parts, among them IC1 TPS40211QDGQRQ1, IC2 LM5164QDDATQ1, Q1 AON7407, Q2 AON7407, U1 INA138, U2 Mounting_Hole_M2, U3 Mounting_Hole_M2, U4 Mounting_Hole_M2, U5 Mounting_Hole_M2

Commit message: Prototyping
Parts:
- moved D13 23.2 mm to (105.4, 146.3)
- moved L4 18.1 mm to (103.3, 149.0), turned to 0 degrees
- moved C16 14.3 mm to (99.6, 148.6), turned to 90 degrees
- moved R9 12.6 mm to (100.4, 152.1)
- moved U1 11.9 mm to (99.7, 154.8)
- moved C22 10.9 mm to (99.2, 157.1)
- moved C15 7.71 mm to (90.9, 148.3)
- moved C7 6.14 mm to (88.4, 148.3), turned to 90 degrees
- moved D16 5.55 mm to (105.0, 151.9)
- moved R10 4.95 mm to (103.3, 154.5)
- moved D5 2.87 mm to (85.9, 149.5)
- moved D2 2.71 mm to (86.2, 153.7)
- moved C6 0.85 mm to (88.1, 151.8), turned to 180 degrees
- moved L3 0.84 mm to (95.2, 148.3), turned to 0 degrees
Routing:
- net Net-(C15-Pad1): track 9.95 -> 21.8 mm
- net Net-(IC2-Pad5): track 12.7 -> 7.57 mm
- net Net-(C6-Pad1): track 14.7 -> 18.6 mm
- net Net-(D13-Pad1): track 2.20 -> 0.00 mm
- net Net-(C15-Pad2): track 3.78 -> 5.55 mm, vias 30 -> 0
- net Net-(C14-Pad1): track 4.65 -> 6.40 mm

Commit message: Prototyping 6 001
Parts:
- moved D6 50.4 mm to (76.2, 93.9)
- moved L1 45.7 mm to (93.0, 89.8), turned to 180 degrees
- moved R2 39.0 mm to (78.6, 92.7), turned to 90 degrees
- moved C5 35.5 mm to (82.6, 81.8), turned to -90 degrees
- moved R1 35.5 mm to (80.7, 92.7), turned to -90 degrees
- moved R8 33.3 mm to (89.0, 92.3), turned to -90 degrees
- moved D17 32.2 mm to (71.6, 87.6)
- moved D12 31.8 mm to (93.1, 83.2), turned to 90 degrees
- moved D4 29.5 mm to (77.4, 80.8)
- moved D11 25.6 mm to (93.1, 93.8)
- moved L2 21.0 mm to (87.6, 83.1)
- moved C13 20.4 mm to (93.8, 87.3)
- moved Z1 20.0 mm to (82.9, 92.6), turned to 90 degrees
- moved Q1 19.6 mm to (89.4, 88.5)
- moved C12 18.8 mm to (82.7, 85.3), turned to 90 degrees
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Connections:
- Q1 pad 10: (no net) -> Net-(D12-Pad2)
- Q1 pad 11: (no net) -> Net-(D12-Pad2)
- Q1 pad 9: (no net) -> Net-(D12-Pad2)
Routing:
- net Net-(C13-Pad1): track 0.00 -> 18.4 mm
- net Net-(C12-Pad1): track 0.00 -> 13.8 mm
- net Net-(D17-Pad1): track 0.00 -> 12.1 mm
- net Net-(C1-Pad1): track 0.00 -> 10.4 mm
- net Net-(Q1-Pad4): track 0.00 -> 9.43 mm
- net Net-(C11-Pad1): track 0.00 -> 8.24 mm
- net Net-(D12-Pad2): track 0.00 -> 7.73 mm
- net Net-(Q1-Pad1): track 0.00 -> 4.76 mm
- net Net-(D6-Pad1): track 0.00 -> 4.56 mm
- net Net-(C10-Pad1): track 0.00 -> 4.39 mm
- net Net-(C1-Pad2): track 0.00 -> 4.21 mm
- net Net-(C3-Pad2): track 0.00 -> 3.77 mm
- net Net-(C9-Pad1): track 0.00 -> 2.54 mm
- net Net-(IC1-Pad8): track 0.00 -> 2.52 mm
- net Net-(C4-Pad2): track 0.00 -> 2.25 mm
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