File: Main_PCB_003/Main_PCB_002.kicad_sch (KiCad schematic)
At the start: 240 parts, among them IC1 TPS40211QDGQRQ1, IC2 LM5164QDDATQ1, IC3 LM3481MM_NOPB, IC4 LM3488MM, IC5 LM3478MMX_NOPB, Q1 AON7407, Q2 AON7407, Q3 AON7407, Q4 AON7407, Q5 AON7407, U1 INA138, U10 MCP9700AT-ETT, U11 MCP9700AT-ETT, U12 MCP9700AT-ETT, U13 MCP9700AT-ETT, U14 INA138, U15 MCP9700AT-ETT, U16 MCP9700AT-ETT, U17 MCP9700AT-ETT, U18 MCP9700AT-ETT, U19 MCP9700AT-ETT, U2 Mounting_Hole_M2, U20 MCP9700AT-ETT, U21 INA138, U22 MCP9700AT-ETT, U23 MCP9700AT-ETT, U3 Mounting_Hole_M2, U4 Mounting_Hole_M2, U5 Mounting_Hole_M2, U6 INA138, U7 INA138, U8 INA138, U9 MCP9700AT-ETT

Commit message: Prototyping 6 001
Parts:
- removed C46, C47, C48, C49, C50, C51, C52, C53, C54, C55, C56, C57, C58, C59, C60: C, Capacitor_SMD:C_0805_2012Metric_Pad1.18x1.45mm_HandSolder, symbol Device:C
- removed D59, D62, D66, D74, D80, D84, D95: +5B, libraries:WireHole_1p2, symbol Connectors_for_Wire:WireHole_1p5
- removed D60: t_IC, libraries:WireHole_1p2, symbol Connectors_for_Wire:WireHole_1p5
- removed D61, D65, D69, D77, D83, D87: Gnd, libraries:WireHole_1p2, symbol Connectors_for_Wire:WireHole_1p5
- removed D63, D67, D75, D81, D85: t_D, libraries:WireHole_1p2, symbol Connectors_for_Wire:WireHole_1p5
- removed D64, D68, D76, D82, D86: t_Q, libraries:WireHole_1p2, symbol Connectors_for_Wire:WireHole_1p5
- removed D70, D79: CS_In, Flat_Wires_Pads:Wire_Hole_1mm, symbol Connectors_for_Wire:Wire_Pad_01
- removed D71, D88: CS_Out, Flat_Wires_Pads:Wire_Hole_1mm, symbol Connectors_for_Wire:Wire_Pad_01
- removed D72, D89: Gnd, Flat_Wires_Pads:Wire_Hole_1mm, symbol Connectors_for_Wire:Wire_Pad_01
- removed D73, D90: U, Flat_Wires_Pads:Wire_Hole_1mm, symbol Connectors_for_Wire:Wire_Pad_01
- removed D78, D91: I, Flat_Wires_Pads:Wire_Hole_1mm, symbol Connectors_for_Wire:Wire_Pad_01
- removed D92: +5V, libraries:WireHole_1p2, symbol Connectors_for_Wire:WireHole_1p5
- removed D93: t LED, libraries:WireHole_1p2, symbol Connectors_for_Wire:WireHole_1p5
- removed D94, D97: GND, libraries:WireHole_1p2, symbol Connectors_for_Wire:WireHole_1p5
- removed D96: t_LED, libraries:WireHole_1p2, symbol Connectors_for_Wire:WireHole_1p5
- removed R31, R32, R33, R34, R35, R36, R37, R38: R, Resistor_SMD:R_0805_2012Metric_Pad1.20x1.40mm_HandSolder, symbol Device:R
- removed U10, U11, U12, U13, U15, U16, U17, U18, U19, U20, U22, U23, U9: MCP9700AT-ETT, Package_TO_SOT_SMD:SOT-23, symbol Sensor_Temperature:MCP9700AT-ETT
- removed U14, U21: INA138, Package_TO_SOT_SMD:SOT-23-5, symbol Amplifier_Current:INA138
- C1, C11, C17, C19, C2, C20, C23, C24, C25, C27, C28, C3, C30, C32, C33, C36, C37, C38, C39, C4, C42, C43, C9: value C -> (none); footprint Capacitor_SMD:C_0805_2012Metric_Pad1.18x1.45mm_HandSolder -> (none)
- C10, C12, C5, C6: value C -> (none); footprint Capacitor_SMD:C_0603_1608Metric_Pad1.08x0.95mm_HandSolder -> (none)
- C13, C15, C16, C18, C21, C26, C29, C34, C35, C40, C41, C7, C8: value C -> (none); footprint Capacitor_SMD:C_1206_3216Metric_Pad1.33x1.80mm_HandSolder -> (none)
- C14, C22, C31, C44, C45: value C -> (none); footprint Capacitor_SMD:C_0402_1005Metric_Pad0.74x0.62mm_HandSolder -> (none)
- D1, D17, D18, D19, D2, D22, D23, D3, D36, D37, D4, D43, D44, D5, D55, D56, D57: value WireHole_1p5 -> (none); footprint libraries:WireHole_1p2 -> (none)
- D10, D11, D13, D14, D15, D16, D39, D53, D54, D6, D7, D8, D9: value Wire_Pad_01 -> (none); footprint Flat_Wires_Pads:Wire_Hole_1mm -> (none)
- D12, D21, D38, D45, D46: value SS36 -> (none); footprint libraries:SODFL4626X120N -> (none)
- D20: value TX6211 -> (none); footprint XDS_Semi:TX6211 -> (none)
- D24, D25, D26, D27, D28, D29, D30, D31, D32, D33, D34, D35, D47, D48, D49: value LED_Cree_XHP50_6V -> (none); footprint LED_SMD:LED_Cree-XHP50_6V -> (none)
- D40, D52: value Gnd -> (none); footprint Flat_Wires_Pads:Wire_Hole_1mm -> (none)
- D41: value Gnd -> (none); footprint libraries:WireHole_1p2 -> (none)
- D42: value In -> (none); footprint libraries:WireHole_1p2 -> (none)
- D50: value Flash LED + -> (none); footprint libraries:WireHole_1p2 -> (none)
- D51: value Out -> (none); footprint Flat_Wires_Pads:Wire_Hole_1mm -> (none)
- D58: value Flash LED - -> (none); footprint libraries:WireHole_1p2 -> (none)
- IC1: value TPS40211QDGQRQ1 -> (none); footprint libraries:SOP50P490X110-11N -> (none)
- IC2: value LM5164QDDATQ1 -> (none); footprint libraries:SOIC127P600X170-9N -> (none)
- IC3: value LM3481MM_NOPB -> (none); footprint libraries:SOP50P490X110-10N -> (none)
- IC4: value LM3488MM -> (none); footprint libraries:SOP65P490X110-8N -> (none)
- IC5: value LM3478MMX_NOPB -> (none); footprint libraries:SOP65P490X110-8N -> (none)
- L1, L5, L7: value TFM201610ALC-R47MTAA -> (none); footprint libraries:INDC2016X80N -> (none)
- L10, L3, L8, L9: value SRP4020TA-100M -> (none); footprint libraries:INDPM4441X200N -> (none)
- L2: value SRP7050AA-220M -> (none); footprint libraries:INDPM5752X300N -> (none)
- L4: value TFM201610ALC-R47MTAA -> (none); footprint libraries:WPN252010UR47MT -> (none)
- L6: value TFM201610ALC-R47MTAA -> (none); footprint libraries:INDPM5752X300N -> (none)
- Q1, Q2, Q3, Q4, Q5: value AON7407 -> (none); footprint libraries:DFN_3X3_EP -> (none)
- R1, R10, R11, R12, R13, R14, R15, R16, R17, R18, R19, R2, R20, R21, R22, R23, R24, R25, R26, R27, R28, R29, R3, R30, R4, R5, R6, R7, R8, R9: value R -> (none); footprint Resistor_SMD:R_0805_2012Metric_Pad1.20x1.40mm_HandSolder -> (none)
- U1, U6, U7, U8: value INA138 -> (none); footprint Package_TO_SOT_SMD:SOT-23-5 -> (none)
- U2, U3, U4, U5: value Mounting_Hole_M2 -> (none); footprint mount_holes:Hole_screw_M1p2 -> (none)
- Z1, Z2: value BZT52-C5V1J -> (none); footprint Diode_SMD:D_SOD-323F -> (none)
Connections:
- net GND: now also C17.2, C18.2, C19.2, C20.2, C21.2, C23.1, C25.2, C26.2, C27.2, C28.2, C29.2, C30.2, C31.2, C34.2, C35.2, C36.2, C37.2, C38.2, C39.2, C40.2, C41.2, C42.2, C43.2, C44.2, C45.2, D19.1 (Conn), D20.1 (GND), D37.1 (Conn), D40.1 (Conn), D41.1 (Conn), D44.1 (Conn), D52.1 (Conn), D54.1 (Conn), IC3.5 (AGND), IC3.7 (PGND), IC4.4 (AGND), IC4.5 (PGND), IC5.4 (AGND), IC5.5 (PGND), R11.2, R13.2, R14.1, R15.1, R17.2, R18.2, R20.1, R21.2, R22.2, R23.2, R24.2, R25.2, R26.2, R28.1, R30.1, U6.2 (GND), U7.2 (GND), U8.2 (GND)
Other:
- moved on the sheet: C14, C15, C16, C20, C22, C23, C24, C25, C26, C27, C28, C29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
