File: Main_PCB_003/_autosave-Main_PCB_001.kicad_sch (KiCad schematic)
At the start: 163 parts, among them IC1 TPS40211QDGQRQ1, IC2 LM5164QDDATQ1, IC3 LM3481MM_NOPB, IC4 LM3488MM, IC5 LM3478MMX_NOPB, Q1 AON7407, Q2 AON7407, Q3 AON7407, Q4 AON7407, Q5 AON7407, U1 INA138, U2 Mounting_Hole_M2, U3 Mounting_Hole_M2, U4 Mounting_Hole_M2, U5 Mounting_Hole_M2, U6 INA138, U7 INA138, U8 INA138

Commit message: Prototyping 6 001
Parts:
- removed C25, C32, C37, C39, C43: C, Capacitor_SMD:C_0805_2012Metric_Pad1.18x1.45mm_HandSolder, symbol Device:C
- removed C35, C41: C, Capacitor_SMD:C_1206_3216Metric_Pad1.33x1.80mm_HandSolder, symbol Device:C
- removed C45: C, Capacitor_SMD:C_0402_1005Metric_Pad0.74x0.62mm_HandSolder, symbol Device:C
- removed D37, D43, D44, D50, D55, D56, D57, D58: WireHole_1p5, libraries:WireHole_1p2, symbol Connectors_for_Wire:WireHole_1p5
- removed D46: SS36, libraries:SODFL4626X120N, symbol SS36:SS36
- removed D47, D48, D49: LED_Cree_XHP50_6V, LED_SMD:LED_Cree-XHP50_6V, symbol LED:LED_Cree_XHP50_6V
- removed D53, D54: Wire_Pad_01, Flat_Wires_Pads:Wire_Hole_1mm, symbol Connectors_for_Wire:Wire_Pad_01
- removed IC4: LM3488MM, libraries:SOP65P490X110-8N, symbol LM3488MM:LM3488MM
- removed L10: SRP4020TA-100M, libraries:INDPM4441X200N, symbol SRP4020TA-100M:SRP4020TA-100M
- removed Q5: AON7407, libraries:DFN_3X3_EP, symbol AON7407:AON7407
- removed R17, R21, R24, R26, R29, R30: R, Resistor_SMD:R_0805_2012Metric_Pad1.20x1.40mm_HandSolder, symbol Device:R
- removed U8: INA138, Package_TO_SOT_SMD:SOT-23-5, symbol Amplifier_Current:INA138
- C?: renamed from C29; footprint Capacitor_SMD:C_1206_3216Metric_Pad1.33x1.80mm_HandSolder -> Capacitor_SMD:C_0805_2012Metric_Pad1.18x1.45mm_HandSolder
- C?: renamed from C40; footprint Capacitor_SMD:C_1206_3216Metric_Pad1.33x1.80mm_HandSolder -> Capacitor_SMD:C_0805_2012Metric_Pad1.18x1.45mm_HandSolder
- C?: renamed from C26; footprint Capacitor_SMD:C_1206_3216Metric_Pad1.33x1.80mm_HandSolder -> Capacitor_SMD:C_0805_2012Metric_Pad1.18x1.45mm_HandSolder
- C?: renamed from C34; footprint Capacitor_SMD:C_1206_3216Metric_Pad1.33x1.80mm_HandSolder -> Capacitor_SMD:C_0805_2012Metric_Pad1.18x1.45mm_HandSolder
- IC?: renamed from IC3; value LM3481MM_NOPB -> (none); footprint libraries:SOP50P490X110-10N -> (none)
- IC?: renamed from IC5; value LM3478MMX_NOPB -> (none); footprint libraries:SOP65P490X110-8N -> (none)
- renumbered C23 to C?, C28 to C?, C44 to C?, C42 to C?, C27 to C?, C33 to C?, C24 to C?, C31 to C?, C38 to C?, C30 to C?, C36 to C?, D52 to D?, D39 to D?, D51 to D?, D38 to D?, D42 to D?, D45 to D?, D40 to D?, D36 to D?, D41 to D?, L9 to L?, L8 to L?, Q4 to Q?, Q3 to Q?, R20 to R?, R22 to R?, R19 to R?, R27 to R?, R15 to R?, R23 to R?, R18 to R?, R16 to R?, R28 to R?, R14 to R?, R25 to R?, U6 to U?, U7 to U?
Connections:
- net GND: no longer C?.1, IC?.5 (AGND), IC?.7 (PGND), R?.1, R?.1
- net at D22.1 (Conn), R12.2, R13.1: now also D35.1 (K)
- net at C?.1, Q?.1 (S_1), Q?.2 (S_2)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: no longer IC?.1 (ISEN)
- net at D23.1 (Conn), L7.2: now also D24.2 (A)
- net at R?.2, U?.1: no longer IC?.4 (FB)
- net at R?.1, R?.2: no longer IC?.2 (UVLO)
- new net: C?.1, R?.1
Other:
- moved on the sheet: C1, C10, C11, C12, C13, C14, C15, C16, C17, C18, C19, C2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
