File: Main_PCB_004/Main_PCB_002.kicad_sch (KiCad schematic)
At the start: 163 parts, among them IC1 TPS40211QDGQRQ1, IC2 LM5164QDDATQ1, IC3 LM3481MM_NOPB, IC4 LM3488MM, IC5 LM3478MMX_NOPB, Q1 AON7407, Q2 AON7407, Q3 AON7407, Q4 AON7407, Q5 AON7407, U1 INA138, U2 Mounting_Hole_M2, U3 Mounting_Hole_M2, U4 Mounting_Hole_M2, U5 Mounting_Hole_M2, U6 INA138, U7 INA138, U8 INA138

Commit message: Prototyping 6 001
Parts:
- added C46, C47, C48, C49, C50, C51, C52, C53, C54, C55, C56, C57, C58, C59, C60: C, Capacitor_SMD:C_0805_2012Metric_Pad1.18x1.45mm_HandSolder, symbol Device:C
- added D59, D60, D61, D62, D63, D64, D65, D66, D67, D68, D69, D74, D75, D76, D77, D80, D81, D82, D83, D84, D85, D86, D87, D92, D93, D94, D95, D96, D97: (no value), libraries:WireHole_1p2, symbol Connectors_for_Wire:WireHole_1p5
- added D70, D71, D72, D73, D78, D79, D88, D89, D90, D91: (no value), Flat_Wires_Pads:Wire_Hole_1mm, symbol Connectors_for_Wire:Wire_Pad_01
- added R31, R32, R33, R34, R35, R36, R37, R38: R, Resistor_SMD:R_0805_2012Metric_Pad1.20x1.40mm_HandSolder, symbol Device:R
- added U10, U11, U12, U13, U15, U16, U17, U18, U19, U20, U22, U23: MCP9700AT-ETT, Package_TO_SOT_SMD:SOT-23, symbol Sensor_Temperature:MCP9700AT-ETT
- added U14, U21: INA138, Package_TO_SOT_SMD:SOT-23-5, symbol Amplifier_Current:INA138
- added U9: (no value), symbol Sensor_Temperature:MCP9700AT-ETT
- D27: value LED_Cree_XHP50_6V -> (none)
- D40, D51, D52: value Wire_Pad_01 -> (none)
- D41, D42, D50, D58: value WireHole_1p5 -> (none)
Connections:
- net at C10.2, C11.2, C12.2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: now also C49.2, C50.2, D69.1 (Conn), U12.3 (GND), U13.3 (GND)
- net at C17.2, C18.2, C19.2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: now also C52.2, C53.2, D77.1 (Conn), U15.3 (GND), U16.3 (GND)
- net at C34.2, C36.2, C38.2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: now also C54.2, C56.2, D83.1 (Conn), U17.3 (GND), U19.3 (GND)
- net at C23.1, C25.2, C26.2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: now also C47.2, C48.2, D65.1 (Conn), U10.3 (GND), U11.3 (GND)
- net at C15.2, C16.2, C22.2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: now also C46.2, D61.1 (Conn), U9.3 (GND)
- net at C35.2, C37.2, C39.2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: now also C55.2, C57.2, D87.1 (Conn), U18.3 (GND), U20.3 (GND)
- new net: D93.1 (Conn), U22.2 (Vout)
- new net: C54.1, C56.1, D80.1 (Conn), U17.1 (Vdd), U19.1 (Vdd)
- new net: D64.1 (Conn), U10.2 (Vout)
- new net: C49.1, C50.1, D66.1 (Conn), U12.1 (Vdd), U13.1 (Vdd)
- new net: D75.1 (Conn), U16.2 (Vout)
- new net: C60.1, D95.1 (Conn), U23.1 (Vdd)
- new net: C58.2, D89.1 (Conn), R36.1, R38.1, U21.2 (GND)
- new net: D91.1 (Conn), R36.2, U21.1
- new net: D68.1 (Conn), U12.2 (Vout)
- new net: C46.1, D59.1 (Conn), U9.1 (Vdd)
- new net: C52.1, C53.1, D74.1 (Conn), U15.1 (Vdd), U16.1 (Vdd)
- new net: D78.1 (Conn), R32.2, U14.1
- new net: C51.2, D72.1 (Conn), R32.1, R34.1, U14.2 (GND)
- new net: C51.1, D70.1 (Conn), R31.1, U14.3 (+), U14.5 (V+)
- new net: D71.1 (Conn), R31.2, R33.2, U14.4 (-)
- new net: D76.1 (Conn), U15.2 (Vout)
- new net: D60.1 (Conn), U9.2 (Vout)
- new net: C60.2, D97.1 (Conn), U23.3 (GND)
- new net: D73.1 (Conn), R33.1, R34.2
- new net: C58.1, D79.1 (Conn), R35.1, U21.3 (+), U21.5 (V+)
- new net: C55.1, C57.1, D84.1 (Conn), U18.1 (Vdd), U20.1 (Vdd)
- new net: D85.1 (Conn), U20.2 (Vout)
- new net: D82.1 (Conn), U17.2 (Vout)
- new net: C47.1, C48.1, D62.1 (Conn), U10.1 (Vdd), U11.1 (Vdd)
- new net: C59.1, D92.1 (Conn), U22.1 (Vdd)
- new net: D81.1 (Conn), U19.2 (Vout)
- new net: D96.1 (Conn), U23.2 (Vout)
- new net: D63.1 (Conn), U11.2 (Vout)
- new net: D86.1 (Conn), U18.2 (Vout)
- new net: C59.2, D94.1 (Conn), U22.3 (GND)
- new net: D90.1 (Conn), R37.1, R38.2
- new net: D67.1 (Conn), U13.2 (Vout)
- new net: D88.1 (Conn), R35.2, R37.2, U21.4 (-)
Other:
- moved on the sheet: C14, C15, C16, C22, C23, C24, C25, C26, C27, C28, C29, C30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
