File: Main_PCB_004/Main_PCB_002.kicad_pcb (KiCad board)
At the start: 4 copper layers, 163 parts, among them IC1 TPS40211QDGQRQ1, IC2 LM5164QDDATQ1, IC3 LM3481MM_NOPB, IC4 LM3488MM, IC5 LM3478MMX_NOPB, Q1 AON7407, Q2 AON7407, Q3 AON7407, Q4 AON7407, Q5 AON7407, U1 INA138, U2 Mounting_Hole_M2, U3 Mounting_Hole_M2, U4 Mounting_Hole_M2, U5 Mounting_Hole_M2, U6 INA138, U7 INA138, U8 INA138

Commit message: Prototyping 6 001
Parts:
- removed U3: Mounting_Hole_M2, mount_holes:Hole_screw_M1p2
- added C46: C, Capacitor_SMD:C_0805_2012Metric_Pad1.18x1.45mm_HandSolder, B.Cu at (132.7, 64.2)
- added C47: C, Capacitor_SMD:C_0805_2012Metric_Pad1.18x1.45mm_HandSolder, B.Cu at (84.2, 123.7)
- added C48: C, Capacitor_SMD:C_0805_2012Metric_Pad1.18x1.45mm_HandSolder, B.Cu at (82.5, 119.9)
- added C49: C, Capacitor_SMD:C_0805_2012Metric_Pad1.18x1.45mm_HandSolder, B.Cu at (93.2, 68.3)
- added C50: C, Capacitor_SMD:C_0805_2012Metric_Pad1.18x1.45mm_HandSolder, B.Cu at (94.4, 65.4)
- added C51: C, Capacitor_SMD:C_0805_2012Metric_Pad1.18x1.45mm_HandSolder, F.Cu at (176.5, 95.7)
- added C52: C, Capacitor_SMD:C_0805_2012Metric_Pad1.18x1.45mm_HandSolder, B.Cu at (138.9, 85.6)
- added C53: C, Capacitor_SMD:C_0805_2012Metric_Pad1.18x1.45mm_HandSolder, B.Cu at (138.0, 88.6)
- added C54: C, Capacitor_SMD:C_0805_2012Metric_Pad1.18x1.45mm_HandSolder, B.Cu at (128.8, 123.0)
- added C55: C, Capacitor_SMD:C_0805_2012Metric_Pad1.18x1.45mm_HandSolder, B.Cu at (100.1, 90.9)
- added C56: C, Capacitor_SMD:C_0805_2012Metric_Pad1.18x1.45mm_HandSolder, B.Cu at (126.5, 114.2)
- added C57: C, Capacitor_SMD:C_0805_2012Metric_Pad1.18x1.45mm_HandSolder, B.Cu at (95.1, 99.3)
- added C58: C, Capacitor_SMD:C_0805_2012Metric_Pad1.18x1.45mm_HandSolder, F.Cu at (72.8, 98.9)
- added C59: C, Capacitor_SMD:C_0805_2012Metric_Pad1.18x1.45mm_HandSolder, F.Cu at (173.7, 122.2)
- added C60: C, Capacitor_SMD:C_0805_2012Metric_Pad1.18x1.45mm_HandSolder, F.Cu at (168.1, 68.0)
- added D59: +5B, libraries:WireHole_1p2, F.Cu at (146.3, 66.6)
- added D60: t_IC, libraries:WireHole_1p2, F.Cu at (146.3, 68.9)
- added D61: Gnd, libraries:WireHole_1p2, F.Cu at (146.3, 71.3)
- added D62: +5B, libraries:WireHole_1p2, F.Cu at (100.4, 123.8)
- added D63: t_D, libraries:WireHole_1p2, F.Cu at (100.3, 126.2)
- added D64: t_Q, libraries:WireHole_1p2, F.Cu at (100.3, 128.5)
- added D65: Gnd, libraries:WireHole_1p2, F.Cu at (100.3, 131.0)
- added D66: +5B, libraries:WireHole_1p2, F.Cu at (101.7, 65.1)
- added D67: t_D, libraries:WireHole_1p2, F.Cu at (101.7, 67.5)
- added D68: t_Q, libraries:WireHole_1p2, F.Cu at (101.8, 69.9)
- added D69: Gnd, libraries:WireHole_1p2, F.Cu at (101.7, 72.4)
- added D70: CS_In, Flat_Wires_Pads:Wire_Hole_1mm, F.Cu at (176.6, 98.5)
- added D71: CS_Out, Flat_Wires_Pads:Wire_Hole_1mm, F.Cu at (183.0, 98.4)
- added D72: Gnd, Flat_Wires_Pads:Wire_Hole_1mm, F.Cu at (174.4, 94.6)
- added D73: U, Flat_Wires_Pads:Wire_Hole_1mm, F.Cu at (182.2, 90.2)
- added D74: +5B, libraries:WireHole_1p2, F.Cu at (144.8, 92.5)
- added D75: t_D, libraries:WireHole_1p2, F.Cu at (144.8, 94.9)
- added D76: t_Q, libraries:WireHole_1p2, F.Cu at (144.8, 97.3)
- added D77: Gnd, libraries:WireHole_1p2, F.Cu at (144.8, 99.7)
- added D78: I, Flat_Wires_Pads:Wire_Hole_1mm, F.Cu at (177.6, 90.2)
- added D79: CS_In, Flat_Wires_Pads:Wire_Hole_1mm, F.Cu at (73.0, 101.9)
- added D80: +5B, libraries:WireHole_1p2, F.Cu at (138.7, 120.2)
- added D81: t_D, libraries:WireHole_1p2, F.Cu at (138.7, 122.8)
- added D82: t_Q, libraries:WireHole_1p2, F.Cu at (138.7, 125.3)
- added D83: Gnd, libraries:WireHole_1p2, F.Cu at (138.6, 127.6)
- added D84: +5B, libraries:WireHole_1p2, F.Cu at (110.3, 96.8)
- added D85: t_D, libraries:WireHole_1p2, F.Cu at (110.3, 99.2)
- added D86: t_Q, libraries:WireHole_1p2, F.Cu at (110.3, 101.5)
- added D87: Gnd, libraries:WireHole_1p2, F.Cu at (110.3, 103.8)
- added D88: CS_Out, Flat_Wires_Pads:Wire_Hole_1mm, F.Cu at (79.4, 101.8)
- added D89: Gnd, Flat_Wires_Pads:Wire_Hole_1mm, F.Cu at (70.8, 97.7)
- added D90: U, Flat_Wires_Pads:Wire_Hole_1mm, F.Cu at (78.7, 93.4)
- added D91: I, Flat_Wires_Pads:Wire_Hole_1mm, F.Cu at (74.7, 93.4)
- added D92: +5V, libraries:WireHole_1p2, F.Cu at (186.1, 120.2)
- added D93: t LED, libraries:WireHole_1p2, F.Cu at (186.1, 122.5)
- added D94: GND, libraries:WireHole_1p2, F.Cu at (186.2, 124.8)
- added D95: +5B, libraries:WireHole_1p2, F.Cu at (174.3, 67.0)
- added D96: t_LED, libraries:WireHole_1p2, F.Cu at (174.3, 69.4)
- added D97: GND, libraries:WireHole_1p2, F.Cu at (174.3, 71.7)
- added R31: R, Resistor_SMD:R_0805_2012Metric_Pad1.20x1.40mm_HandSolder, F.Cu at (179.8, 98.2)
- added R32: R, Resistor_SMD:R_0805_2012Metric_Pad1.20x1.40mm_HandSolder, F.Cu at (177.4, 92.5)
- added R33: R, Resistor_SMD:R_0805_2012Metric_Pad1.20x1.40mm_HandSolder, F.Cu at (183.1, 95.5)
- added R34: R, Resistor_SMD:R_0805_2012Metric_Pad1.20x1.40mm_HandSolder, F.Cu at (181.4, 92.5)
- added R35: R, Resistor_SMD:R_0805_2012Metric_Pad1.20x1.40mm_HandSolder, F.Cu at (76.2, 101.6)
- added R36: R, Resistor_SMD:R_0805_2012Metric_Pad1.20x1.40mm_HandSolder, F.Cu at (73.7, 95.8)
- added R37: R, Resistor_SMD:R_0805_2012Metric_Pad1.20x1.40mm_HandSolder, F.Cu at (79.4, 98.9)
- added R38: R, Resistor_SMD:R_0805_2012Metric_Pad1.20x1.40mm_HandSolder, F.Cu at (77.7, 95.8)
- added U10: MCP9700AT-ETT, Package_TO_SOT_SMD:SOT-23, B.Cu at (87.2, 123.3)
- added U11: MCP9700AT-ETT, Package_TO_SOT_SMD:SOT-23, B.Cu at (85.5, 119.7)
- added U12: MCP9700AT-ETT, Package_TO_SOT_SMD:SOT-23, B.Cu at (93.3, 71.2)
- added U13: MCP9700AT-ETT, Package_TO_SOT_SMD:SOT-23, B.Cu at (97.2, 66.0)
- added U14: INA138, Package_TO_SOT_SMD:SOT-23-5, F.Cu at (179.9, 95.4)
- added U15: MCP9700AT-ETT, Package_TO_SOT_SMD:SOT-23, B.Cu at (138.9, 91.3)
- added U16: MCP9700AT-ETT, Package_TO_SOT_SMD:SOT-23, B.Cu at (141.9, 86.6)
- added U17: MCP9700AT-ETT, Package_TO_SOT_SMD:SOT-23, B.Cu at (129.0, 120.4)
- added U18: MCP9700AT-ETT, Package_TO_SOT_SMD:SOT-23, B.Cu at (97.9, 99.2)
- added U19: MCP9700AT-ETT, Package_TO_SOT_SMD:SOT-23, B.Cu at (126.6, 117.0)
- added U20: MCP9700AT-ETT, Package_TO_SOT_SMD:SOT-23, B.Cu at (100.1, 93.8)
- added U21: INA138, Package_TO_SOT_SMD:SOT-23-5, F.Cu at (76.0, 98.6)
- added U22: MCP9700AT-ETT, Package_TO_SOT_SMD:SOT-23, F.Cu at (170.3, 122.4)
- added U23: MCP9700AT-ETT, Package_TO_SOT_SMD:SOT-23, F.Cu at (168.0, 70.8)
- added U9: MCP9700AT-ETT, Package_TO_SOT_SMD:SOT-23, B.Cu at (132.6, 67.2)
- D24, D25, D26, D27, D28, D29, D30, D31, D32, D33, D34, D35, D47, D48, D49: moved to B.Cu
- D40, D52: value Wire_Pad_01 -> Gnd
- D41: value WireHole_1p5 -> Gnd
- D42: value WireHole_1p5 -> In
- D50: value WireHole_1p5 -> Flash LED +
- D51: value Wire_Pad_01 -> Out
- D58: value WireHole_1p5 -> Flash LED -
- moved U4 207.3 mm to (66.9, 138.3)
- moved U5 175.8 mm to (66.8, 57.3)
- moved D10 135.5 mm to (145.8, 136.9)
- moved D14 132.2 mm to (149.4, 136.8)
- moved D9 125.6 mm to (142.1, 136.9)
- moved U2 123.4 mm to (192.2, 138.2)
- moved D15 112.8 mm to (150.2, 114.1)
- moved R11 103.0 mm to (136.9, 94.7)
- moved C17 102.9 mm to (128.8, 90.9)
- moved C20 102.9 mm to (132.8, 90.8)
- moved D20 102.9 mm to (130.7, 91.2)
- moved D22 102.9 mm to (131.8, 98.9)
- moved D23 102.9 mm to (145.2, 88.4)
- moved L5 102.9 mm to (128.4, 85.4)
- moved L6 102.9 mm to (136.2, 86.6)
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Connections:
- Q1 pad 10: (no net) -> Net-(D12-Pad2)
- Q1 pad 11: (no net) -> Net-(D12-Pad2)
- Q1 pad 9: (no net) -> Net-(D12-Pad2)
- Q3 pad 10: (no net) -> Net-(D38-Pad2)
- Q3 pad 11: (no net) -> Net-(D38-Pad2)
- Q3 pad 9: (no net) -> Net-(D38-Pad2)
- Q4 pad 10: (no net) -> Net-(D45-Pad2)
- Q4 pad 11: (no net) -> Net-(D45-Pad2)
- Q4 pad 9: (no net) -> Net-(D45-Pad2)
Routing:
- net Net-(D10-Pad1): track 0.00 -> 402.4 mm
- net GND: track 0.00 -> 289.2 mm
- net Net-(D14-Pad1): track 0.00 -> 222.8 mm, vias 0 -> 2
- net Net-(D31-Pad1): track 0.00 -> 46.5 mm
- net Net-(D27-Pad1): track 0.00 -> 45.4 mm
- net Net-(C34-Pad1): track 0.00 -> 43.7 mm
- net Net-(D24-Pad2): track 0.00 -> 40.6 mm
- net Net-(C47-Pad1): track 0.00 -> 29.2 mm
- net Net-(C59-Pad2): track 0.00 -> 28.1 mm
- net Net-(D7-Pad1): track 0.00 -> 28.0 mm
- net Net-(C54-Pad1): track 0.00 -> 23.7 mm
- net Net-(C55-Pad1): track 0.00 -> 21.6 mm
- net Net-(C26-Pad1): track 0.00 -> 21.3 mm
- net Net-(C59-Pad1): track 0.00 -> 19.5 mm
- net Net-(C52-Pad1): track 0.00 -> 19.4 mm
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- added copper zone on B.Cu, net Net-(C10-Pad2)
- added copper zone on F.Cu, net Net-(C10-Pad2)
- added copper zone on B.Cu, net Net-(C15-Pad2)
- added copper zone on F.Cu, net Net-(C15-Pad2)
- added copper zone on B.Cu, net Net-(C23-Pad1)
- added copper zone on F.Cu, net Net-(C23-Pad1)
- added copper zone on B.Cu, net Net-(C34-Pad2)
- added copper zone on F.Cu, net Net-(C34-Pad2)
- added copper zone on B.Cu, net Net-(C35-Pad2)
- added copper zone on F.Cu, net Net-(C35-Pad2)
- added copper zone on B.Cu, net Net-(C52-Pad2)
- added copper zone on F.Cu, net Net-(C52-Pad2)
Other:
- board outline added: 133.3 x 88.9 mm
- copper layers 4 -> 2
- board text added: "En"
- board text added: "Gnd"
- board text added: "In"
- board text added: "LED+"
- board text added: "LED-"
- board text added: "LM3478"
- board text added: "LM3481"
- board text added: "LM3488"
- board text added: "LM5164"
- board text added: "Out"
- board text added: "TPS40211"
- board text added: "XDS TD6211"

Commit message: Prototyping 6 001
Parts:
- added ?: , , F.Cu at (137.2, 113.0)
- added ?: , , F.Cu at (151.1, 82.5)
- added ?: , , F.Cu at (87.6, 82.5)
- added ?: , , F.Cu at (105.4, 85.1)
- added ?: , , F.Cu at (105.4, 82.5)
- added ?: , , F.Cu at (148.6, 82.5)
- added ?: , , F.Cu at (109.2, 62.2)
- added ?: , , F.Cu at (71.1, 81.3)
- added ?: , , F.Cu at (121.9, 110.5)
- added ?: , , F.Cu at (171.4, 135.9)
- added ?: , , F.Cu at (76.2, 83.8)
- added ?: , , F.Cu at (123.2, 81.3)
- added ?: , , F.Cu at (106.7, 74.9)
- added ?: , , F.Cu at (174.0, 135.9)
- added ?: , , F.Cu at (148.6, 77.5)
- added ?: , , F.Cu at (148.6, 85.1)
- added ?: , , F.Cu at (156.2, 71.1)
- added ?: , , F.Cu at (148.6, 71.1)
- added ?: , , F.Cu at (102.9, 82.5)
- added ?: , , F.Cu at (102.9, 85.1)
- added ?: , , F.Cu at (166.4, 133.3)
- added ?: , , F.Cu at (181.6, 130.8)
- added ?: , , F.Cu at (128.3, 81.3)
- added ?: , , F.Cu at (166.4, 130.8)
- added ?: , , F.Cu at (133.3, 78.7)
- added ?: , , F.Cu at (158.8, 133.3)
- added ?: , , F.Cu at (73.7, 91.4)
- added ?: , , F.Cu at (120.7, 78.7)
- added ?: , , F.Cu at (130.8, 78.7)
- added ?: , , F.Cu at (153.7, 80.0)
- added ?: , , F.Cu at (186.9, 95.2)
- added ?: , , F.Cu at (73.7, 81.3)
- added ?: , , F.Cu at (148.6, 74.9)
- added ?: , , F.Cu at (148.6, 61.0)
- added ?: , , F.Cu at (85.1, 115.6)
- added ?: , , F.Cu at (119.4, 113.0)
- added ?: , , F.Cu at (74.9, 113.0)
- added ?: , , F.Cu at (153.7, 82.5)
- added ?: , , F.Cu at (109.2, 72.4)
- added ?: , , F.Cu at (90.2, 82.5)
- added ?: , , F.Cu at (78.7, 81.3)
- added ?: , , F.Cu at (127.0, 113.0)
- added ?: , , F.Cu at (87.6, 113.0)
- added ?: , , F.Cu at (132.1, 113.0)
- added ?: , , F.Cu at (176.5, 135.9)
- added ?: , , F.Cu at (156.2, 68.6)
- added ?: , , F.Cu at (127.0, 110.5)
- added ?: , , F.Cu at (184.2, 135.9)
- added ?: , , F.Cu at (163.8, 130.8)
- added ?: , , F.Cu at (76.2, 91.4)
- added ?: , , F.Cu at (171.4, 133.3)
- added ?: , , F.Cu at (82.5, 115.6)
- added ?: , , F.Cu at (179.1, 133.3)
- added ?: , , F.Cu at (90.2, 113.0)
- added ?: , , F.Cu at (156.2, 63.5)
- added ?: , , F.Cu at (156.2, 74.9)
- added ?: , , F.Cu at (95.2, 85.1)
- added ?: , , F.Cu at (156.0, 95.2)
- added ?: , , F.Cu at (90.2, 115.6)
- added ?: , , F.Cu at (72.4, 113.0)
- added ?: , , F.Cu at (124.5, 110.5)
- added ?: , , F.Cu at (71.1, 83.8)
- added ?: , , F.Cu at (92.7, 115.6)
- added ?: , , F.Cu at (80.0, 115.6)
- added ?: , , F.Cu at (109.2, 67.3)
- added ?: , , F.Cu at (153.7, 68.6)
- added ?: , , F.Cu at (87.6, 115.6)
- added ?: , , F.Cu at (109.2, 74.9)
- added ?: , , F.Cu at (153.7, 77.5)
- added ?: , , F.Cu at (153.7, 133.3)
- added ?: , , F.Cu at (181.6, 133.3)
- added ?: , , F.Cu at (106.7, 69.8)
- added ?: , , F.Cu at (78.7, 88.9)
- added ?: , , F.Cu at (151.1, 74.9)
- added ?: , , F.Cu at (76.2, 86.4)
- added ?: , , F.Cu at (151.1, 71.1)
- added ?: , , F.Cu at (118.1, 78.7)
- added ?: , , F.Cu at (108.0, 85.1)
- added ?: , , F.Cu at (174.0, 133.3)
- added ?: , , F.Cu at (125.7, 78.7)
- added ?: , , F.Cu at (106.7, 62.2)
- added ?: , , F.Cu at (156.2, 135.9)
- added ?: , , F.Cu at (171.7, 95.1)
- added ?: , , F.Cu at (151.1, 63.5)
- added ?: , , F.Cu at (77.5, 115.6)
- added ?: , , F.Cu at (153.7, 61.0)
- added ?: , , F.Cu at (151.1, 68.6)
- added ?: , , F.Cu at (111.8, 62.2)
- added ?: , , F.Cu at (116.8, 110.5)
- added ?: , , F.Cu at (153.7, 71.1)
- added ?: , , F.Cu at (120.7, 81.3)
- added ?: , , F.Cu at (153.7, 63.5)
- added ?: , , F.Cu at (168.9, 135.9)
- added ?: , , F.Cu at (161.3, 135.9)
- added ?: , , F.Cu at (151.1, 85.1)
- added ?: , , F.Cu at (73.7, 88.9)
- added ?: , , F.Cu at (78.7, 91.4)
- added ?: , , F.Cu at (161.3, 130.8)
- added ?: , , F.Cu at (78.7, 83.8)
- added ?: , , F.Cu at (118.1, 81.3)
- added ?: , , F.Cu at (132.1, 110.5)
- added ?: , , F.Cu at (78.7, 86.4)
- added ?: , , F.Cu at (151.1, 61.0)
- added ?: , , F.Cu at (76.2, 88.9)
- added ?: , , F.Cu at (158.8, 130.8)
- added ?: , , F.Cu at (119.4, 110.5)
- added ?: , , F.Cu at (134.6, 110.5)
- added ?: , , F.Cu at (80.0, 113.0)
- added ?: , , F.Cu at (153.7, 130.8)
- added ?: , , F.Cu at (156.2, 130.8)
- added ?: , , F.Cu at (95.2, 82.5)
- added ?: , , F.Cu at (111.8, 64.8)
- added ?: , , F.Cu at (164.1, 95.1)
- added ?: , , F.Cu at (171.4, 130.8)
- added ?: , , F.Cu at (97.8, 85.1)
- added ?: , , F.Cu at (138.4, 81.3)
- added ?: , , F.Cu at (135.9, 78.7)
- added ?: , , F.Cu at (184.2, 133.3)
- added ?: , , F.Cu at (71.1, 91.4)
- added ?: , , F.Cu at (87.6, 85.1)
- added ?: , , F.Cu at (151.1, 80.0)
- added ?: , , F.Cu at (106.7, 72.4)
- added ?: , , F.Cu at (156.2, 77.5)
- added ?: , , F.Cu at (174.0, 130.8)
- added ?: , , F.Cu at (85.1, 113.0)
- added ?: , , F.Cu at (153.7, 66.0)
- added ?: , , F.Cu at (163.8, 135.9)
- added ?: , , F.Cu at (71.1, 86.4)
- added ?: , , F.Cu at (179.3, 95.2)
- added ?: , , F.Cu at (158.8, 135.9)
- added ?: , , F.Cu at (111.8, 72.4)
- added ?: , , F.Cu at (92.7, 113.0)
- added ?: , , F.Cu at (137.2, 110.5)
- added ?: , , F.Cu at (153.7, 85.1)
- added ?: , , F.Cu at (125.7, 81.3)
- added ?: , , F.Cu at (73.7, 86.4)
- added ?: , , F.Cu at (123.2, 78.7)
- added ?: , , F.Cu at (128.3, 78.7)
- added ?: , , F.Cu at (100.3, 82.5)
- added ?: , , F.Cu at (181.6, 135.9)
- added ?: , , F.Cu at (129.5, 110.5)
- added ?: , , F.Cu at (148.6, 80.0)
- added ?: , , F.Cu at (156.2, 133.3)
- added ?: , , F.Cu at (111.8, 74.9)
- added ?: , , F.Cu at (106.7, 64.8)
- added ?: , , F.Cu at (109.2, 69.8)
- added ?: , , F.Cu at (156.2, 66.0)
- added ?: , , F.Cu at (156.2, 85.1)
- added ?: , , F.Cu at (179.1, 130.8)
- added ?: , , F.Cu at (90.2, 85.1)
- added ?: , , F.Cu at (73.7, 83.8)
- added ?: , , F.Cu at (176.5, 130.8)
- added ?: , , F.Cu at (148.6, 63.5)
- added ?: , , F.Cu at (148.6, 68.6)
- added ?: , , F.Cu at (138.4, 78.7)
- added ?: , , F.Cu at (121.9, 113.0)
- added ?: , , F.Cu at (109.2, 64.8)
- added ?: , , F.Cu at (176.5, 133.3)
- added ?: , , F.Cu at (124.5, 113.0)
- added ?: , , F.Cu at (92.7, 85.1)
- added ?: , , F.Cu at (161.3, 133.3)
- added ?: , , F.Cu at (82.5, 113.0)
- added ?: , , F.Cu at (168.9, 133.3)
- added ?: , , F.Cu at (100.3, 85.1)
- added ?: , , F.Cu at (151.1, 77.5)
- added ?: , , F.Cu at (153.7, 135.9)
- added ?: , , F.Cu at (72.4, 115.6)
- added ?: , , F.Cu at (135.9, 81.3)
- added ?: , , F.Cu at (106.7, 67.3)
- added ?: , , F.Cu at (168.9, 130.8)
- added ?: , , F.Cu at (92.7, 82.5)
- added ?: , , F.Cu at (129.5, 113.0)
- added ?: , , F.Cu at (111.8, 69.8)
- added ?: , , F.Cu at (111.8, 67.3)
- added ?: , , F.Cu at (156.2, 82.5)
- added ?: , , F.Cu at (71.1, 88.9)
- added ?: , , F.Cu at (166.4, 135.9)
- added ?: , , F.Cu at (179.1, 135.9)
- added ?: , , F.Cu at (116.8, 113.0)
- added ?: , , F.Cu at (134.6, 113.0)
- added ?: , , F.Cu at (156.2, 80.0)
- added ?: , , F.Cu at (153.7, 74.9)
- added ?: , , F.Cu at (151.1, 66.0)
- added ?: , , F.Cu at (130.8, 81.3)
- added ?: , , F.Cu at (163.8, 133.3)
- added ?: , , F.Cu at (156.2, 61.0)
- added ?: , , F.Cu at (148.6, 66.0)
- added ?: , , F.Cu at (74.9, 115.6)
- added ?: , , F.Cu at (76.2, 81.3)
- added ?: , , F.Cu at (77.5, 113.0)
- added ?: , , F.Cu at (108.0, 82.5)
- added ?: , , F.Cu at (184.2, 130.8)
- added ?: , , F.Cu at (97.8, 82.5)
- added ?: , , F.Cu at (133.3, 81.3)
- added D33: LED_Cree_XHP50_6V, LED_SMD:LED_Cree-XHP50_6V, B.Cu at (175.5, 95.2)
- added D33: LED_Cree_XHP50_6V, LED_SMD:LED_Cree-XHP50_6V, B.Cu at (183.1, 95.2)
- added D33: LED_Cree_XHP50_6V, LED_SMD:LED_Cree-XHP50_6V, B.Cu at (167.9, 95.2)
- added D33: LED_Cree_XHP50_6V, LED_SMD:LED_Cree-XHP50_6V, B.Cu at (160.3, 95.2)
- moved C51 21.8 mm to (181.8, 74.5)
- moved D72 21.8 mm to (179.7, 73.5)
- moved D70 21.8 mm to (181.9, 77.3)
- moved D71 21.8 mm to (188.3, 77.2)
- moved D73 21.8 mm to (187.6, 69.1)
- moved D78 21.8 mm to (183.0, 69.1)
- moved R31 21.8 mm to (185.2, 77.1)
- moved R32 21.8 mm to (182.7, 71.3)
- moved R33 21.8 mm to (188.4, 74.4)
- moved R34 21.8 mm to (186.7, 71.3)
- moved U14 21.8 mm to (185.2, 74.2)
- moved D24 8.62 mm to (179.3, 122.7)
- moved D26 8.62 mm to (164.0, 122.7)
- moved D28 8.62 mm to (179.3, 113.9)
- moved D31 8.62 mm to (156.4, 113.9)
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Other:
- board text added: "+"
- board text added: "-"
