File: Main_PCB_005/Main_PCB_002.kicad_pcb (KiCad board)
At the start: 2 copper layers, 133.3 x 88.9 mm, 440 parts, among them IC1 TPS40211QDGQRQ1, IC2 LM5164QDDATQ1, IC3 LM3481MM_NOPB, IC4 LM3488MM, IC5 LM3478MMX_NOPB, IC6 MAX998EUT+T, Q1 AON7407, Q2 AON7407, Q3 AON7407, Q4 AON7407, Q5 AON7407, U1 INA138, U10 MCP9700AT-ETT, U11 MCP9700AT-ETT, U12 MCP9700AT-ETT, U13 MCP9700AT-ETT, U14 INA138, U15 MCP9700AT-ETT, U16 MCP9700AT-ETT, U17 MCP9700AT-ETT, U18 MCP9700AT-ETT, U19 MCP9700AT-ETT, U2 Mounting_Hole_M2, U20 MCP9700AT-ETT, U21 INA138, U22 MCP9700AT-ETT, U23 MCP9700AT-ETT, U24 Mounting_Hole_M2, U25 Mounting_Hole_M2, U26 Mounting_Hole_M2, U27 Mounting_Hole_M2, U28 Mounting_Hole_M2, U3 Mounting_Hole_M2, U4 Mounting_Hole_M2, U5 Mounting_Hole_M2, U6 INA138, U7 INA138, U8 INA138, U9 MCP9700AT-ETT

Commit message: Prototyping 06
Parts:
- added ?: , , F.Cu at (89.6, 140.4)
- added ?: , , F.Cu at (121.5, 140.2)
- added ?: , , F.Cu at (111.4, 142.7)
- added ?: , , F.Cu at (104.9, 140.3)
- added ?: , , F.Cu at (76.9, 140.4)
- added ?: , , F.Cu at (113.9, 140.2)
- added ?: , , F.Cu at (116.4, 140.2)
- added ?: , , F.Cu at (82.0, 142.9)
- added ?: , , F.Cu at (121.5, 142.7)
- added ?: , , F.Cu at (84.5, 142.9)
- added ?: , , F.Cu at (124.1, 140.2)
- added ?: , , F.Cu at (87.1, 140.4)
- added ?: , , F.Cu at (97.3, 140.3)
- added ?: , , F.Cu at (111.4, 140.2)
- added ?: , , F.Cu at (94.7, 142.9)
- added ?: , , F.Cu at (116.4, 142.7)
- added ?: , , F.Cu at (92.2, 140.4)
- added ?: , , F.Cu at (79.5, 140.4)
- added ?: , , F.Cu at (74.4, 140.4)
- added ?: , , F.Cu at (129.1, 142.7)
- added ?: , , F.Cu at (76.9, 142.9)
- added ?: , , F.Cu at (119.0, 140.2)
- added ?: , , F.Cu at (124.1, 142.7)
- added ?: , , F.Cu at (131.7, 142.7)
- added ?: , , F.Cu at (126.6, 142.7)
- added ?: , , F.Cu at (131.7, 140.2)
- added ?: , , F.Cu at (126.6, 140.2)
- added ?: , , F.Cu at (129.1, 140.2)
- added ?: , , F.Cu at (119.0, 142.7)
- added ?: , , F.Cu at (99.8, 140.3)
- added ?: , , F.Cu at (79.5, 142.9)
- added ?: , , F.Cu at (82.0, 140.4)
- added ?: , , F.Cu at (99.8, 142.8)
- added ?: , , F.Cu at (74.4, 142.9)
- added ?: , , F.Cu at (102.3, 140.3)
- added ?: , , F.Cu at (102.3, 142.8)
- added ?: , , F.Cu at (97.3, 142.8)
- added ?: , , F.Cu at (87.1, 142.9)
- added ?: , , F.Cu at (113.9, 142.7)
- added ?: , , F.Cu at (89.6, 142.9)
- added ?: , , F.Cu at (84.5, 140.4)
- added ?: , , F.Cu at (94.7, 140.4)
- added ?: , , F.Cu at (104.9, 142.8)
- added ?: , , F.Cu at (92.2, 142.9)
- moved ? 110.3 mm to (71.0, 79.9), turned to 90 degrees
- moved ? 109.3 mm to (73.6, 79.9), turned to 90 degrees
- moved ? 108.4 mm to (76.1, 79.9), turned to 90 degrees
- moved ? 106.9 mm to (71.0, 82.4), turned to 90 degrees
- moved ? 105.8 mm to (73.6, 82.4), turned to 90 degrees
- moved ? 104.9 mm to (76.1, 82.4), turned to 90 degrees
- moved ? 103.5 mm to (71.0, 85.0), turned to 90 degrees
- moved R41 102.6 mm to (158.8, 142.7), turned to 0 degrees
- moved ? 102.4 mm to (73.6, 85.0), turned to 90 degrees
- moved U26 101.7 mm to (155.9, 142.7), turned to 90 degrees
- moved R43 101.7 mm to (164.3, 140.6), turned to 90 degrees
- moved ? 101.4 mm to (76.1, 85.0), turned to 90 degrees
- moved ? 100.1 mm to (71.0, 87.5), turned to 90 degrees
- moved ? 99.0 mm to (73.6, 87.5), turned to 90 degrees
- moved R42 99.0 mm to (162.0, 139.2), turned to -90 degrees
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Routing:
- net GND: track 331.3 -> 346.6 mm
- net Net-(D10-Pad1): track 402.4 -> 417.0 mm
- net Net-(D23-Pad1): track 0.00 -> 3.48 mm
- net Net-(C52-Pad1): track 22.8 -> 20.8 mm
- net Net-(C55-Pad1): track 21.6 -> 23.5 mm
- net Net-(D75-Pad1): track 8.15 -> 9.62 mm
- net Net-(D76-Pad1): track 7.80 -> 9.27 mm
Other:
- board size 133.3 x 88.9 mm -> 133.3 x 96.5 mm
