File: PCB_Research_Noise/Main_PCB_002.kicad_sch (KiCad schematic)
At the start: 262 parts, among them IC1 TPS40211QDGQRQ1, IC2 LM5164QDDATQ1, IC3 LM3481MM_NOPB, IC4 LM3488MM, IC5 LM3478MMX_NOPB, Q1 AON7407, Q2 AON7407, Q3 AON7407, Q4 AON7407, Q5 AON7407, U1 INA138, U10 MCP9700AT-ETT, U11 MCP9700AT-ETT, U12 MCP9700AT-ETT, U13 MCP9700AT-ETT, U14 INA138, U15 MCP9700AT-ETT, U16 MCP9700AT-ETT, U17 MCP9700AT-ETT, U18 MCP9700AT-ETT, U19 MCP9700AT-ETT, U2 Mounting_Hole_M2, U20 MCP9700AT-ETT, U21 INA138, U22 MCP9700AT-ETT, U23 MCP9700AT-ETT, U24 Mounting_Hole_M2, U25 Mounting_Hole_M2, U26 Mounting_Hole_M2, U27 Mounting_Hole_M2, U28 Mounting_Hole_M2, U3 Mounting_Hole_M2, U4 Mounting_Hole_M2, U5 Mounting_Hole_M2, U6 INA138, U7 INA138, U8 INA138, U9 MCP9700AT-ETT

Commit message: PCB for radiated noise research 002
Parts:
- removed C14, C22, C31, C44, C45: C, Capacitor_SMD:C_0402_1005Metric_Pad0.74x0.62mm_HandSolder, symbol Device:C
- removed C15, C16, C18, C21, C26, C29, C34, C35, C40, C41, C7: C, Capacitor_SMD:C_1206_3216Metric_Pad1.33x1.80mm_HandSolder, symbol Device:C
- removed C17, C19, C20, C23, C24, C25, C27, C28, C30, C32, C33, C36, C37, C38, C39, C42, C43, C46, C47, C48, C52, C53, C54, C55, C56, C57, C59, C60: C, Capacitor_SMD:C_0805_2012Metric_Pad1.18x1.45mm_HandSolder, symbol Device:C
- removed C6: C, Capacitor_SMD:C_0603_1608Metric_Pad1.08x0.95mm_HandSolder, symbol Device:C
- removed C61: C, symbol Device:C
- removed D10, D100, D101, D102, D103, D104, D105, D106, D107, D13, D14, D15, D16, D39, D53, D54, D7, D8, D9: Wire_Pad_01, Flat_Wires_Pads:Wire_Hole_1mm, symbol Connectors_for_Wire:Wire_Pad_01
- removed D18, D19, D2, D22, D23, D3, D36, D37, D43, D44, D5, D55, D56, D57, D98, D99: WireHole_1p5, libraries:WireHole_1p2, symbol Connectors_for_Wire:WireHole_1p5
- removed D20: TX6211, XDS_Semi:TX6211, symbol XDS_Semi:TX6211
- removed D21, D38, D45, D46: SS36, libraries:SODFL4626X120N, symbol SS36:SS36
- removed D24, D25, D26, D27, D28, D29, D30, D31, D32, D33, D34, D35, D47, D48, D49: LED_Cree_XHP50_6V, LED_SMD:LED_Cree-XHP50_6V, symbol LED:LED_Cree_XHP50_6V
- removed D40, D52: Gnd, Flat_Wires_Pads:Wire_Hole_1mm, symbol Connectors_for_Wire:Wire_Pad_01
- removed D41, D61, D65, D77, D83, D87: Gnd, libraries:WireHole_1p2, symbol Connectors_for_Wire:WireHole_1p5
- removed D42: In, libraries:WireHole_1p2, symbol Connectors_for_Wire:WireHole_1p5
- removed D50: Flash LED +, libraries:WireHole_1p2, symbol Connectors_for_Wire:WireHole_1p5
- removed D51: Out, Flat_Wires_Pads:Wire_Hole_1mm, symbol Connectors_for_Wire:Wire_Pad_01
- removed D58: Flash LED -, libraries:WireHole_1p2, symbol Connectors_for_Wire:WireHole_1p5
- removed D59, D62, D74, D80, D84, D95: +5B, libraries:WireHole_1p2, symbol Connectors_for_Wire:WireHole_1p5
- removed D60: t_IC, libraries:WireHole_1p2, symbol Connectors_for_Wire:WireHole_1p5
- removed D63, D75, D81, D85: t_D, libraries:WireHole_1p2, symbol Connectors_for_Wire:WireHole_1p5
- removed D64, D76, D82, D86: t_Q, libraries:WireHole_1p2, symbol Connectors_for_Wire:WireHole_1p5
- removed D92: +5V, libraries:WireHole_1p2, symbol Connectors_for_Wire:WireHole_1p5
- removed D93: t LED, libraries:WireHole_1p2, symbol Connectors_for_Wire:WireHole_1p5
- removed D94, D97: GND, libraries:WireHole_1p2, symbol Connectors_for_Wire:WireHole_1p5
- removed D96: t_LED, libraries:WireHole_1p2, symbol Connectors_for_Wire:WireHole_1p5
- removed IC2: LM5164QDDATQ1, libraries:SOIC127P600X170-9N, symbol LM5164QDDATQ1:LM5164QDDATQ1
- removed IC3: LM3481MM_NOPB, libraries:SOP50P490X110-10N, symbol LM3481MM_NOPB:LM3481MM_NOPB
- removed IC4: LM3488MM, libraries:SOP65P490X110-8N, symbol LM3488MM:LM3488MM
- removed IC5: LM3478MMX_NOPB, libraries:SOP65P490X110-8N, symbol LM3478MMX_NOPB:LM3478MMX_NOPB
- removed IC6: (no value), symbol MAX998EUT+T:MAX998EUT+T
- removed L10, L3, L8, L9: SRP4020TA-100M, libraries:INDPM4441X200N, symbol SRP4020TA-100M:SRP4020TA-100M
- removed L4: TFM201610ALC-R47MTAA, libraries:WPN252010UR47MT, symbol TFM201610ALC-R47MTAA:TFM201610ALC-R47MTAA
- removed L5, L7: TFM201610ALC-R47MTAA, libraries:INDC2016X80N, symbol TFM201610ALC-R47MTAA:TFM201610ALC-R47MTAA
- removed L6: TFM201610ALC-R47MTAA, libraries:INDPM5752X300N, symbol TFM201610ALC-R47MTAA:TFM201610ALC-R47MTAA
- removed Q2, Q3, Q4, Q5: AON7407, libraries:DFN_3X3_EP, symbol AON7407:AON7407
- removed R10, R11, R12, R13, R14, R15, R16, R17, R18, R19, R20, R21, R22, R23, R24, R25, R26, R27, R28, R29, R30, R39, R40, R41, R42, R43, R5, R9: R, Resistor_SMD:R_0805_2012Metric_Pad1.20x1.40mm_HandSolder, symbol Device:R
- removed U1, U6, U7, U8: INA138, Package_TO_SOT_SMD:SOT-23-5, symbol Amplifier_Current:INA138
- removed U10, U11, U15, U16, U17, U18, U19, U20, U22, U23, U9: MCP9700AT-ETT, Package_TO_SOT_SMD:SOT-23, symbol Sensor_Temperature:MCP9700AT-ETT
- removed U24, U25, U26, U27, U28: Mounting_Hole_M2, mount_holes:Hole_screw_M1p2, symbol Mounting_Holes:Mounting_Hole_M2
- removed Z2: BZT52-C5V1J, Diode_SMD:D_SOD-323F, symbol Diode:MM3Zxx
- added C? (x16): C, Capacitor_SMD:C_0603_1608Metric_Pad1.08x0.95mm_HandSolder, symbol Device:C
- added C? (x2): C, Capacitor_SMD:C_0805_2012Metric_Pad1.18x1.45mm_HandSolder, symbol Device:C
- added L? (x2): SRP7050AA-220M, libraries:INDPM5752X300N, symbol SRP7050AA-220M:SRP7050AA-220M
- added R? (x2): (no value), symbol Device:R
- added R? (x5): R, Resistor_SMD:R_0805_2012Metric_Pad1.20x1.40mm_HandSolder, symbol Device:R
- D17: value WireHole_1p5 -> (none); footprint libraries:WireHole_1p2 -> (none)
- D72: value Gnd -> (none); footprint Flat_Wires_Pads:Wire_Hole_1mm -> (none)
- Z1: value BZT52-C5V1J -> (none); footprint Diode_SMD:D_SOD-323F -> (none)
Connections:
- net at C12.1, C5.1, C8.1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: now also R?.1, R?.2; no longer D4.1 (Conn), L2.1
- net at C10.2, C11.2, C12.2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: now also C?.2, C?.2, C?.2, C?.2, C?.2, C?.2, C?.2, C?.2, C?.2, C?.2, C?.2, C?.2, C?.2, C?.2, C?.2, C?.2
- net at D12.1, Z1.1 (K): now also R?.2; no longer C13.1, L1.2
- net at C10.1, L1.1: now also R?.2; no longer D11.1 (Conn)
- net at C58.2, D89.1 (Conn), R36.1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: now also C?.2
- net at C51.2, D72.1 (Conn), R32.1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: now also C?.2
- net at R33.1, R34.2: now also R?.2; no longer D73.1 (Conn)
- net at R37.1, R38.2: now also R?.2; no longer D90.1 (Conn)
- new net: L2.1, R?.2
- new net: C?.1, C?.1, C?.1, C?.1, C?.1, C?.1, D4.1 (Conn), L?.1
- new net: C?.1, C?.1, C?.1, C?.1, C?.1, C?.1, L?.2, R?.1
- new net: C?.1, C?.1, L?.1, R?.2
- new net: C?.1, C?.1, L?.2, R?.1
- new net: C?.1, D73.1 (Conn), R?.1
- new net: C?.1, D90.1 (Conn), R?.1
- new net: C13.1, L1.2, R?.1
- new net: D11.1 (Conn), R?.1
Other:
- moved on the sheet: C1, C10, C11, C12, C13, C2, C3, C4, C49, C5, C50, C51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

Commit message: Noise research for TSP40211 003
Parts:
- removed D11: Wire_Pad_01, Flat_Wires_Pads:Wire_Hole_1mm, symbol Connectors_for_Wire:Wire_Pad_01
- removed D71: CS_Out, Flat_Wires_Pads:Wire_Hole_1mm, symbol Connectors_for_Wire:Wire_Pad_01
- removed D79: CS_In, Flat_Wires_Pads:Wire_Hole_1mm, symbol Connectors_for_Wire:Wire_Pad_01
- removed R?: R, Resistor_SMD:R_0805_2012Metric_Pad1.20x1.40mm_HandSolder, symbol Device:R
- added C30, C31, C32, C33, C34, C35, C36, C37: C, Capacitor_SMD:C_0805_2012Metric_Pad1.18x1.45mm_HandSolder, symbol Device:C
- added D10, D11, D13, D14, D2, D3, D5, D7, D8, D9: WireHole_1p5, libraries:WireHole_1p2, symbol Connectors_for_Wire:WireHole_1p5
- C10, C5: footprint Capacitor_SMD:C_0603_1608Metric_Pad1.08x0.95mm_HandSolder -> Capacitor_SMD:C_0805_2012Metric_Pad1.18x1.45mm_HandSolder
- C14, C15, C16, C17, C18, C19, C20, C21, C22, C23, C24, C25, C26, C27: renamed from C?; footprint Capacitor_SMD:C_0603_1608Metric_Pad1.08x0.95mm_HandSolder -> Capacitor_SMD:C_0805_2012Metric_Pad1.18x1.45mm_HandSolder
- C8: footprint Capacitor_SMD:C_1206_3216Metric_Pad1.33x1.80mm_HandSolder -> Capacitor_SMD:C_0805_2012Metric_Pad1.18x1.45mm_HandSolder
- D17: value (none) -> WireHole_1p5; footprint (none) -> libraries:WireHole_1p2
- D72: value (none) -> Gnd; footprint (none) -> Flat_Wires_Pads:Wire_Hole_1mm
- R11, R9: renamed from R?; value (none) -> R; footprint (none) -> Resistor_SMD:R_0805_2012Metric_Pad1.20x1.40mm_HandSolder
- U2, U3, U4, U5: footprint mount_holes:Hole_screw_M1p2 -> Mounting_Wuerth:Mounting_Wuerth_WA-SMST-2.7mm_H1mm_9774010951
- Z1: value (none) -> BZT52-C5V1J; footprint (none) -> Diode_SMD:D_SOD-323F
- gave numbers to parts that had none: 10
Connections:
- net at C12.1, C5.1, C8.1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: now also D8.1 (Conn); no longer R9.2
- net at C10.2, C11.2, C12.2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: now also C29.2, C51.2, C58.2, C6.2, D72.1 (Conn), D89.1 (Conn), R32.1, R34.1, R36.1, R38.1, U14.2 (GND), U21.2 (GND), C30.2, C31.2, C32.2, C33.2, C34.2, C35.2, C36.2, C37.2
- net at C14.1, C15.1, C16.1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: now also R31.2, R33.2, U14.4 (-), D9.1 (Conn); no longer D4.1 (Conn)
- net at C10.1, L1.1: now also C31.1, C32.1, C36.1, D11.1 (Conn)
- net at C17.1, C19.1, L3.1: now also D4.1 (Conn); no longer R10.2
- net at C58.1, R35.1, U21.3 (+)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: now also D14.1 (Conn)
- net at C13.1, R12.1: now also C30.1, D10.1 (Conn); no longer L1.2
- new net: C33.1, C34.1, C35.1, C37.1, D13.1 (Conn), L1.2
- new net: D7.1 (Conn), R9.2
- new net: D3.1 (Conn), R10.2
Other:
- moved on the sheet: C10, C13, C29, C51, C58, C6, D1, D12, D70, D72, D73, D78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
