File: NoiseResearch_TPS40211_Core/Main_PCB_003.kicad_pcb (KiCad board)
At the start: 2 copper layers, 37.3 x 20.1 mm, 42 parts, among them IC1 TPS40211QDGQRQ1, Q1 AON7407, U12 MCP9700AT-ETT, U13 MCP9700AT-ETT, U2 Mounting_Hole_M2, U3 Mounting_Hole_M2, U4 Mounting_Hole_M2, U5 Mounting_Hole_M2

Commit message: Noise research for TSP40211 005
Connections:
- Q1 pad 10: (no net) -> Net-(Q1-D_1)
- Q1 pad 11: (no net) -> Net-(Q1-D_1)
- Q1 pad 9: (no net) -> Net-(Q1-D_1)
Changed lines of the file:
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@@
     (pad "8" smd rect (at -0.975 -1.5) (size 0.3 0.4) (layers "F.Cu" "F.Paste" "F.Mask")
       (net 13 "Net-(Q1-D_1)") (pinfunction "D_4") (pintype "passive"))
-    (pad "9" smd rect (at -1.415 0 270) (size 0.38 0.43) (layers "F.Cu" "F.Paste" "F.Mask"))
-    (pad "10" smd rect (at 0 -0.36) (size 1.98 2.45) (layers "F.Cu" "F.Paste" "F.Mask"))
-    (pad "11" smd rect (at 1.415 0 270) (size 0.38 0.43) (layers "F.Cu" "F.Paste" "F.Mask"))
+    (pad "9" smd rect (at -1.415 0 270) (size 0.38 0.43) (layers "F.Cu" "F.Paste" "F.Mask")
+      (net 13 "Net-(Q1-D_1)"))
+    (pad "10" smd rect (at 0 -0.36) (size 1.98 2.45) (layers "F.Cu" "F.Paste" "F.Mask")
+      (net 13 "Net-(Q1-D_1)"))
+    (pad "11" smd rect (at 1.415 0 270) (size 0.38 0.43) (layers "F.Cu" "F.Paste" "F.Mask")
+      (net 13 "Net-(Q1-D_1)"))
   )
   (footprint "Resistor_SMD:R_0805_2012Metric_Pad1.20x1.40mm_HandSolder" (layer "F.Cu")
