File: NoiseResearch_TPS40211_Light/Main_PCB_002.kicad_sch (KiCad schematic)
At the start: 33 parts, among them IC1 TPS40211QDGQRQ1, Q1 AON7407, U2 Mounting_Hole_M2, U3 Mounting_Hole_M2, U4 Mounting_Hole_M2, U5 Mounting_Hole_M2

Commit message: BANO Step-Dn 001
Parts:
- removed D12: SS36, libraries:SODFL4626X120N, symbol SS36:SS36
- removed Q1: AON7407, libraries:DFN_3X3_EP, symbol AON7407:AON7407
- added CR1: PMEG10020ELRX, CFP3_SOD123W_NEX, symbol 2023-11-01_15-59-24:PMEG10020ELRX
- added L1, L3: VLS3012HBX-3R3M, IND_VLS3012HBX-3R3M_TDK, symbol 2023-11-01_16-17-53:VLS3012HBX-3R3M
- added Q2: SI7852DP-T1, POWERPAK_SO-8_SINGLE_VIS, symbol 2023-10-30_16-32-45:SI7852DP-T1
- added R10, R5, R9: R, symbol Device:R
- added U1: MAX17504ATP+, 21-0140_T2055+4C_MXM, symbol 2023-11-01_15-44-04:MAX17504ATP+
- added U6: LMR51420XDDCR, SOT23_DDC_TEX, symbol 2023-11-01_15-51-33:LMR51420XDDCR
- added U7, U8: TLV9061IDCKR, DCK5_TEX, symbol 2023-11-01_15-51-52:TLV9061IDCKR
Connections:
- net at R6.2: now also Q2.4
- net at R7.2, R8.1: now also Q2.1, Q2.2, Q2.3
- net at R12.2: now also CR1.1
- net at L2.2: now also CR1.2, Q2.5, Q2.6, Q2.7, Q2.8

Commit message: BANO Step-Dn 002
Parts:
- removed L3: VLS3012HBX-3R3M, IND_VLS3012HBX-3R3M_TDK, symbol 2023-11-01_16-17-53:VLS3012HBX-3R3M
- removed U1: MAX17504ATP+, 21-0140_T2055+4C_MXM, symbol 2023-11-01_15-44-04:MAX17504ATP+
- removed U6: LMR51420XDDCR, SOT23_DDC_TEX, symbol 2023-11-01_15-51-33:LMR51420XDDCR
- removed U7, U8: TLV9061IDCKR, DCK5_TEX, symbol 2023-11-01_15-51-52:TLV9061IDCKR
- added C10, C15, C16, C18, C19, C23, C25, C7: C, Capacitor_SMD:C_0805_2012Metric_Pad1.18x1.45mm_HandSolder, symbol Device:C
- added C14, C17, C20, C21, C22, C24, C6: C, Capacitor_SMD:C_0603_1608Metric_Pad1.08x0.95mm_HandSolder, symbol Device:C
- added CR2: MMSZ5228B-7-F, SOD123_DIO, symbol SOD123_DIO:MMSZ5228B-7-F
- added D11, D12, D13, D14, D15, D16, D18, D19, D2, D22, D23, D24, D25, D26, D3, D4, D5, D7, D9: WireHole_1p5, libraries:WireHole_1p2, symbol Connectors_for_Wire:WireHole_1p5
- added D20: BAT54S, Package_TO_SOT_SMD:SOT-23, symbol Diode:BAT54S
- added D21: LED, LED_SMD:LED_0603_1608Metric_Pad1.05x0.95mm_HandSolder, symbol Device:LED
- added L4: TFM252012ALMA-3R3MTAA, ul_TFM252012ALMA-3R3MTAA:IND_TFM252012_TDK, symbol IND_TFM252012_TDK:TFM252012ALMA-3R3MTAA
- added R13, R14, R15, R17: R, LED_SMD:LED_0805_2012Metric_Pad1.15x1.40mm_HandSolder, symbol Device:R
- added R16, R22, R23, R24, R25: R, LED_SMD:LED_0603_1608Metric_Pad1.05x0.95mm_HandSolder, symbol Device:R
- added R18, R19, R20, R21: 3314G-1-103E, ul_3314G-1-103E:POT_3314G, symbol 3314G:3314G-1-103E
- added U1: LMR51420XDDCR, ul_LMR51420XDDCR:SOT23_DDC_TEX, symbol SOT23_DDC_TEX:LMR51420XDDCR
- added U10, U6: TLV9061IDCKR, ul_TLV9061IDCKR:DCK5_TEX, symbol DCK5_TEX:TLV9061IDCKR
- added U11, U15: MMSZ4697T1G, ul_MMSZ4697T1G:SOD-123_ONS, symbol MMSZ4697T1G:MMSZ4697T1G
- added U12: SI7489DP-T1-E3, ul_SI7489DP-T1-E3:MOSFET_65DP-T1-E3_VIS, symbol SI7489DP:SI7489DP-T1-E3
- added U13, U14: AO3401A, ul_AO3401A:SOT-23-3L_AOS, symbol AO3401A:AO3401A
- added U7: NE555DR, ul_NE555DR:D8, symbol NE555DB:NE555DR
- added U8: ZXTR2012K-13, ul_ZXTR2012K-13:TO252-3L_DIO, symbol ZXTR2012K:ZXTR2012K-13
- added U9: MAX17504ATP+, 21-0140_T2055+4C_MXM, symbol 21-0140_T2055&plus_4C_MXM:MAX17504ATP+
- CR1: footprint CFP3_SOD123W_NEX -> ul_PMEG10020ELRX:CFP3_SOD123W_NEX
- L1: footprint IND_VLS3012HBX-3R3M_TDK -> ul_VLS3012HBX-3R3M:IND_VLS3012HBX-3R3M_TDK
- Q2: footprint POWERPAK_SO-8_SINGLE_VIS -> ul_SI7852DP-T1:POWERPAK_SO-8_SINGLE_VIS
- R10, R5, R9: footprint (none) -> LED_SMD:LED_0805_2012Metric_Pad1.15x1.40mm_HandSolder
Connections:
- net GND: now also U15.1 (CATHODE)
- net at C11.1, IC1.7 (ISNS), R7.1: now also U15.2 (ANODE)
- net at R10.1: now also R9.2, U10.3 (IN-)
- net at R10.2: now also U10.4 (OUT), U9.9 (FB)
- net at R9.1: now also R5.2, C10.2, C14.2, C15.2, C18.2, C7.2, D15.1 (Conn), D5.1 (Conn), R16.2, U10.2 (V-), U9.13 (SGND), U9.14 (PGND), U9.15 (PGND), U9.16 (PGND), U9.21 (EPAD)
- net at R5.1: now also D4.1 (Conn), U10.1 (IN+)
- net at L1.1: now also C16.1, D7.1 (Conn)
- net at L1.2: now also C17.2, U1.2 (SW)
- new net: D25.1 (Conn), U13.1 (G), U14.1 (G), U7.3 (OUT)
- new net: R22.2, U13.3 (D)
- new net: D21.2 (A), R23.1
- new net: C21.1, R23.2, R25.2, U8.3 (VOUT)
- new net: C24.1, U7.5 (CONT)
- new net: C23.1, D20.3 (COM), U7.2 (TRIG), U7.6 (THRES)
- new net: C25.1, U7.4 (RESET), U7.8 (VCC)
- new net: R19.3, R20.1, U7.7 (DISCH)
- new net: C22.1, D22.1 (Conn), R24.1, U11.2 (ANODE), U12.1 (S), U12.2 (S), U12.3 (S), U8.2 (VIN)
- new net: R16.1, U9.10 (RT)
- new net: C17.1, U1.6 (CB)
- new net: C19.1, D16.1 (Conn), R17.2, U1.3 (VIN)
- new net: C7.1, D2.1 (Conn), U9.1 (VIN), U9.2 (VIN), U9.3 (VIN)
- new net: C16.2, C19.2, C20.2, CR2.2, D18.1 (Conn), R13.2, R15.1, U1.1 (GND), U6.2 (V-)
- new net: D12.1 (Conn), U9.11 (MODE)
- new net: R22.1, R24.2, U11.1 (CATHODE), U12.4 (G)
- new net: C6.1, U9.20 (BST)
- new net: C6.2, L4.2, U9.17 (LX), U9.18 (LX), U9.19 (LX)
- new net: C15.1, D3.1 (Conn), L4.1
- new net: C10.1, C18.1, D11.1 (Conn), U10.5 (V+), U9.12 (VCC)
- new net: D24.1 (Conn), U12.5 (D), U12.6 (D), U12.7 (D), U12.8 (D)
- new net: D14.1 (Conn), U9.4 (EN/UVLO)
- new net: C14.1, U9.7 (SS)
- new net: R18.3, R19.1, R19.2
- new net: D20.1 (A), R18.1, R18.2
- new net: D21.1 (K), D26.1 (Conn), R25.1, U14.3 (D)
- new net: D9.1 (Conn), R13.1, U6.1 (IN+)
- new net: C20.1, CR2.1, R17.1, U6.5 (V+)
- new net: R14.1, R15.2, U6.3 (IN-)
- new net: R14.2, U1.4 (FB), U6.4 (OUT)
- new net: R20.2, R20.3, R21.1
- new net: D20.2 (K), R21.2, R21.3
- new net: D19.1 (Conn), U1.5 (EN)
- new net GND1: C21.2, C22.2, C23.2, C24.2, C25.2, D23.1 (Conn), U13.2 (S), U14.2 (S), U7.1 (GND), U8.1 (GND)
Other:
- moved on the sheet: D1, L1, R10, R5, R9
