File: BANO_Control_Module_Atmel/Main_PCB_002.kicad_pcb (KiCad board)
At the start: 2 copper layers, 45.7 x 26.7 mm, 27 parts, among them U11 MMSZ4697T1G, U12 SI7489DP-T1-E3, U13 AO3401A, U14 AO3401A, U7 NE555DR, U8 ZXTR2012K-13

Commit message: BANO Step-Dn 003
Parts:
- removed C23, C25: C, Capacitor_SMD:C_0805_2012Metric_Pad1.18x1.45mm_HandSolder
- removed C24: C, Capacitor_SMD:C_0603_1608Metric_Pad1.08x0.95mm_HandSolder
- removed D20: BAT54S, Package_TO_SOT_SMD:SOT-23
- removed R18, R19, R20, R21: 3314G-1-103E, ul_3314G-1-103E:POT_3314G
- removed U8: ZXTR2012K-13, ul_ZXTR2012K-13:TO252-3L_DIO
- added C1: C, Capacitor_SMD:C_0805_2012Metric_Pad1.18x1.45mm_HandSolder, F.Cu at (109.2, 87.6)
- added C2: C, Capacitor_SMD:C_0805_2012Metric_Pad1.18x1.45mm_HandSolder, F.Cu at (109.2, 90.6)
- added C3: C, Capacitor_SMD:C_0805_2012Metric_Pad1.18x1.45mm_HandSolder, F.Cu at (109.2, 93.6)
- added C4: C, Capacitor_SMD:C_0805_2012Metric_Pad1.18x1.45mm_HandSolder, F.Cu at (109.2, 96.6)
- added C5: C, Capacitor_SMD:C_0805_2012Metric_Pad1.18x1.45mm_HandSolder, F.Cu at (100.8, 119.3)
- added C6: C, Capacitor_SMD:C_0805_2012Metric_Pad1.18x1.45mm_HandSolder, F.Cu at (103.8, 123.1)
- added C7: C, Capacitor_SMD:C_0805_2012Metric_Pad1.18x1.45mm_HandSolder, F.Cu at (100.8, 123.1)
- added D5: WireHole_1p5, Wire_holes:WireHole_1p2, F.Cu at (121.9, 96.9)
- added D6: WireHole_1p5, Wire_holes:WireHole_1p2, F.Cu at (162.5, 136.6)
- added D7: WireHole_1p5, Wire_holes:WireHole_1p2, F.Cu at (124.5, 94.3)
- added L1: L, ul_VLS3012HBX-3R3M:IND_VLS3012HBX-3R3M_TDK-L, F.Cu at (133.3, 103.1)
- added R1: R, Resistor_SMD:R_0603_1608Metric_Pad0.98x0.95mm_HandSolder, F.Cu at (113.7, 102.7)
- added R2: R, Resistor_SMD:R_0603_1608Metric_Pad0.98x0.95mm_HandSolder, F.Cu at (113.7, 105.2)
- added R3: R, Resistor_SMD:R_0603_1608Metric_Pad0.98x0.95mm_HandSolder, F.Cu at (113.7, 107.7)
- added R4: R, Resistor_SMD:R_0603_1608Metric_Pad0.98x0.95mm_HandSolder, F.Cu at (113.7, 110.2)
- added R5: R, Resistor_SMD:R_0603_1608Metric_Pad0.98x0.95mm_HandSolder, F.Cu at (113.7, 112.7)
- added R6: R, Resistor_SMD:R_0603_1608Metric_Pad0.98x0.95mm_HandSolder, F.Cu at (113.7, 115.2)
- added R7: R, Resistor_SMD:R_0603_1608Metric_Pad0.98x0.95mm_HandSolder, F.Cu at (118.1, 102.7)
- added U1: SI7489DP-T1-E3, ul_SI7489DP-T1-E3:MOSFET_65DP-T1-E3_VIS, F.Cu at (112.6, 124.0)
- added U2: MMSZ4697T1G, ul_MMSZ4697T1G:SOD-123_ONS, F.Cu at (133.3, 108.6)
- added U3: ATtiny25-20S, Package_SO:SOIC-8W_5.3x5.3mm_P1.27mm, F.Cu at (125.9, 89.6)
- added U4: ZXTR2005ZQ-13, ul_ZXTR2005ZQ-13:SOT-89_4P5X2P45_DIO, F.Cu at (132.7, 96.4)
- added U5: FBMH4525HM162NT, ul_FBMH4525HM162NT:FBMH4525HM162NT_TAY, F.Cu at (95.9, 121.5)
- added U6: LM5164DDAT, ul_LM5164DDAT:DDA0008E-IPC_A, F.Cu at (125.6, 103.9)
- C21, C22: footprint Capacitor_SMD:C_0603_1608Metric_Pad1.08x0.95mm_HandSolder -> Capacitor_SMD:C_0805_2012Metric_Pad1.18x1.45mm_HandSolder
- U7: value NE555DR -> INA168; footprint ul_NE555DR:D8 -> Package_TO_SOT_SMD:SOT-23-5
- moved D1 47.6 mm to (121.9, 94.3)
- moved U12 47.6 mm to (116.4, 97.6)
- moved R25 43.9 mm to (118.1, 112.7), turned to 0 degrees
- moved D23 43.8 mm to (89.8, 125.2)
- moved D22 43.4 mm to (90.0, 121.5)
- moved R23 41.8 mm to (118.1, 107.7), turned to 0 degrees
- moved C21 41.1 mm to (109.2, 108.7), turned to 0 degrees
- moved D24 41.0 mm to (127.1, 94.3)
- moved D26 39.1 mm to (127.1, 99.5)
- moved R24 38.4 mm to (118.1, 110.2), turned to 0 degrees
- moved R22 37.0 mm to (118.1, 105.2), turned to 0 degrees
- moved D25 33.6 mm to (127.1, 96.9)
- moved C22 32.2 mm to (109.2, 111.7), turned to 0 degrees
- moved U14 29.9 mm to (127.8, 109.6), turned to 0 degrees
- moved U13 29.9 mm to (123.0, 109.6), turned to 0 degrees
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Connections:
- C22 pad 1: Net-(D22-Conn) -> Net-(D6-Conn)
- R24 pad 1: Net-(D22-Conn) -> Net-(U11-ANODE)
- U11 pad 2: Net-(D22-Conn) -> Net-(U11-ANODE)
- U12 pad 1: Net-(D22-Conn) -> Net-(U11-ANODE)
- U12 pad 2: Net-(D22-Conn) -> Net-(U11-ANODE)
- U12 pad 3: Net-(D22-Conn) -> Net-(U11-ANODE)
- U7 pad 1: GND1 -> Net-(U6-FB)
- U7 pad 2: Net-(D20-COM) -> GND1
- U7 pad 3: Net-(D25-Conn) -> Net-(U7-+)
- U7 pad 4: Net-(U7-RESET) -> Net-(D6-Conn)
- U7 pad 5: Net-(U7-CONT) -> Net-(U7-+)
Routing:
- net Net-(D22-Conn): track 44.3 -> 0.00 mm
- net Net-(D20-COM): track 30.2 -> 0.00 mm
- net Net-(U7-DISCH): track 20.6 -> 0.00 mm
- net Net-(U3-VCC): track 20.2 -> 0.00 mm, vias 2 -> 0
- net Net-(D25-Conn): track 16.8 -> 0.00 mm
- net Net-(U7-RESET): track 10.2 -> 0.00 mm, vias 2 -> 0
- net Net-(D20-A): track 9.71 -> 0.00 mm
- net Net-(D20-K): track 9.51 -> 0.00 mm
- net Net-(R20-Pad2): track 9.40 -> 0.00 mm
- net Net-(D21-K): track 9.23 -> 0.00 mm
- net Net-(R18-Pad3): track 9.10 -> 0.00 mm
- net Net-(U11-CATHODE): track 9.04 -> 0.00 mm
- net Net-(D24-Conn): track 8.60 -> 0.00 mm
- net Net-(U7-CONT): track 3.23 -> 0.00 mm
- net Net-(U13-D): track 2.98 -> 0.00 mm
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- removed copper zone on B.Cu, net GND1
- removed copper zone on F.Cu, net GND1
Other:
- board outline removed
- board text removed: "GND"
- board text removed: "PWR"
- board text removed: "U"
- board text removed: "in"
