File: BANO_Control_Module_Atmel/Main_PCB_002.kicad_sch (KiCad schematic)
At the start: 25 parts, among them U1 SI7489DP-T1-E3, U11 MMSZ4697T1G, U12 SI7489DP-T1-E3, U13 AO3401A, U14 AO3401A, U2 MMSZ4697T1G, U3 ATtiny25-20S, U4 ZXTR2005ZQ-13, U5 FBMH4525HM162NT, U6 LM5164DDAT, U8 ZXTR2012K-13

Commit message: BANO Step-Dn 003
Parts:
- removed U8: ZXTR2012K-13, ul_ZXTR2012K-13:TO252-3L_DIO, symbol ZXTR2012K:ZXTR2012K-13
- added C1, C2, C3, C4, C5, C6, C7: C, Capacitor_SMD:C_0805_2012Metric_Pad1.18x1.45mm_HandSolder, symbol Device:C
- added D5, D6, D7: WireHole_1p5, Wire_holes:WireHole_1p2, symbol Connectors_for_Wire:WireHole_1p5
- added L1: L, ul_VLS3012HBX-3R3M:IND_VLS3012HBX-3R3M_TDK-L, symbol Device:L
- added R2, R3, R4, R5, R6, R7: R, Resistor_SMD:R_0603_1608Metric_Pad0.98x0.95mm_HandSolder, symbol Device:R
- added U7: INA168, Package_TO_SOT_SMD:SOT-23-5, symbol Amplifier_Current:INA168
- C21, C22: footprint Capacitor_SMD:C_0603_1608Metric_Pad1.08x0.95mm_HandSolder -> Capacitor_SMD:C_0805_2012Metric_Pad1.18x1.45mm_HandSolder
- U4: footprint SOT-89_4P5X2P45_DIO -> ul_ZXTR2005ZQ-13:SOT-89_4P5X2P45_DIO
- U5: footprint FBMH4525HM162NT_TAY -> ul_FBMH4525HM162NT:FBMH4525HM162NT_TAY
- U6: footprint DDA0008E-IPC_A -> ul_LM5164DDAT:DDA0008E-IPC_A
Connections:
- net GND1: now also U4.1, U6.1 (GND), U6.9 (EP), C2.2, C3.2, C4.2, C5.2, C6.2, C7.2, D7.1 (Conn), R2.2, R4.2, R5.2, U7.2 (GND)
- net at D25.1 (Conn), U13.1 (G), U14.1 (G): now also U3.2 (XTAL1/PB3)
- net at C21.1, R23.2, R25.2: now also U3.8 (VCC), U4.3
- net at R24.1, U1.1 (S), U1.2 (S)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: now also R6.1; no longer C22.1
- net at U1.5 (D), U1.6 (D), U1.7 (D)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: now also U5.2, U6.2 (VIN), U6.3 (EN_UVLO), C5.1, C6.1, C7.1; no longer D22.1 (Conn)
- net at U6.4 (RON): now also R2.1
- net at U6.5 (FB): now also R4.1, U7.1
- net at U6.7 (BST): now also C1.1
- net at U6.8 (SW): now also C1.2, L1.1
- net at U5.1: now also D22.1 (Conn)
- net at U4.2: now also C22.1, D6.1 (Conn), R3.1, U7.4 (-)
- net at U3.3 (XTAL2/PB4): now also R7.1
- net at U3.7 (PB2): now also C3.1, R5.1, R6.2
- new net: C2.1, L1.2, R3.2, U7.3 (+), U7.5 (V+)
- new net: C4.1, D5.1 (Conn), R7.2
Other:
- moved on the sheet: C21, C22, D1, D21, D22, D23, D24, D25, D26, R1, R22, R23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
