File: BANO_StepDown_LM5160_Total/Main_PCB_002.kicad_sch (KiCad schematic)
At the start: 26 parts, among them U1 LM5160ADNTR, U2 TLV9061IDCKR

Commit message: BANO Step-Dn 004
Parts:
- removed D1, D2: WireHole_1p5, Wire_holes:WireHole_1p2, symbol Connectors_for_Wire:WireHole_1p5
- added D6, D7, D8: LED_Cree_XHP50_6V, LED_SMD:LED_Cree-XHP50_6V, symbol LED:LED_Cree_XHP50_6V
- C1, C2, C26, C27, C3: footprint Capacitor_SMD:C_0603_1608Metric_Pad1.08x0.95mm_HandSolder -> Capacitor_SMD:C_0402_1005Metric_Pad0.74x0.62mm_HandSolder
- C28, C5: footprint Capacitor_SMD:C_0805_2012Metric_Pad1.18x1.45mm_HandSolder -> Capacitor_SMD:C_0603_1608Metric_Pad1.08x0.95mm_HandSolder
- C4, C6: footprint Capacitor_SMD:C_0805_2012Metric_Pad1.18x1.45mm_HandSolder -> Capacitor_SMD:C_0402_1005Metric_Pad0.74x0.62mm_HandSolder
- R1, R15, R3, R4, R6, R7, R9: footprint Resistor_SMD:R_0603_1608Metric_Pad0.98x0.95mm_HandSolder -> Resistor_SMD:R_0402_1005Metric_Pad0.72x0.64mm_HandSolder
Connections:
- net GND2: now also D6.3 (PAD), D7.3 (PAD), D8.3 (PAD)
- net at C28.1, C4.1, L1.1: now also D6.2 (A)
- net at R2.1, U2.1 (IN+): now also D8.1 (K)
- new net: D6.1 (K), D7.2 (A)
- new net: D7.1 (K), D8.2 (A)
Other:
- moved on the sheet: D27, D28
