File: BANO_StepDown_LM5160_Control_Module/Main_PCB_002.kicad_pcb (KiCad board)
At the start: 2 copper layers, 88.9 x 22.2 mm, 87 parts, among them Q1 BSS123, U1 INA193, U3 LM5164DDA, U4 SI7489DP-T1-E3, U5 SI7489DP-T1-E3, U6 STM32G031G8Ux, U7 SI7489DP-T1-E3, U8 LM5164DDA

Commit message: BANO MainModule Double Strob
Parts:
- removed D22, D23, D24, D25, D26, D27, D28, D29, D30: WireHole_1p5, Wire_holes:WireHole_1p2
- removed LED2, LED3: HSMW-C191-U0000, ul_HSMW-C191-U0000:LED_91-U0000
- removed Q1: BSS123, Package_TO_SOT_SMD:SOT-23
- removed R21, R22, R29, R30, R31: R, Resistor_SMD:R_0402_1005Metric_Pad0.72x0.64mm_HandSolder
- removed R23, R24, R25, R26, R27, R28: BLM18KG102SH1D, ul_BLM18KG102SH1D:RES_0603_1P6XP8_MUR
- removed U6: STM32G031G8Ux, Package_DFN_QFN:QFN-28_4x4mm_P0.5mm
- removed U7: SI7489DP-T1-E3, ul_SI7852DP-T1:POWERPAK_SO-8_SINGLE_VIS
- removed U8: LM5164DDA, Package_SO:HSOP-8-1EP_3.9x4.9mm_P1.27mm_EP2.41x3.1mm_ThermalVias
- added C16: C, Capacitor_SMD:C_0603_1608Metric_Pad1.08x0.95mm_HandSolder, F.Cu at (121.4, 109.6)
- added C17: C, Capacitor_SMD:C_0805_2012Metric_Pad1.18x1.45mm_HandSolder, F.Cu at (89.8, 76.9)
- added C18: C, Capacitor_SMD:C_0805_2012Metric_Pad1.18x1.45mm_HandSolder, F.Cu at (89.8, 79.9)
- added C19: C, Capacitor_SMD:C_0805_2012Metric_Pad1.18x1.45mm_HandSolder, F.Cu at (89.8, 82.9)
- added C20: C, Capacitor_SMD:C_0805_2012Metric_Pad1.18x1.45mm_HandSolder, F.Cu at (51.1, 125.1)
- added C21: C, Capacitor_SMD:C_0805_2012Metric_Pad1.18x1.45mm_HandSolder, F.Cu at (89.8, 88.9)
- added C22: C, Capacitor_SMD:C_0805_2012Metric_Pad1.18x1.45mm_HandSolder, F.Cu at (43.1, 113.3)
- added C23: C, Capacitor_SMD:C_0805_2012Metric_Pad1.18x1.45mm_HandSolder, F.Cu at (38.3, 113.3)
- added C24: C, Capacitor_SMD:C_0805_2012Metric_Pad1.18x1.45mm_HandSolder, F.Cu at (94.6, 82.9)
- added C25: C, Capacitor_SMD:C_0805_2012Metric_Pad1.18x1.45mm_HandSolder, F.Cu at (48.8, 79.5)
- added C26: C, Capacitor_SMD:C_0805_2012Metric_Pad1.18x1.45mm_HandSolder, F.Cu at (43.6, 79.6)
- added C5: C, Capacitor_SMD:C_0805_2012Metric_Pad1.18x1.45mm_HandSolder, F.Cu at (64.2, 73.6)
- added C6: C, Capacitor_SMD:C_0805_2012Metric_Pad1.18x1.45mm_HandSolder, F.Cu at (59.9, 73.6)
- added L1: SWPA4030S1R0NT, ul_VLS252012HBU-220M:IND_VLS252012_TDK, F.Cu at (62.0, 70.8)
- added L4: SWPA4030S1R0NT, ul_VLS252012HBU-220M:IND_VLS252012_TDK, F.Cu at (41.1, 110.0)
- added L5: SWPA4030S1R0NT, ul_VLS252012HBU-220M:IND_VLS252012_TDK, F.Cu at (45.8, 76.5)
- added U2: STM32G031G8Ux, Package_DFN_QFN:QFN-28_4x4mm_P0.5mm, F.Cu at (103.4, 118.9)
- C1: footprint Capacitor_SMD:C_0805_2012Metric_Pad1.18x1.45mm_HandSolder -> Capacitor_SMD:C_0402_1005Metric_Pad0.74x0.62mm_HandSolder
- C10, C11, C14, C8: footprint Capacitor_SMD:C_0603_1608Metric_Pad1.08x0.95mm_HandSolder -> Capacitor_SMD:C_0805_2012Metric_Pad1.18x1.45mm_HandSolder
- C12, C13, C7: footprint Capacitor_SMD:C_0402_1005Metric_Pad0.74x0.62mm_HandSolder -> Capacitor_SMD:C_0603_1608Metric_Pad1.08x0.95mm_HandSolder
- C9: footprint Capacitor_SMD:C_0805_2012Metric -> Capacitor_SMD:C_0805_2012Metric_Pad1.18x1.45mm_HandSolder
- D14, D6: value MM5Zxx -> WireHole_1p5; footprint Diode_SMD:D_SOD-523 -> Wire_holes:WireHole_1p2
- D20: value BAT54C -> WireHole_1p5; footprint Package_TO_SOT_SMD:SOT-23 -> Wire_holes:WireHole_1p2
- D4: value WireHole_1p5 -> 1N5711UR; footprint Wire_holes:WireHole_1p2 -> Diode_SMD:D_MELF
- R1: value R -> BLM18KG102SH1D; footprint Resistor_SMD:R_0603_1608Metric_Pad0.98x0.95mm_HandSolder -> ul_BLM18KG102SH1D:RES_0603_1P6XP8_MUR
- R13: value R -> BLM18KG102SH1D; footprint Resistor_SMD:R_0402_1005Metric_Pad0.72x0.64mm_HandSolder -> ul_BLM18KG102SH1D:RES_0603_1P6XP8_MUR
- R15, R4, R5, R6, R7, R9: value BLM18KG102SH1D -> R; footprint ul_BLM18KG102SH1D:RES_0603_1P6XP8_MUR -> Resistor_SMD:R_0402_1005Metric_Pad0.72x0.64mm_HandSolder
- U1: value INA193 -> SI7489DP-T1-E3; footprint Package_TO_SOT_SMD:SOT-23-5 -> ul_SI7852DP-T1:POWERPAK_SO-8_SINGLE_VIS
- U3: value LM5164DDA -> LM5160ADNTR; footprint Package_SO:HSOP-8-1EP_3.9x4.9mm_P1.27mm_EP2.41x3.1mm_ThermalVias -> ul_LM5160ADNTR:DNT0012B
- U4: value SI7489DP-T1-E3 -> LM5160ADNTR; footprint ul_SI7852DP-T1:POWERPAK_SO-8_SINGLE_VIS -> ul_LM5160ADNTR:DNT0012B
- U5: value SI7489DP-T1-E3 -> TLV9061IDCKR; footprint ul_SI7852DP-T1:POWERPAK_SO-8_SINGLE_VIS -> ul_TLV9061IDCKR:DCK5_TEX
- moved C15 79.4 mm to (33.1, 89.7), turned to 0 degrees
- moved D8 77.5 mm to (81.6, 91.7)
- moved D9 76.0 mm to (81.6, 94.3)
- moved L2 74.7 mm to (34.0, 86.8), turned to 0 degrees
- moved D18 73.5 mm to (86.8, 91.7)
- moved D1 69.8 mm to (79.0, 91.7)
- moved U1 67.1 mm to (47.1, 97.0)
- moved LED1 65.8 mm to (83.2, 133.8), turned to 0 degrees
- moved D13 65.4 mm to (84.2, 91.7)
- moved R1 64.5 mm to (76.1, 63.0), turned to 0 degrees
- moved U4 63.5 mm to (139.9, 112.0), turned to 0 degrees
- moved D21 61.1 mm to (86.8, 99.5)
- moved C3 57.9 mm to (80.2, 79.9), turned to 0 degrees
- moved C10 56.1 mm to (85.0, 79.9)
- moved D11 56.0 mm to (81.6, 99.5), turned to 0 degrees
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Connections:
- C1 pad 1: Net-(C1-Pad1) -> Net-(U2-PA4)
- C10 pad 1: Net-(D26-Conn) -> Net-(U3-VIN)
- C11 pad 1: Net-(U6-PF2) -> Net-(U4-SS)
- C12 pad 1: Net-(D14-A) -> Net-(D16-Conn)
- C13 pad 1: Net-(U6-PA4) -> Net-(U3-BST)
- C13 pad 2: GND2 -> Net-(C13-Pad2)
- C14 pad 1: Net-(U8-BST) -> Net-(U3-VCC)
- C14 pad 2: Net-(U8-SW) -> GND2
- C15 pad 1: Net-(U1-+) -> Net-(C15-Pad1)
- C2 pad 1: Net-(C2-Pad1) -> Net-(D2-Conn)
- C3 pad 1: Net-(C3-Pad1) -> Net-(D3-Conn)
- C4 pad 1: Net-(D26-Conn) -> Net-(U2-PF2)
- C7 pad 1: Net-(D5-A) -> Net-(D16-Conn)
- C8 pad 1: Net-(U3-BST) -> Net-(U3-VIN)
- C8 pad 2: Net-(U3-SW) -> GND2
- C9 pad 1: Net-(D26-Conn) -> Net-(U3-SS)
- D12 pad 1: Net-(D12-Conn) -> GND2
- D16 pad 1: Net-(D15-Conn) -> Net-(D16-Conn)
- D18 pad 1: GND2 -> Net-(D18-Conn)
- D20 pad 1: Net-(D24-Conn) -> Net-(D19-Conn)
- D4 pad 1: GND2 -> Net-(D4-K)
- D5 pad 1: Net-(D25-Conn) -> Net-(D4-K)
- D6 pad 1: Net-(D24-Conn) -> Net-(D6-Conn)
- L2 pad 1: Net-(D26-Conn) -> Net-(C15-Pad1)
- L2 pad 2: Net-(U3-BST) -> Net-(C13-Pad2)
- L3 pad 1: Net-(U1-+) -> Net-(D16-Conn)
- L3 pad 2: Net-(U8-BST) -> Net-(C16-Pad2)
- LED1 pad 1: unconnected-(LED1-Pad1) -> GND2
- R1 pad 1: Net-(U1--) -> Net-(D1-Conn)
- R1 pad 2: Net-(U1-+) -> Net-(R1-Pad2)
- R10 pad 1: GND2 -> Net-(LED1-Pad2)
- R10 pad 2: Net-(D5-A) -> Net-(U2-PB0)
- R11 pad 1: Net-(D6-A) -> Net-(U3-RON)
- R11 pad 2: Net-(D24-Conn) -> Net-(U3-VIN)
- R12 pad 1: GND2 -> Net-(U4-RON)
- R12 pad 2: Net-(U3-RON) -> Net-(U3-VIN)
- R13 pad 1: GND2 -> Net-(D16-Conn)
- R13 pad 2: Net-(U3-FB) -> Net-(D13-Conn)
- R14 pad 1: Net-(U3-FB) -> Net-(C17-Pad2)
- R14 pad 2: Net-(D26-Conn) -> Net-(C13-Pad2)
- R15 pad 1: Net-(U6-PA3) -> GND2
- R15 pad 2: Net-(D11-Conn) -> Net-(D21-Conn)
- R16 pad 1: Net-(U6-PA0) -> Net-(U3-FB)
- R16 pad 2: Net-(U3-EN/UVLO) -> Net-(C19-Pad2)
- R17 pad 1: GND2 -> Net-(U4-FB)
- R17 pad 2: Net-(U6-PA0) -> Net-(D16-Conn)
- R18 pad 1: Net-(U6-PA1) -> GND2
- R18 pad 2: Net-(D26-Conn) -> Net-(U4-FB)
- R19 pad 1: GND2 -> Net-(U5-IN-)
- R19 pad 2: Net-(U6-PA1) -> Net-(U3-FB)
- R2 pad 1: Net-(U6-PB4) -> Net-(D3-Conn)
- R2 pad 2: Net-(D22-Conn) -> Net-(U2-PB5)
- R20 pad 2: Net-(D14-A) -> Net-(U5-IN-)
- R3 pad 1: Net-(U6-PB5) -> Net-(D2-Conn)
- R3 pad 2: Net-(D24-Conn) -> Net-(U2-PB4)
- R4 pad 1: Net-(D12-Conn) -> Net-(U2-PA4)
- R4 pad 2: Net-(C1-Pad1) -> Net-(R1-Pad2)
- R5 pad 1: Net-(D3-Conn) -> GND2
- R5 pad 2: Net-(C2-Pad1) -> Net-(D5-A)
- R6 pad 1: Net-(U1--) -> Net-(U2-PA1)
- R6 pad 2: Net-(D2-Conn) -> Net-(D16-Conn)
- R7 pad 1: Net-(D13-Conn) -> GND2
- R7 pad 2: Net-(R21-Pad2) -> Net-(U2-PA1)
- R8 pad 1: Net-(Q1-D) -> Net-(U2-PA0)
- R8 pad 2: Net-(D6-A) -> Net-(U3-VIN)
- R9 pad 1: Net-(U6-PA2) -> GND2
- R9 pad 2: Net-(D10-Conn) -> Net-(U2-PA0)
- U1 pad 1: Net-(U8-FB) -> Net-(D4-K)
- U1 pad 2: GND2 -> Net-(D4-K)
- U1 pad 3: Net-(U1-+) -> Net-(D4-K)
- U1 pad 4: Net-(U1--) -> Net-(D5-A)
- U1 pad 5: Net-(D26-Conn) -> Net-(D3-Conn)
- U3 pad 2: Net-(U3-EN/UVLO) -> GND2
- U3 pad 3: Net-(U3-EN/UVLO) -> Net-(U3-VIN)
- U3 pad 4: Net-(U3-RON) -> Net-(U2-PA6)
- U3 pad 5: Net-(U3-FB) -> Net-(U3-RON)
- U3 pad 6: unconnected-(U3-PGOOD-Pad6) -> Net-(U3-SS)
- U3 pad 7: Net-(U3-BST) -> unconnected-(U3-FPWM-Pad7)
- U3 pad 8: Net-(U3-SW) -> Net-(U3-FB)
- U3 pad 9: GND2 -> Net-(U3-VCC)
- U4 pad 1: Net-(D25-Conn) -> GND2
- U4 pad 2: Net-(D25-Conn) -> GND2
- U4 pad 3: Net-(D25-Conn) -> Net-(U3-VIN)
- U4 pad 4: Net-(D5-A) -> Net-(U3-VIN)
- U4 pad 5: Net-(C2-Pad1) -> Net-(U4-RON)
- U4 pad 6: Net-(C2-Pad1) -> Net-(U4-SS)
- U4 pad 7: Net-(C2-Pad1) -> unconnected-(U4-FPWM-Pad7)
- U4 pad 8: Net-(C2-Pad1) -> Net-(U4-FB)
- U5 pad 1: Net-(D24-Conn) -> Net-(D21-Conn)
- U5 pad 2: Net-(D24-Conn) -> GND2
- U5 pad 3: Net-(D24-Conn) -> Net-(U5-IN-)
- U5 pad 4: Net-(D6-A) -> Net-(U3-FB)
- U5 pad 5: Net-(C3-Pad1) -> Net-(D16-Conn)
Routing:
- net Net-(D26-Conn): track 85.5 -> 0.00 mm, vias 3 -> 0
- net Net-(D24-Conn): track 70.5 -> 0.00 mm, vias 2 -> 0
- net Net-(D22-Conn): track 69.5 -> 0.00 mm, vias 2 -> 0
- net Net-(U6-PA0): track 48.9 -> 0.00 mm
- net Net-(U6-PA1): track 28.9 -> 0.00 mm
- net Net-(Q1-G): track 24.7 -> 0.00 mm, vias 2 -> 0
- net Net-(U8-FB): track 23.6 -> 0.00 mm
- net Net-(C1-Pad1): track 17.8 -> 0.00 mm
- net Net-(C2-Pad1): track 16.6 -> 0.00 mm
- net Net-(U3-FB): track 15.3 -> 0.00 mm
- net Net-(D25-Conn): track 14.5 -> 0.00 mm
- net Net-(D14-Conn): track 14.2 -> 0.00 mm
- net Net-(U6-PA13): track 14.1 -> 0.00 mm
- net Net-(U6-PA14): track 13.2 -> 0.00 mm
- net Net-(U6-PB7): track 12.6 -> 0.00 mm, vias 2 -> 0
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- removed copper zone on B.Cu, net GND2
- removed copper zone on F.Cu, net GND2
Other:
- board outline removed
- board text removed: "3.3B"
- board text removed: "CLK"
- board text removed: "GND"
- board text removed: "IO"
- board text removed: "RX"
- board text removed: "TX"
- board text removed: "UART1"
- board text removed: "UART2"
- board text removed: "НАВ"
- board text removed: "СТРОБ"
- board text removed: "Синхро"

Commit message: PCB work 4
Parts:
- removed C22, C23, C24, C25, C26: C, Capacitor_SMD:C_0805_2012Metric_Pad1.18x1.45mm_HandSolder
- removed L4, L5: SWPA4030S1R0NT, ul_VLS252012HBU-220M:IND_VLS252012_TDK
- removed R17, R18, R19, R20: R, Resistor_SMD:R_0402_1005Metric_Pad0.72x0.64mm_HandSolder
- added D22: WireHole_1p5, Wire_holes:WireHole_0p7, F.Cu at (86.5, 52.8)
- added D23: WireHole_1p5, Wire_holes:WireHole_0p7, F.Cu at (88.6, 63.8)
- added D24: WireHole_1p5, Wire_holes:WireHole_0p7, F.Cu at (88.0, 52.8)
- added D25: WireHole_1p5, Wire_holes:WireHole_0p7, F.Cu at (90.2, 63.8)
- added D26: WireHole_1p5, Wire_holes:WireHole_0p7, F.Cu at (89.5, 52.8)
- added D27: WireHole_1p5, Wire_holes:WireHole_0p7, F.Cu at (91.7, 63.8)
- C1: footprint Capacitor_SMD:C_0402_1005Metric_Pad0.74x0.62mm_HandSolder -> Capacitor_SMD:C_0805_2012Metric_Pad1.18x1.45mm_HandSolder
- C10, C14, C8: footprint Capacitor_SMD:C_0805_2012Metric_Pad1.18x1.45mm_HandSolder -> Capacitor_SMD:C_0603_1608Metric_Pad1.08x0.95mm_HandSolder
- C11, C17, C18, C20, C21, C3, C6, C9: footprint Capacitor_SMD:C_0805_2012Metric_Pad1.18x1.45mm_HandSolder -> Capacitor_SMD:C_0402_1005Metric_Pad0.74x0.62mm_HandSolder
- C13, C16, C7: footprint Capacitor_SMD:C_0603_1608Metric_Pad1.08x0.95mm_HandSolder -> Capacitor_SMD:C_0402_1005Metric_Pad0.74x0.62mm_HandSolder
- C4: footprint Capacitor_SMD:C_0603_1608Metric_Pad1.08x0.95mm_HandSolder -> Capacitor_SMD:C_0805_2012Metric_Pad1.18x1.45mm_HandSolder
- D10, D11, D12, D13, D14, D20, D21, D6, D7, D8, D9: footprint Wire_holes:WireHole_1p2 -> Wire_holes:WireHole_0p7
- D15, D16, D17, D18: footprint Wire_holes:WireHole_1p2 -> Wire_holes:WireHole_0p8
- D5: footprint Diode_SMD:D_SOD-523 -> Diode_SMD:D_SOD-923
- L1: value SWPA4030S1R0NT -> SWPA8040S220MT; footprint ul_VLS252012HBU-220M:IND_VLS252012_TDK -> SWPA8040:IND_SWPA8040S_SNL
- L2, L3: value SWPA4030S1R0NT -> SWPA3015S4R7MT; footprint ul_VLS252012HBU-220M:IND_VLS252012_TDK -> ul_SWPA3015S4R7MT:IND_SWPA3015S_SNL
- R1, R13: value BLM18KG102SH1D -> R; footprint ul_BLM18KG102SH1D:RES_0603_1P6XP8_MUR -> Resistor_SMD:R_0402_1005Metric_Pad0.72x0.64mm_HandSolder
- R16: footprint Resistor_SMD:R_0402_1005Metric_Pad0.72x0.64mm_HandSolder -> Resistor_SMD:R_0603_1608Metric_Pad0.98x0.95mm_HandSolder
- U5: value TLV9061IDCKR -> INA193; footprint ul_TLV9061IDCKR:DCK5_TEX -> Package_TO_SOT_SMD:SOT-23-5
- moved U4 79.8 mm to (82.0, 57.1)
- moved C20 78.6 mm to (100.4, 64.0), turned to 180 degrees
- moved LED1 78.0 mm to (104.8, 58.9), turned to 90 degrees
- moved L3 75.1 mm to (88.3, 55.2), turned to 180 degrees
- moved C1 75.0 mm to (58.4, 56.6), turned to -90 degrees
- moved R10 72.1 mm to (80.7, 61.9), turned to 180 degrees
- moved C15 68.7 mm to (95.8, 61.5), turned to -90 degrees
- moved L2 63.2 mm to (90.9, 59.3), turned to 180 degrees
- moved C16 62.9 mm to (86.0, 57.7)
- moved U2 62.5 mm to (98.8, 56.5)
- moved D4 62.5 mm to (65.4, 55.0), turned to 180 degrees
- moved C13 58.5 mm to (88.5, 61.9)
- moved R11 58.1 mm to (79.1, 57.2), turned to 90 degrees
- moved U3 54.8 mm to (84.5, 61.4)
- moved D7 52.6 mm to (98.0, 53.1)
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Connections:
- C1 pad 1: Net-(U2-PA4) -> Net-(D2-Conn)
- C10 pad 1: Net-(U3-VIN) -> Net-(D11-Conn)
- C12 pad 1: Net-(D16-Conn) -> Net-(U3-BST)
- C12 pad 2: GND2 -> Net-(C12-Pad2)
- C13 pad 1: Net-(U3-BST) -> Net-(U3-VCC)
- C13 pad 2: Net-(C13-Pad2) -> GND2
- C14 pad 1: Net-(U3-VCC) -> Net-(U4-BST)
- C14 pad 2: GND2 -> Net-(C14-Pad2)
- C15 pad 1: Net-(C15-Pad1) -> Net-(U5-+)
- C16 pad 1: Net-(U4-BST) -> Net-(U4-VCC)
- C16 pad 2: Net-(C16-Pad2) -> GND2
- C17 pad 1: Net-(C15-Pad1) -> Net-(U5-+)
- C18 pad 1: Net-(U4-VCC) -> Net-(C17-Pad2)
- C18 pad 2: GND2 -> Net-(U3-FB)
- C19 pad 1: Net-(C17-Pad2) -> Net-(D13-Conn)
- C19 pad 2: Net-(C19-Pad2) -> GND2
- C2 pad 1: Net-(D2-Conn) -> Net-(D3-Conn)
- C20 pad 1: Net-(D16-Conn) -> Net-(D13-Conn)
- C21 pad 1: Net-(D16-Conn) -> Net-(D13-Conn)
- C3 pad 1: Net-(D3-Conn) -> Net-(U2-PA5)
- C4 pad 1: Net-(U2-PF2) -> Net-(D4-K)
- C5 pad 1: Net-(D4-K) -> Net-(D11-Conn)
- C6 pad 1: Net-(U3-VIN) -> Net-(U2-PF2)
- C7 pad 1: Net-(D16-Conn) -> Net-(D13-Conn)
- C8 pad 1: Net-(U3-VIN) -> Net-(D11-Conn)
- D10 pad 1: Net-(D10-Conn) -> GND2
- D12 pad 1: GND2 -> Net-(D12-Conn)
- D14 pad 1: Net-(D14-Conn) -> GND2
- D17 pad 1: GND2 -> Net-(D16-Conn)
- D18 pad 1: Net-(D18-Conn) -> GND2
- D19 pad 1: Net-(D19-Conn) -> GND2
- D20 pad 1: Net-(D19-Conn) -> GND2
- D21 pad 1: Net-(D21-Conn) -> GND2
- L1 pad 1: Net-(U3-VIN) -> Net-(D11-Conn)
- L2 pad 1: Net-(C15-Pad1) -> Net-(U5-+)
- L2 pad 2: Net-(C13-Pad2) -> Net-(C12-Pad2)
- L3 pad 1: Net-(D16-Conn) -> Net-(D13-Conn)
- L3 pad 2: Net-(C16-Pad2) -> Net-(C14-Pad2)
- R1 pad 1: Net-(D1-Conn) -> Net-(D3-Conn)
- R1 pad 2: Net-(R1-Pad2) -> Net-(U2-PB5)
- R10 pad 1: Net-(LED1-Pad2) -> Net-(U3-RON)
- R10 pad 2: Net-(U2-PB0) -> Net-(D11-Conn)
- R11 pad 1: Net-(U3-RON) -> Net-(U4-RON)
- R11 pad 2: Net-(U3-VIN) -> Net-(D11-Conn)
- R12 pad 1: Net-(U4-RON) -> Net-(C17-Pad2)
- R12 pad 2: Net-(U3-VIN) -> Net-(C12-Pad2)
- R13 pad 1: Net-(D16-Conn) -> Net-(R13-Pad1)
- R13 pad 2: Net-(D13-Conn) -> Net-(U3-FB)
- R14 pad 1: Net-(C17-Pad2) -> Net-(U4-FB)
- R14 pad 2: Net-(C13-Pad2) -> Net-(D13-Conn)
- R15 pad 2: Net-(D21-Conn) -> Net-(U4-FB)
- R16 pad 1: Net-(U3-FB) -> Net-(D15-Conn)
- R16 pad 2: Net-(C19-Pad2) -> Net-(U5-+)
- R2 pad 1: Net-(D3-Conn) -> Net-(D2-Conn)
- R2 pad 2: Net-(U2-PB5) -> Net-(U2-PB4)
- R3 pad 1: Net-(D2-Conn) -> Net-(U2-PA5)
- R3 pad 2: Net-(U2-PB4) -> Net-(D1-Conn)
- R4 pad 1: Net-(U2-PA4) -> GND2
- R4 pad 2: Net-(R1-Pad2) -> Net-(D5-A)
- R5 pad 1: GND2 -> Net-(U2-PA1)
- R5 pad 2: Net-(D5-A) -> Net-(D13-Conn)
- R6 pad 1: Net-(U2-PA1) -> GND2
- R6 pad 2: Net-(D16-Conn) -> Net-(U2-PA1)
- R7 pad 1: GND2 -> Net-(U2-PA0)
- R7 pad 2: Net-(U2-PA1) -> Net-(D11-Conn)
- R8 pad 1: Net-(U2-PA0) -> GND2
- R8 pad 2: Net-(U3-VIN) -> Net-(U2-PA0)
- R9 pad 1: GND2 -> Net-(LED1-Pad2)
- R9 pad 2: Net-(U2-PA0) -> Net-(U2-PB0)
- U2 pad 10: Net-(U2-PA4) -> unconnected-(U2-PA4-Pad10)
- U2 pad 11: Net-(D15-Conn) -> Net-(U2-PA5)
- U2 pad 12: Net-(U2-PA6) -> unconnected-(U2-PA6-Pad12)
- U2 pad 20: Net-(D10-Conn) -> Net-(D8-Conn)
- U2 pad 21: Net-(D11-Conn) -> Net-(D9-Conn)
- U2 pad 22: unconnected-(U2-PA15-Pad22) -> Net-(D12-Conn)
- U2 pad 23: unconnected-(U2-PB3-Pad23) -> Net-(U2-PB3)
- U2 pad 26: Net-(D9-Conn) -> unconnected-(U2-PB6-Pad26)
- U2 pad 27: Net-(D8-Conn) -> unconnected-(U2-PB7-Pad27)
- U2 pad 3: Net-(D16-Conn) -> Net-(D13-Conn)
- U3 pad 11: Net-(C13-Pad2) -> Net-(C12-Pad2)
- U3 pad 12: Net-(C13-Pad2) -> Net-(C12-Pad2)
- U3 pad 3: Net-(U3-VIN) -> Net-(D11-Conn)
- U3 pad 4: Net-(U2-PA6) -> Net-(U2-PB3)
- U4 pad 11: Net-(C16-Pad2) -> Net-(C14-Pad2)
- U4 pad 12: Net-(C16-Pad2) -> Net-(C14-Pad2)
- U4 pad 3: Net-(U3-VIN) -> Net-(D11-Conn)
- U4 pad 4: Net-(U3-VIN) -> Net-(D11-Conn)
- U5 pad 1: Net-(D21-Conn) -> Net-(R13-Pad1)
- U5 pad 3: Net-(U5-IN-) -> Net-(U5-+)
- U5 pad 4: Net-(U3-FB) -> Net-(D15-Conn)
- U5 pad 5: Net-(D16-Conn) -> Net-(D13-Conn)
Routing:
- net Net-(D11-Conn): track 0.00 -> 19.8 mm
- net Net-(D4-K): track 0.00 -> 19.2 mm
- net Net-(U4-FB): track 0.00 -> 10.6 mm
- net Net-(R13-Pad1): track 0.00 -> 9.40 mm
- net Net-(C12-Pad2): track 0.00 -> 8.17 mm
- net Net-(U5-+): track 0.00 -> 8.00 mm
- net Net-(D2-Conn): track 0.00 -> 7.93 mm
- net Net-(D13-Conn): track 0.00 -> 7.86 mm
- net Net-(U3-FB): track 0.00 -> 7.74 mm
- net Net-(D3-Conn): track 0.00 -> 7.46 mm
- net Net-(U4-SS): track 0.00 -> 5.26 mm
- net Net-(C14-Pad2): track 0.00 -> 4.68 mm
- net Net-(D5-A): track 0.00 -> 3.43 mm
- net Net-(C17-Pad2): track 0.00 -> 2.57 mm
- net Net-(U3-BST): track 0.00 -> 1.84 mm
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
Commit message: PCB work 4
Parts:
- moved D17 50.8 mm to (105.0, 56.4)
- moved D18 50.7 mm to (105.0, 58.1)
- moved D16 29.5 mm to (58.6, 53.4)
- moved D15 27.2 mm to (60.4, 53.4)
- moved D10 5.93 mm to (98.0, 51.9), turned to 90 degrees
- moved LED1 4.89 mm to (102.5, 54.6), turned to -90 degrees
- moved D6 2.98 mm to (93.8, 51.8)
- moved D7 2.98 mm to (95.4, 51.8)
- moved D8 2.90 mm to (101.0, 51.9), turned to 90 degrees
- moved D9 2.84 mm to (99.5, 51.9), turned to 90 degrees
- moved C9 1.30 mm to (79.4, 63.1)
- moved R10 1.28 mm to (79.4, 62.0)
- moved R9 0.97 mm to (102.8, 56.7)
- moved D11 0.88 mm to (102.8, 58.4)
- moved D12 0.88 mm to (102.8, 59.9)
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Routing:
- net Net-(U2-PB5): track 0.00 -> 44.5 mm, vias 0 -> 2
- net Net-(D12-Conn): track 0.00 -> 37.6 mm, vias 0 -> 1
- net Net-(U2-PB3): track 0.00 -> 27.3 mm, vias 0 -> 3
- net Net-(U2-PA0): track 1.10 -> 17.4 mm, vias 0 -> 2
- net Net-(D6-Conn): track 0.00 -> 12.2 mm, vias 0 -> 1
- net Net-(D7-Conn): track 0.00 -> 11.7 mm, vias 0 -> 1
- net Net-(U2-PA1): track 1.60 -> 11.6 mm, vias 0 -> 2
- net Net-(D8-Conn): track 0.00 -> 4.64 mm
- net Net-(D9-Conn): track 0.00 -> 3.98 mm
- net Net-(D13-Conn): track 7.86 -> 11.4 mm
- net Net-(U2-PB0): track 0.00 -> 3.20 mm
- net Net-(LED1-Pad2): track 0.00 -> 1.91 mm
- net Net-(U3-RON): track 1.45 -> 3.18 mm
- net Net-(U2-PF2): track 0.00 -> 1.69 mm
- net Net-(U3-SS): track 1.49 -> 2.84 mm
Other:
- copper layers 2 -> 4

Commit message: PCB work 5
Parts:
- moved D21 4.78 mm to (91.9, 63.9), turned to 180 degrees
- moved D20 4.62 mm to (89.7, 52.0), turned to 180 degrees
- moved D26 4.52 mm to (85.1, 52.0), turned to 180 degrees
- moved D27 4.37 mm to (87.3, 63.9), turned to 180 degrees
- moved D23 1.73 mm to (90.4, 63.9), turned to 180 degrees
- moved D22 1.57 mm to (88.2, 52.0), turned to 180 degrees
- moved D24 1.47 mm to (86.7, 52.0), turned to 180 degrees
- moved D25 1.32 mm to (88.8, 63.9), turned to 180 degrees
- moved R1 0.91 mm to (59.0, 62.9)
- moved R9 0.83 mm to (102.0, 56.8), turned to -90 degrees
- moved C20 0.51 mm to (100.9, 64.0)
- moved R11 0.42 mm to (79.1, 57.6)
- moved LED1 0.08 mm to (102.5, 54.6)
Routing:
- net Net-(D15-Conn): track 1.74 -> 57.3 mm, vias 0 -> 1
- net Net-(U2-PA5): track 0.00 -> 54.4 mm, vias 0 -> 2
- net Net-(D16-Conn): track 0.00 -> 51.6 mm
- net Net-(D13-Conn): track 11.4 -> 58.2 mm
- net Net-(D11-Conn): track 19.4 -> 53.5 mm, vias 0 -> 1
- net Net-(D12-Conn): track 37.6 -> 45.8 mm
- net Net-(U2-PB3): track 27.3 -> 29.0 mm
- net Net-(D3-Conn): track 7.46 -> 8.78 mm
- net Net-(R13-Pad1): track 9.40 -> 10.4 mm
- net Net-(D7-Conn): track 11.7 -> 10.9 mm
- net Net-(U2-PB0): track 3.20 -> 2.44 mm
- net Net-(D6-Conn): track 12.2 -> 11.4 mm
- net Net-(U2-PB5): track 44.5 -> 45.1 mm
- net Net-(LED1-Pad2): track 1.91 -> 1.25 mm

Commit message: PCB work 6
Parts:
- moved D13 44.6 mm to (59.5, 52.3), turned to -90 degrees
- moved D14 42.7 mm to (61.1, 52.3), turned to -90 degrees
- moved D12 40.9 mm to (62.6, 52.3), turned to -90 degrees
- moved D11 39.2 mm to (64.1, 52.3), turned to -90 degrees
- moved D15 9.35 mm to (60.5, 62.8)
- moved D16 9.35 mm to (58.7, 62.8)
- moved R1 4.96 mm to (60.4, 58.2), turned to 90 degrees
- moved D17 1.50 mm to (103.6, 57.0)
- moved D18 1.50 mm to (103.6, 58.7)
- moved C1 0.65 mm to (58.4, 55.9)
- moved C2 0.65 mm to (58.4, 59.8)
- moved C3 0.65 mm to (55.9, 57.3)
- moved D1 0.65 mm to (55.3, 60.4)
- moved D19 0.65 mm to (55.3, 55.3)
- moved D2 0.65 mm to (60.4, 55.3)
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Routing:
- net Net-(U2-PB4): track 0.00 -> 40.4 mm, vias 0 -> 3
- net Net-(D13-Conn): track 58.2 -> 82.1 mm, vias 0 -> 1
- net Net-(D12-Conn): track 45.8 -> 66.8 mm
- net Net-(D15-Conn): track 57.3 -> 44.1 mm
- net Net-(D11-Conn): track 53.5 -> 62.5 mm
- net GND2: track 0.50 -> 3.96 mm, vias 0 -> 20
- net Net-(U2-PB5): track 45.1 -> 42.1 mm
- net Net-(D3-Conn): track 8.78 -> 10.8 mm
- net Net-(D1-Conn): track 0.00 -> 1.97 mm
- net Net-(U2-PA5): track 54.4 -> 53.1 mm
- net Net-(D16-Conn): track 51.6 -> 50.4 mm
- net Net-(D4-K): track 19.2 -> 18.6 mm
- net (no net): vias 0 -> 1

Commit message: PCB work 6
Parts:
- added D28: WireHole_1p5, Wire_holes:WireHole_2p0, F.Cu at (55.6, 52.3)
- added D29: WireHole_1p5, Wire_holes:WireHole_2p0, F.Cu at (55.6, 63.2)
- added D30: WireHole_1p5, Wire_holes:WireHole_2p0, F.Cu at (104.4, 52.6)
- added D31: WireHole_1p5, Wire_holes:WireHole_2p0, F.Cu at (104.4, 63.2)
- moved D13 1.52 mm to (61.1, 52.3)
- moved D14 1.50 mm to (59.6, 52.3)
- moved LED1 0.67 mm to (102.4, 55.3)
- moved R9 0.47 mm to (102.0, 57.2)
Connections:
- U3 pad V: (no net) -> GND2
- U4 pad V: (no net) -> GND2
Routing:
- net Net-(D13-Conn): track 82.1 -> 80.6 mm
- net Net-(D2-Conn): track 8.30 -> 7.44 mm
- net (no net): vias 1 -> 0
- added copper zone on B.Cu, net GND2
- added copper zone on F.Cu, net GND2
- added copper zone on In1.Cu, net GND2
- added copper zone on In2.Cu, net GND2
Other:
- board outline added: 52.4 x 14.4 mm
- board text added: "+Uф"
- board text added: "3В"
- board text added: "DIO"
- board text added: "En"
- board text added: "Rx"
- board text added: "Tx"
- board text added: "clk"
- board text added: "БXО"
- board text added: "СТР"
- board text added: "змл"
- board text added: "снхр"
