File: BANO_StepDown_LM5160_Control_Module/Main_PCB_002.kicad_sch (KiCad schematic)
At the start: 87 parts, among them Q1 BSS123, U1 INA193, U3 LM5164DDA, U4 SI7489DP-T1-E3, U5 SI7489DP-T1-E3, U6 STM32G031G8Ux, U7 SI7489DP-T1-E3, U8 LM5164DDA

Commit message: BANO MainModule Double Strob
Parts:
- removed C1: C, Capacitor_SMD:C_0805_2012Metric_Pad1.18x1.45mm_HandSolder, symbol Device:C
- removed C12, C7: C, Capacitor_SMD:C_0402_1005Metric_Pad0.74x0.62mm_HandSolder, symbol Device:C
- removed C4: C, Capacitor_SMD:C_0603_1608Metric_Pad1.08x0.95mm_HandSolder, symbol Device:C
- removed D14, D6: MM5Zxx, Diode_SMD:D_SOD-523, symbol Diode:MM5Zxx
- removed D20: BAT54C, Package_TO_SOT_SMD:SOT-23, symbol Diode:BAT54C
- removed D22, D23, D24, D25, D26, D27, D28, D29, D30, D4, D7: WireHole_1p5, Wire_holes:WireHole_1p2, symbol Connectors_for_Wire:WireHole_1p5
- removed LED1, LED2: HSMW-C191-U0000, ul_HSMW-C191-U0000:LED_91-U0000, symbol HSMW-C191:HSMW-C191-U0000
- removed Q1: BSS123, Package_TO_SOT_SMD:SOT-23, symbol Transistor_FET:BSS123
- removed R1: R, Resistor_SMD:R_0603_1608Metric_Pad0.98x0.95mm_HandSolder, symbol Device:R
- removed R10, R13, R22, R29, R30, R8: R, Resistor_SMD:R_0402_1005Metric_Pad0.72x0.64mm_HandSolder, symbol Device:R
- removed R15, R23, R24, R25, R26, R27, R28, R4, R5, R6, R9: BLM18KG102SH1D, ul_BLM18KG102SH1D:RES_0603_1P6XP8_MUR, symbol BLM18KG102SH1D:BLM18KG102SH1D
- removed U1: INA193, Package_TO_SOT_SMD:SOT-23-5, symbol Amplifier_Current:INA193
- removed U3, U8: LM5164DDA, Package_SO:HSOP-8-1EP_3.9x4.9mm_P1.27mm_EP2.41x3.1mm_ThermalVias, symbol Regulator_Switching:LM5164DDA
- removed U4, U5, U7: SI7489DP-T1-E3, ul_SI7852DP-T1:POWERPAK_SO-8_SINGLE_VIS, symbol SI7489DP:SI7489DP-T1-E3
- added C10, C11, C17, C18, C19, C20, C21, C22, C23, C24, C25, C26, C5, C6: C, Capacitor_SMD:C_0805_2012Metric_Pad1.18x1.45mm_HandSolder, symbol Device:C
- added C13, C16: C, Capacitor_SMD:C_0603_1608Metric_Pad1.08x0.95mm_HandSolder, symbol Device:C
- added D14, D20, D21: WireHole_1p5, Wire_holes:WireHole_1p2, symbol Connectors_for_Wire:WireHole_1p5
- added D4: 1N5711UR, Diode_SMD:D_MELF, symbol Diode:1N5711UR
- added L1, L4, L5: SWPA4030S1R0NT, ul_VLS252012HBU-220M:IND_VLS252012_TDK, symbol SWPA4030S1R0NT:SWPA4030S1R0NT
- added R15, R16, R17, R18, R19, R5: R, Resistor_SMD:R_0402_1005Metric_Pad0.72x0.64mm_HandSolder, symbol Device:R
- added U1: SI7489DP-T1-E3, ul_SI7852DP-T1:POWERPAK_SO-8_SINGLE_VIS, symbol SI7489DP:SI7489DP-T1-E3
- added U3, U4: LM5160ADNTR, ul_LM5160ADNTR:DNT0012B, symbol LM5160ADNTR:LM5160ADNTR
- added U5: TLV9061IDCKR, ul_TLV9061IDCKR:DCK5_TEX, symbol DCK5_TEX:TLV9061IDCKR
- C14, C8: footprint Capacitor_SMD:C_0603_1608Metric_Pad1.08x0.95mm_HandSolder -> Capacitor_SMD:C_0805_2012Metric_Pad1.18x1.45mm_HandSolder
- C9: footprint Capacitor_SMD:C_0805_2012Metric -> Capacitor_SMD:C_0805_2012Metric_Pad1.18x1.45mm_HandSolder
- renumbered C13 to C1, C11 to C4, C10 to C7, D13 to D1, D8 to D10, D9 to D11, D10 to D6, D11 to D7, D1 to D8, D21 to D9, LED3 to LED1, R7 to R1, R31 to R10, R21 to R4, R18 to R6, R19 to R7, R16 to R8, R17 to R9, U6 to U2
Connections:
- net GND2: now also C14.2, C8.2, D12.1 (Conn), LED1.1, C10.2, C11.2, C18.2, C20.2, C22.2, C23.2, C24.2, C25.2, C26.2, C5.2, C6.2, R15.1, R18.1, R5.1, U3.1 (AGND), U3.13 (PAD), U3.2 (PGND), U4.1 (AGND), U4.13 (PAD), U4.2 (PGND), U5.2 (V-); no longer D18.1 (Conn), R12.1
- net at D19.1 (Conn): now also D20.1 (Conn)
- net at R20.2: now also R19.1, U5.3 (IN-)
- net at R2.1: now also C3.1, D3.1 (Conn), U1.5 (D), U1.6 (D), U1.7 (D), U1.8 (D); no longer U2.24 (PB4)
- net at R2.2: now also U2.25 (PB5)
- net at R11.2: now also C8.1, R12.2, R8.2, C10.1, C22.1, C6.1, L1.1, L4.2, U3.3 (VIN), U4.3 (VIN), U4.4 (EN_UVLO); no longer R3.2
- net at D7.1 (Conn): now also U2.9 (PA3)
- net at C15.1: now also L2.1, C17.1, C25.1, L5.2; no longer L3.1
- net at C7.1, R6.2, U2.3 (VDD): now also D16.1 (Conn), L3.1, C20.1, C21.1, C24.1, R17.2, U5.5 (V+); no longer C9.1, L2.1, R14.2
- net at L3.2: now also C16.2, U4.11 (SW), U4.12 (SW); no longer C14.1
- net at C2.1: now also D2.1 (Conn), R3.1, D4.2 (A)
- net at R14.1: now also C17.2, C19.1
- net at L2.2: now also R14.2, C13.2, U3.11 (SW), U3.12 (SW); no longer C8.1
- net at U2.27 (PB7): now also D8.1 (Conn)
- net at D5.2 (A): now also R5.2, U1.4 (G)
- net at D5.1 (K): now also C5.1, D4.1 (K), L1.2, U1.1 (S), U1.2 (S), U1.3 (S)
- net at U2.20 (PA13): now also D10.1 (Conn)
- net at U2.11 (PA5): now also D15.1 (Conn)
- net at U2.12 (PA6): now also U3.4 (EN_UVLO)
- net at U2.21 (PA14): now also D11.1 (Conn)
- net at U2.26 (PB6): now also D9.1 (Conn)
- net at U2.8 (PA2): now also D6.1 (Conn)
- net at R11.1: now also U3.5 (RON)
- new net: R16.1, R19.2, U3.8 (FB), U5.4 (OUT)
- new net: R12.1, U4.5 (RON)
- new net: C19.2, R16.2
- new net: C21.2, R17.1, R18.2, U4.8 (FB)
- new net: C23.1, D14.1 (Conn), L4.1
- new net: R3.2, U2.24 (PB4)
- new net: D21.1 (Conn), R15.2, U5.1 (IN+)
- new net: C13.1, U3.10 (BST)
- new net: C26.1, D18.1 (Conn), L5.1
- new net: C16.1, U4.10 (BST)
- new net: C9.1, U3.6 (SS)
- new net: C14.1, U3.9 (VCC)
- new net: C18.1, U4.9 (VCC)
- new net: C11.1, U4.6 (SS)
Other:
- moved on the sheet: C1, C4, C7, D1, D10, D11, D6, D7, D8, D9, LED1, R1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

Commit message: BANO MainModule Double Strob
Parts:
- removed C22, C23, C25, C26: C, Capacitor_SMD:C_0805_2012Metric_Pad1.18x1.45mm_HandSolder, symbol Device:C
- removed D8, D9: WireHole_1p5, Wire_holes:WireHole_1p2, symbol Connectors_for_Wire:WireHole_1p5
- removed L4, L5: SWPA4030S1R0NT, ul_VLS252012HBU-220M:IND_VLS252012_TDK, symbol SWPA4030S1R0NT:SWPA4030S1R0NT
- removed R19, R20: R, Resistor_SMD:R_0402_1005Metric_Pad0.72x0.64mm_HandSolder, symbol Device:R
- removed U5: TLV9061IDCKR, ul_TLV9061IDCKR:DCK5_TEX, symbol DCK5_TEX:TLV9061IDCKR
- added R13: R, Resistor_SMD:R_0402_1005Metric_Pad0.72x0.64mm_HandSolder, symbol Device:R
- added U6: INA193, Package_TO_SOT_SMD:SOT-23-5, symbol Amplifier_Current:INA193
Connections:
- net GND2: now also U6.2 (GND)
- net at U3.8 (FB): now also C19.2, R16.2; no longer R16.1
- net at C10.1, C6.1, C8.1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: now also D14.1 (Conn)
- net at C15.1, C17.1, L2.1: now also R13.2, U6.3 (+)
- net at C20.1, C21.1, C24.1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: now also U6.5 (V+)
- net at C1.1, R4.1: now also U2.11 (PA5); no longer U2.10 (PA4)
- net at D15.1 (Conn): now also U2.22 (PA15); no longer U2.11 (PA5)
- net at U2.12 (PA6): no longer U3.4 (EN_UVLO)
- net at U2.23 (PB3): now also U3.4 (EN_UVLO)
- net at D18.1 (Conn): now also R13.1, U6.4 (-)
- new net: R16.1, U6.1
Other:
- moved on the sheet: C15, C17, C19, C24, D18, D19, D20, D21, L2, R14, R15, R16

Commit message: BANO MainModule Double Strob
Parts:
- removed R1: BLM18KG102SH1D, ul_BLM18KG102SH1D:RES_0603_1P6XP8_MUR, symbol BLM18KG102SH1D:BLM18KG102SH1D
- removed R15: R, Resistor_SMD:R_0402_1005Metric_Pad0.72x0.64mm_HandSolder, symbol Device:R
- renumbered C2 to C1, C13 to C12, C14 to C13, C16 to C14, C18 to C16, C19 to C18, C20 to C19, C3 to C2, C24 to C20, C1 to C3, C5 to C4, C6 to C5, C4 to C6, D12 to D10, D14 to D11, D15 to D12, D16 to D13, D17 to D14, D18 to D15, D19 to D16, D20 to D17, D21 to D18, D10 to D8, D11 to D9, R2 to R1, R11 to R10, R12 to R11, R14 to R12, R16 to R13, R17 to R14, R18 to R15, R13 to R16, R3 to R2, R4 to R3, R5 to R4, R6 to R5, R7 to R6, R8 to R7, R9 to R8, R10 to R9, U6 to U5
Connections:
- net GND2: now also D18.1 (Conn)
- net at D1.1 (Conn): now also R3.2
Other:
- moved on the sheet: C3, C4, C5, C6, C7, D1, L1, R3, R7, R8

Commit message: PCB work 3
Parts:
- removed L1, L2, L3: SWPA4030S1R0NT, ul_VLS252012HBU-220M:IND_VLS252012_TDK, symbol SWPA4030S1R0NT:SWPA4030S1R0NT
- added L1: SWPA8040S220MT, SWPA8040:IND_SWPA8040S_SNL, symbol SWPA8040:SWPA8040S220MT
- added L2, L3: SWPA3015S4R7MT, ul_SWPA3015S4R7MT:IND_SWPA3015S_SNL, symbol ul_SWPA3015S4R7MT:SWPA3015S4R7MT
Connections:
- net at C10.1, C5.1, C8.1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: now also L1.1
- net at C15.1, C17.1, R16.2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: now also L2.1
- net at C4.1, D4.1 (K), D5.1 (K)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: now also L1.2
- net at C19.1, C20.1, C21.1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: now also L3.1
- net at C12.2, R12.2, U3.11 (SW)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: now also L2.2
- net at C14.2, U4.11 (SW), U4.12 (SW): now also L3.2
Changed lines of the file:
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@@
+    )
+  )
+  (symbol (lib_id "ul_SWPA3015S4R7MT:SWPA3015S4R7MT") (at 445.77 240.03 0) (unit 1)
+    (in_bom yes) (on_board yes) (dnp no) (fields_autoplaced)
+    (property "Reference" "L2" (at 453.39 232.41 0)
+      (effects (font (size 1.524 1.524)))
+    )
+    (property "Value" "SWPA3015S4R7MT" (at 453.39 234.95 0)
+      (effects (font (size 1.524 1.524)))
+    )
+    (property "Footprint" "ul_SWPA3015S4R7MT:IND_SWPA3015S_SNL" (at 445.77 240.03 0)
+      (effects (font (size 1.27 1.27) italic) hide)
+    )
+    (property "Datasheet" "SWPA3015S4R7MT" (at 445.77 240.03 0)
+      (effects (font (size 1.27 1.27) italic) hide)
+    )
+    (pin "1")
+    (pin "2")
+    (instances
+      (project "Main_PCB_002"
+        (path "/68e09be7-3bbc-4443-a838-209ce20b2bef"
+          (reference "L2") (unit 1)
+        )
+      )
     )
   )
@@
     )
   )
-  (symbol (lib_id "SWPA4030S1R0NT:SWPA4030S1R0NT") (at 464.82 153.67 0) (unit 1)
-    (in_bom yes) (on_board yes) (dnp no)
-    (property "Reference" "L3" (at 469.9 148.59 0)
-      (effects (font (size 1.524 1.524)))
-    )
-    (property "Value" "SWPA4030S1R0NT" (at 482.6 149.86 0)
-      (effects (font (size 1.524 1.524)))
-    )
-    (property "Footprint" "ul_VLS252012HBU-220M:IND_VLS252012_TDK" (at 464.82 153.67 0)
-      (effects (font (size 1.27 1.27) italic) hide)
-    )
-    (property "Datasheet" "SWPA4030S1R0NT" (at 464.82 153.67 0)
-      (effects (font (size 1.27 1.27) italic) hide)
-    )
-    (pin "1")
-    (pin "2")
-    (instances
-      (project "Main_PCB_002"
-        (path "/68e09be7-3bbc-4443-a838-209ce20b2bef"
-          (reference "L3") (unit 1)
-        )
-      )
-    )
-  )
   (symbol (lib_id "Connectors_for_Wire:WireHole_1p5") (at 556.26 259.08 0) (unit 1)
     (in_bom yes) (on_board yes) (dnp no)
@@
     )
   )
-  (symbol (lib_id "SWPA4030S1R0NT:SWPA4030S1R0NT") (at 445.77 240.03 0) (unit 1)
-    (in_bom yes) (on_board yes) (dnp no)
-    (property "Reference" "L2" (at 448.31 233.68 0)
+  (symbol (lib_id "Device:R") (at 394.97 237.49 270) (unit 1)
+    (in_bom yes) (on_board yes) (dnp no)
+    (property "Reference" "R10" (at 393.7 242.57 0)
+      (effects (font (size 1.27 1.27)) (justify right))
+    )
+    (property "Value" "R" (at 396.24 241.3 0)
+      (effects (font (size 1.27 1.27)) (justify right))
+    )
+    (property "Footprint" "Resistor_SMD:R_0402_1005Metric_Pad0.72x0.64mm_HandSolder" (at 394.97 235.712 90)
+      (effects (font (size 1.27 1.27)) hide)
+    )
+    (property "Datasheet" "~" (at 394.97 237.49 0)
+      (effects (font (size 1.27 1.27)) hide)
+    )
+    (pin "1")
+    (pin "2")
+    (instances
+      (project "Main_PCB_002"
+        (path "/68e09be7-3bbc-4443-a838-209ce20b2bef"
+          (reference "R10") (unit 1)
+        )
+      )
+    )
+  )
+  (symbol (lib_id "ul_SWPA3015S4R7MT:SWPA3015S4R7MT") (at 464.82 153.67 0) (unit 1)
+    (in_bom yes) (on_board yes) (dnp no) (fields_autoplaced)
+    (property "Reference" "L3" (at 472.44 146.05 0)
       (effects (font (size 1.524 1.524)))
     )
-    (property "Value" "SWPA4030S1R0NT" (at 458.47 236.22 0)
+    (property "Value" "SWPA3015S4R7MT" (at 472.44 148.59 0)
       (effects (font (size 1.524 1.524)))
     )
-    (property "Footprint" "ul_VLS252012HBU-220M:IND_VLS252012_TDK" (at 445.77 240.03 0)
+    (property "Footprint" "ul_SWPA3015S4R7MT:IND_SWPA3015S_SNL" (at 464.82 153.67 0)
       (effects (font (size 1.27 1.27) italic) hide)
     )
-    (property "Datasheet" "SWPA4030S1R0NT" (at 445.77 240.03 0)
+    (property "Datasheet" "SWPA3015S4R7MT" (at 464.82 153.67 0)
       (effects (font (size 1.27 1.27) italic) hide)
     )
@@
       (project "Main_PCB_002"
         (path "/68e09be7-3bbc-4443-a838-209ce20b2bef"
-          (reference "L2") (unit 1)
-        )
-      )
-    )
-  )
-  (symbol (lib_id "Device:R") (at 394.97 237.49 270) (unit 1)
-    (in_bom yes) (on_board yes) (dnp no)
-    (property "Reference" "R10" (at 393.7 242.57 0)
-      (effects (font (size 1.27 1.27)) (justify right))
-    )
-    (property "Value" "R" (at 396.24 241.3 0)
-      (effects (font (size 1.27 1.27)) (justify right))
-    )
-    (property "Footprint" "Resistor_SMD:R_0402_1005Metric_Pad0.72x0.64mm_HandSolder" (at 394.97 235.712 90)
-      (effects (font (size 1.27 1.27)) hide)
-    )
-    (property "Datasheet" "~" (at 394.97 237.49 0)
-      (effects (font (size 1.27 1.27)) hide)
-    )
-    (pin "1")
-    (pin "2")
-    (instances
-      (project "Main_PCB_002"
-        (path "/68e09be7-3bbc-4443-a838-209ce20b2bef"
-          (reference "R10") (unit 1)
+          (reference "L3") (unit 1)
         )
       )
@@
     )
   )
-  (symbol (lib_id "Device:C") (at 302.26 350.52 0) (unit 1)
-    (in_bom yes) (on_board yes) (dnp no)
-    (property "Reference" "C6" (at 298.45 347.98 0)
-      (effects (font (size 1.27 1.27)) (justify left))
-    )
-    (property "Value" "C" (at 298.45 351.79 0)
-      (effects (font (size 1.27 1.27)) (justify left))
-    )
-    (property "Footprint" "Capacitor_SMD:C_0603_1608Metric_Pad1.08x0.95mm_HandSolder" (at 303.2252 354.33 0)
-      (effects (font (size 1.27 1.27)) hide)
-    )
-    (property "Datasheet" "~" (at 302.26 350.52 0)
-      (effects (font (size 1.27 1.27)) hide)
-    )
-    (pin "1")
-    (pin "2")
-    (instances
-      (project "Main_PCB_002"
-        (path "/68e09be7-3bbc-4443-a838-209ce20b2bef"
-          (reference "C6") (unit 1)
-        )
-      )
-    )
-  )
-  (symbol (lib_id "SWPA4030S1R0NT:SWPA4030S1R0NT") (at 284.48 143.51 0) (unit 1)
+  (symbol (lib_id "SWPA8040:SWPA8040S220MT") (at 284.48 143.51 0) (unit 1)
     (in_bom yes) (on_board yes) (dnp no) (fields_autoplaced)
     (property "Reference" "L1" (at 292.1 135.89 0)
       (effects (font (size 1.524 1.524)))
     )
-    (property "Value" "SWPA4030S1R0NT" (at 292.1 138.43 0)
+    (property "Value" "SWPA8040S220MT" (at 292.1 138.43 0)
       (effects (font (size 1.524 1.524)))
     )
-    (property "Footprint" "ul_VLS252012HBU-220M:IND_VLS252012_TDK" (at 284.48 143.51 0)
+    (property "Footprint" "SWPA8040:IND_SWPA8040S_SNL" (at 284.48 143.51 0)
       (effects (font (size 1.27 1.27) italic) hide)
     )
-    (property "Datasheet" "SWPA4030S1R0NT" (at 284.48 143.51 0)
+    (property "Datasheet" "SWPA8040S220MT" (at 284.48 143.51 0)
       (effects (font (size 1.27 1.27) italic) hide)
     )
@@
         )
       )
+    )
+  )
+  (symbol (lib_id "Device:C") (at 302.26 350.52 0) (unit 1)
+    (in_bom yes) (on_board yes) (dnp no)
+    (property "Reference" "C6" (at 298.45 347.98 0)
+      (effects (font (size 1.27 1.27)) (justify left))
+    )
+    (property "Value" "C" (at 298.45 351.79 0)
+      (effects (font (size 1.27 1.27)) (justify left))
+    )
+    (property "Footprint" "Capacitor_SMD:C_0603_1608Metric_Pad1.08x0.95mm_HandSolder" (at 303.2252 354.33 0)
+      (effects (font (size 1.27 1.27)) hide)
+    )
+    (property "Datasheet" "~" (at 302.26 350.52 0)
+      (effects (font (size 1.27 1.27)) hide)
+    )
+    (pin "1")
+    (pin "2")
+    (instances
+      (project "Main_PCB_002"
+        (path "/68e09be7-3bbc-4443-a838-209ce20b2bef"
+          (reference "C6") (unit 1)
+        )
+      )

Commit message: PCB work 3
Parts:
- C10, C8: footprint Capacitor_SMD:C_0805_2012Metric_Pad1.18x1.45mm_HandSolder -> Capacitor_SMD:C_0603_1608Metric_Pad1.08x0.95mm_HandSolder
- C11, C13, C16, C17, C18, C20, C21, C9: footprint Capacitor_SMD:C_0805_2012Metric_Pad1.18x1.45mm_HandSolder -> Capacitor_SMD:C_0402_1005Metric_Pad0.74x0.62mm_HandSolder
- C6, C7: footprint Capacitor_SMD:C_0603_1608Metric_Pad1.08x0.95mm_HandSolder -> Capacitor_SMD:C_0402_1005Metric_Pad0.74x0.62mm_HandSolder
- R16: footprint Resistor_SMD:R_0402_1005Metric_Pad0.72x0.64mm_HandSolder -> Resistor_SMD:R_0603_1608Metric_Pad0.98x0.95mm_HandSolder
Other:
- moved on the sheet: C10, C11, C14, C16, C19, C21, D12, D13, D14, L3, R11, R14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

Commit message: PCB work 4
Parts:
- added D19: WireHole_1p5, Wire_holes:WireHole_1p2, symbol Connectors_for_Wire:WireHole_1p5
- added D20, D21, D22, D23, D24, D25, D26, D27: WireHole_1p5, Wire_holes:WireHole_0p7, symbol Connectors_for_Wire:WireHole_1p5
- D10, D11, D12, D13, D14, D6, D7, D8, D9: footprint Wire_holes:WireHole_1p2 -> Wire_holes:WireHole_0p7
- D15, D16, D17, D18: footprint Wire_holes:WireHole_1p2 -> Wire_holes:WireHole_0p8
- D5: footprint Diode_SMD:D_SOD-523 -> Diode_SMD:D_SOD-923
Connections:
- net GND2: now also D19.1 (Conn), D20.1 (Conn), D21.1 (Conn)
- net at C10.1, C5.1, C8.1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: now also D26.1 (Conn), D27.1 (Conn)
- net at C19.1, C20.1, C21.1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: now also D22.1 (Conn), D23.1 (Conn)
- net at D12.1 (Conn), U2.22 (PA15): now also D24.1 (Conn), D25.1 (Conn)
Other:
- moved on the sheet: D11, D12, D13, D14

Commit message: PCB work 6
Parts:
- added D28, D29, D30, D31: WireHole_1p5, Wire_holes:WireHole_2p0, symbol Connectors_for_Wire:WireHole_1p5
Connections:
- net GND2: now also D28.1 (Conn), D29.1 (Conn), D30.1 (Conn), D31.1 (Conn)
Changed lines of the file:
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@@
   (junction (at 492.76 248.92) (diameter 0) (color 0 0 0 0)
   )
+  (junction (at 553.72 173.99) (diameter 0) (color 0 0 0 0)
+  )
   (junction (at 411.48 157.48) (diameter 0) (color 0 0 0 0)
   )
   (junction (at 300.99 144.78) (diameter 0) (color 0 0 0 0)
   )
+  (junction (at 553.72 176.53) (diameter 0) (color 0 0 0 0)
+  )
   (junction (at 491.49 172.72) (diameter 0) (color 0 0 0 0)
   )
@@
   (junction (at 387.35 144.78) (diameter 0) (color 0 0 0 0)
   )
+  (junction (at 553.72 179.07) (diameter 0) (color 0 0 0 0)
+  )
   (junction (at 234.95 160.02) (diameter 0) (color 0 0 0 0)
   )
@@
     (stroke (width 0) (type default))
   )
+  (wire (pts (xy 556.26 171.45) (xy 553.72 171.45))
+    (stroke (width 0) (type default))
+  )
   (wire (pts (xy 491.49 160.02) (xy 491.49 154.94))
     (stroke (width 0) (type default))
@@
     (stroke (width 0) (type default))
   )
+  (wire (pts (xy 553.72 179.07) (xy 553.72 181.61))
+    (stroke (width 0) (type default))
+  )
+  (wire (pts (xy 553.72 176.53) (xy 553.72 179.07))
+    (stroke (width 0) (type default))
+  )
   (wire (pts (xy 471.17 240.03) (xy 471.17 242.57))
     (stroke (width 0) (type default))
@@
     (stroke (width 0) (type default))
   )
+  (wire (pts (xy 556.26 179.07) (xy 553.72 179.07))
+    (stroke (width 0) (type default))
+  )
   (wire (pts (xy 441.96 252.73) (xy 448.31 252.73))
     (stroke (width 0) (type default))
@@
     (stroke (width 0) (type default))
   )
+  (wire (pts (xy 556.26 176.53) (xy 553.72 176.53))
+    (stroke (width 0) (type default))
+  )
   (wire (pts (xy 457.2 144.78) (xy 462.28 144.78))
     (stroke (width 0) (type default))
@@
     (stroke (width 0) (type default))
   )
+  (wire (pts (xy 556.26 173.99) (xy 553.72 173.99))
+    (stroke (width 0) (type default))
+  )
   (wire (pts (xy 411.48 149.86) (xy 411.48 157.48))
     (stroke (width 0) (type default))
@@
     (stroke (width 0) (type default))
   )
+  (wire (pts (xy 553.72 171.45) (xy 553.72 173.99))
+    (stroke (width 0) (type default))
+  )
   (wire (pts (xy 504.19 259.08) (xy 504.19 260.35))
     (stroke (width 0) (type default))
@@
   )
   (wire (pts (xy 471.17 250.19) (xy 471.17 252.73))
+    (stroke (width 0) (type default))
+  )
+  (wire (pts (xy 553.72 173.99) (xy 553.72 176.53))
     (stroke (width 0) (type default))
   )
@@
     )
   )
+  (symbol (lib_id "Connectors_for_Wire:WireHole_1p5") (at 556.26 179.07 0) (unit 1)
+    (in_bom yes) (on_board yes) (dnp no)
+    (property "Reference" "D30" (at 558.8 181.61 0)
+      (effects (font (size 1.27 1.27)) (justify left))
+    )
+    (property "Value" "WireHole_1p5" (at 561.34 176.53 0)
+      (effects (font (size 1.27 1.27)) (justify left))
+    )
+    (property "Footprint" "Wire_holes:WireHole_2p0" (at 556.26 180.34 0)
+      (effects (font (size 1.27 1.27)) hide)
+    )
+    (property "Datasheet" "" (at 556.26 180.34 0)
+      (effects (font (size 1.27 1.27)) hide)
+    )
+    (pin "1")
+    (instances
+      (project "Main_PCB_002"
+        (path "/68e09be7-3bbc-4443-a838-209ce20b2bef"
+          (reference "D30") (unit 1)
+        )
+      )
+    )
+  )
   (symbol (lib_id "Connectors_for_Wire:WireHole_1p5") (at 554.99 140.97 0) (unit 1)
     (in_bom yes) (on_board yes) (dnp no)
@@
         (path "/68e09be7-3bbc-4443-a838-209ce20b2bef"
           (reference "#PWR016") (unit 1)
+        )
+      )
+    )
+  )
+  (symbol (lib_id "Connectors_for_Wire:WireHole_1p5") (at 556.26 176.53 0) (unit 1)
+    (in_bom yes) (on_board yes) (dnp no)
+    (property "Reference" "D29" (at 558.8 179.07 0)
+      (effects (font (size 1.27 1.27)) (justify left))
+    )
+    (property "Value" "WireHole_1p5" (at 561.34 173.99 0)
+      (effects (font (size 1.27 1.27)) (justify left))
+    )
+    (property "Footprint" "Wire_holes:WireHole_2p0" (at 556.26 177.8 0)
+      (effects (font (size 1.27 1.27)) hide)
+    )
+    (property "Datasheet" "" (at 556.26 177.8 0)
+      (effects (font (size 1.27 1.27)) hide)
+    )
+    (pin "1")
+    (instances
+      (project "Main_PCB_002"
+        (path "/68e09be7-3bbc-4443-a838-209ce20b2bef"
+          (reference "D29") (unit 1)
         )
       )
@@
     )
   )
+  (symbol (lib_id "power:GND2") (at 553.72 181.61 0) (unit 1)
+    (in_bom yes) (on_board yes) (dnp no) (fields_autoplaced)
+    (property "Reference" "#PWR030" (at 553.72 187.96 0)
+      (effects (font (size 1.27 1.27)) hide)
+    )
+    (property "Value" "GND2" (at 553.72 186.69 0)
+      (effects (font (size 1.27 1.27)))
+    )
+    (property "Footprint" "" (at 553.72 181.61 0)
+      (effects (font (size 1.27 1.27)) hide)
+    )
+    (property "Datasheet" "" (at 553.72 181.61 0)
+      (effects (font (size 1.27 1.27)) hide)
+    )
+    (pin "1")
+    (instances
+      (project "Main_PCB_002"
+        (path "/68e09be7-3bbc-4443-a838-209ce20b2bef"
+          (reference "#PWR030") (unit 1)
+        )
+      )
+    )
+  )
   (symbol (lib_id "Device:C") (at 229.87 166.37 0) (unit 1)
     (in_bom yes) (on_board yes) (dnp no)
@@
         )
       )
+    )
+  )
+  (symbol (lib_id "Connectors_for_Wire:WireHole_1p5") (at 556.26 171.45 0) (unit 1)
+    (in_bom yes) (on_board yes) (dnp no)
+    (property "Reference" "D31" (at 558.8 173.99 0)
+      (effects (font (size 1.27 1.27)) (justify left))
+    )
+    (property "Value" "WireHole_1p5" (at 561.34 168.91 0)
+      (effects (font (size 1.27 1.27)) (justify left))
+    )
+    (property "Footprint" "Wire_holes:WireHole_2p0" (at 556.26 172.72 0)
+      (effects (font (size 1.27 1.27)) hide)
+    )
+    (property "Datasheet" "" (at 556.26 172.72 0)
+      (effects (font (size 1.27 1.27)) hide)
+    )
+    (pin "1")
+    (instances
+      (project "Main_PCB_002"
+        (path "/68e09be7-3bbc-4443-a838-209ce20b2bef"
+          (reference "D31") (unit 1)
+        )
+      )
+    )
+  )
+  (symbol (lib_id "Connectors_for_Wire:WireHole_1p5") (at 556.26 173.99 0) (unit 1)
+    (in_bom yes) (on_board yes) (dnp no)
+    (property "Reference" "D28" (at 558.8 176.53 0)
+      (effects (font (size 1.27 1.27)) (justify left))
+    )
+    (property "Value" "WireHole_1p5" (at 561.34 171.45 0)
+      (effects (font (size 1.27 1.27)) (justify left))
+    )
+    (property "Footprint" "Wire_holes:WireHole_2p0" (at 556.26 175.26 0)
+      (effects (font (size 1.27 1.27)) hide)
+    )
+    (property "Datasheet" "" (at 556.26 175.26 0)
+      (effects (font (size 1.27 1.27)) hide)
+    )
+    (pin "1")
+    (instances
+      (project "Main_PCB_002"
+        (path "/68e09be7-3bbc-4443-a838-209ce20b2bef"
+          (reference "D28") (unit 1)
+        )
+      )
