File: BANO_StepDown_LM5160_Total_Duplicate/BANO_StepDown_LM5160_Total_Duplicate.kicad_pcb (KiCad board)
At the start: 2 copper layers, 55 x 10 mm, 48 parts, among them U1 LM5160ADNTR, U2 TLV9061IDCKR, U3 LM5160ADNTR, U4 TLV9061IDCKR

Commit message: BANO Step-Dn 004 Double DC 002
Parts:
- D10, D11, D9: moved to B.Cu
- D2, D27, D28, D3: footprint Wire_holes:WireHole_1p2 -> Wire_holes:WireHole_0p8
- L2, L3: footprint ul_SWPA4030S1R0NT:IND_SWPA4030S_SNL -> ul_SWPA3015S4R7MT:IND_SWPA3015S_SNL
- R5, R9: footprint Resistor_SMD:R_0603_1608Metric_Pad0.98x0.95mm_HandSolder -> Resistor_SMD:R_0402_1005Metric_Pad0.72x0.64mm_HandSolder
- moved D10 5.79 mm to (87.8, 103.7), turned to 180 degrees
- moved D11 5.79 mm to (87.8, 110.2), turned to 180 degrees
- moved D9 5.79 mm to (87.8, 97.3), turned to 180 degrees
- moved R9 1.59 mm to (122.4, 123.9), turned to 0 degrees
- moved L2 1.59 mm to (122.0, 121.5)
- moved C8 0.88 mm to (103.3, 121.8)
- moved C10 0.88 mm to (100.4, 120.2)
- moved C12 0.88 mm to (102.9, 120.2)
- moved C13 0.88 mm to (92.7, 124.4)
- moved C7 0.88 mm to (110.2, 120.0)
- moved R10 0.88 mm to (96.3, 120.6)
- moved R11 0.88 mm to (96.3, 122.8)
- moved R7 0.88 mm to (98.1, 120.2)
- moved R8 0.88 mm to (94.0, 120.2)
- moved R6 0.88 mm to (102.3, 121.8)
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Routing:
- net Net-(D2-Conn): track 25.8 -> 8.64 mm, vias 0 -> 3
- net Net-(U1-RON): track 1.61 -> 7.49 mm
- net Net-(D27-Conn): track 5.79 -> 0.43 mm
- net Net-(D3-Conn): track 57.5 -> 55.0 mm
- net Net-(U1-VIN): track 2.06 -> 3.72 mm
Other:
- copper layers 2 -> 4

Commit message: PCB work
Parts:
- added ?: , , F.Cu at (118.6, 128.3)
- moved L3 0.67 mm to (112.0, 123.8)
- moved R9 0.59 mm to (123.0, 123.9)
- moved C26 0.38 mm to (123.8, 124.8)
- moved D2 0.21 mm to (116.9, 124.8)
- moved D27 0.11 mm to (116.9, 123.3)
- moved D3 0.11 mm to (116.9, 120.5)
- moved C27 0.06 mm to (130.8, 121.3)
- moved D28 0.05 mm to (116.9, 121.9)
Routing:
- net Net-(U1-VIN): track 3.72 -> 8.32 mm
- net Net-(U2-OUT): track 8.07 -> 12.2 mm, vias 0 -> 2
- net GND2: track 2.27 -> 6.12 mm
- net Net-(C27-Pad2): track 7.40 -> 8.97 mm
- net Net-(D8-K): track 3.97 -> 2.42 mm, vias 1 -> 2
- net Net-(D2-Conn): track 8.64 -> 8.07 mm
- net Net-(U1-FB): vias 0 -> 1
- net Net-(D3-Conn): vias 0 -> 2
- net (no net): vias 0 -> 2

Commit message: PCB work 2
Parts:
- removed D2: WireHole_1p5, Wire_holes:WireHole_0p8
- added C18: C, Capacitor_SMD:C_0805_2012Metric_Pad1.18x1.45mm_HandSolder, B.Cu at (135.7, 122.8)
- added C19: C, Capacitor_SMD:C_0805_2012Metric_Pad1.18x1.45mm_HandSolder, B.Cu at (93.7, 123.6)
- R5, R9: footprint Resistor_SMD:R_0402_1005Metric_Pad0.72x0.64mm_HandSolder -> Resistor_SMD:R_0603_1608Metric_Pad0.98x0.95mm_HandSolder
- moved D9 34.1 mm to (110.4, 122.8), turned to 0 degrees
- moved D10 25.5 mm to (104.6, 122.8), turned to 0 degrees
- moved D8 17.5 mm to (129.7, 122.7)
- moved D11 16.8 mm to (98.9, 122.8), turned to 0 degrees
- moved D7 16.8 mm to (124.1, 122.7)
- moved D6 16.4 mm to (118.4, 122.7)
- moved ? 5.52 mm to (114.1, 125.1)
- moved C26 4.14 mm to (119.7, 125.0)
- moved C1 3.74 mm to (137.2, 120.8)
- moved R3 3.41 mm to (133.8, 124.4)
- moved L1 3.39 mm to (130.9, 122.4)
- moved C5 3.39 mm to (123.8, 121.0)
- moved C4 3.38 mm to (129.9, 125.1)
- moved U2 3.38 mm to (136.3, 122.8)
- moved C6 3.38 mm to (127.7, 125.1)
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Routing:
- net Net-(D9-A): track 0.00 -> 24.8 mm, vias 0 -> 2
- net Net-(D6-A): track 7.11 -> 25.7 mm, vias 1 -> 2
- net Net-(D2-Conn): track 8.07 -> 18.7 mm, vias 3 -> 2
- net Net-(U3-VIN): track 0.00 -> 9.40 mm
- net Net-(D27-Conn): track 0.43 -> 8.74 mm
- net Net-(U3-FB): track 0.00 -> 7.58 mm, vias 0 -> 2
- net Net-(U2-OUT): track 12.2 -> 5.21 mm
- net Net-(D11-K): track 0.00 -> 6.80 mm, vias 0 -> 2
- net Net-(C9-Pad2): track 0.00 -> 6.30 mm
- net Net-(U1-RON): track 7.24 -> 1.96 mm
- net Net-(D8-K): track 2.42 -> 7.57 mm
- net Net-(U4-OUT): track 0.00 -> 5.06 mm, vias 0 -> 2
- net Net-(D3-Conn): track 55.0 -> 51.4 mm
- net Net-(U4-IN-): track 0.00 -> 2.80 mm
- net Net-(C10-Pad2): track 0.00 -> 2.34 mm
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
Commit message: BANO MainModule Double Strob
Parts:
- moved R5 0.32 mm to (109.2, 121.4)
- moved R9 0.28 mm to (119.4, 124.0)
Routing:
- net Net-(U1-VIN): track 7.56 -> 8.90 mm

Commit message: PCB work 6
Parts:
- C11, C28: footprint Capacitor_SMD:C_0603_1608Metric_Pad1.08x0.95mm_HandSolder -> Capacitor_SMD:C_0402_1005Metric_Pad0.74x0.62mm_HandSolder
- moved L4 0.22 mm to (97.5, 123.2)
- moved C19 0.08 mm to (93.8, 123.6)
- moved R7 0.06 mm to (96.0, 120.3)
Connections:
- U1 pad V: (no net) -> GND2
- U3 pad V: (no net) -> GND2
Routing:
- net Net-(D11-K): track 6.80 -> 2.27 mm
- net Net-(D9-A): track 24.8 -> 28.4 mm
- net Net-(D3-Conn): track 51.4 -> 53.2 mm
- net Net-(U3-FB): track 7.58 -> 8.55 mm
- added copper zone on B.Cu, net GND2
- added copper zone on F.Cu, net GND2
- added copper zone on In1.Cu, net GND2
- added copper zone on In2.Cu, net GND2
Other:
- board text added: "3.3"
- board text added: "En"
