File: BANO_StepDown_LM5160_Total_Duplicate/BANO_StepDown_LM5160_Total_Duplicate.kicad_sch (KiCad schematic)
At the start: 48 parts, among them U1 LM5160ADNTR, U2 TLV9061IDCKR, U3 LM5160ADNTR, U4 TLV9061IDCKR

Commit message: BANO Step-Dn 004 Double DC 002
Parts:
- D2, D27, D28, D3: footprint Wire_holes:WireHole_1p2 -> Wire_holes:WireHole_0p8
- L2, L3: footprint ul_SWPA4030S1R0NT:IND_SWPA4030S_SNL -> ul_SWPA3015S4R7MT:IND_SWPA3015S_SNL
- R5, R9: footprint Resistor_SMD:R_0603_1608Metric_Pad0.98x0.95mm_HandSolder -> Resistor_SMD:R_0402_1005Metric_Pad0.72x0.64mm_HandSolder
Changed lines of the file:
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@@
       (effects (font (size 1.524 1.524)))
     )
-    (property "Footprint" "ul_SWPA4030S1R0NT:IND_SWPA4030S_SNL" (at 246.38 92.71 0)
+    (property "Footprint" "ul_SWPA3015S4R7MT:IND_SWPA3015S_SNL" (at 246.38 92.71 0)
       (effects (font (size 1.27 1.27) italic) hide)
     )
@@
       (effects (font (size 1.27 1.27)) (justify left))
     )
-    (property "Footprint" "Wire_holes:WireHole_1p2" (at 222.25 100.33 0)
+    (property "Footprint" "Wire_holes:WireHole_0p8" (at 222.25 100.33 0)
       (effects (font (size 1.27 1.27)) hide)
     )
@@
       (effects (font (size 1.27 1.27)) (justify left))
     )
-    (property "Footprint" "Wire_holes:WireHole_1p2" (at 222.25 116.84 0)
+    (property "Footprint" "Wire_holes:WireHole_0p8" (at 222.25 116.84 0)
       (effects (font (size 1.27 1.27)) hide)
     )
@@
       (effects (font (size 1.27 1.27)) (justify left))
     )
-    (property "Footprint" "Wire_holes:WireHole_1p2" (at 218.44 177.8 0)
+    (property "Footprint" "Wire_holes:WireHole_0p8" (at 218.44 177.8 0)
       (effects (font (size 1.27 1.27)) hide)
     )
@@
       (effects (font (size 1.27 1.27)))
     )
-    (property "Footprint" "Resistor_SMD:R_0603_1608Metric_Pad0.98x0.95mm_HandSolder" (at 279.4 211.328 90)
+    (property "Footprint" "Resistor_SMD:R_0402_1005Metric_Pad0.72x0.64mm_HandSolder" (at 279.4 211.328 90)
       (effects (font (size 1.27 1.27)) hide)
     )
@@
       (effects (font (size 1.524 1.524)))
     )
-    (property "Footprint" "ul_SWPA4030S1R0NT:IND_SWPA4030S_SNL" (at 246.38 204.47 0)
+    (property "Footprint" "ul_SWPA3015S4R7MT:IND_SWPA3015S_SNL" (at 246.38 204.47 0)
       (effects (font (size 1.27 1.27) italic) hide)
     )
@@
       (effects (font (size 1.27 1.27)) (justify left))
     )
-    (property "Footprint" "Wire_holes:WireHole_1p2" (at 222.25 91.44 0)
+    (property "Footprint" "Wire_holes:WireHole_0p8" (at 222.25 91.44 0)
       (effects (font (size 1.27 1.27)) hide)
     )
@@
       (effects (font (size 1.27 1.27)))
     )
-    (property "Footprint" "Resistor_SMD:R_0603_1608Metric_Pad0.98x0.95mm_HandSolder" (at 279.4 99.568 90)
-      (effects (font (size 1.27 1.27)) hide)
-    )
+    (property "Footprint" "Resistor_SMD:R_0402_1005Metric_Pad0.72x0.64mm_HandSolder" (at 279.4 99.568 90)
+      (effects (font (size 1.27 1.27)) hide)
+    )

Commit message: PCB work 2
Parts:
- added C18, C19: C, Capacitor_SMD:C_0805_2012Metric_Pad1.18x1.45mm_HandSolder, symbol Device:C
- D2: footprint Wire_holes:WireHole_0p8 -> Connector_Pin:Pin_D0.7mm_L6.5mm_W1.8mm_FlatFork
- D27, D28, D3: footprint Wire_holes:WireHole_0p8 -> Wire_holes:WireHole_1p2
- L2, L3: footprint ul_SWPA3015S4R7MT:IND_SWPA3015S_SNL -> ul_SWPA4030S1R0NT:IND_SWPA4030S_SNL
- R5, R9: footprint Resistor_SMD:R_0402_1005Metric_Pad0.72x0.64mm_HandSolder -> Resistor_SMD:R_0603_1608Metric_Pad0.98x0.95mm_HandSolder
Connections:
- net GND2: now also C18.2, C19.2
- net at C28.1, C4.1, D6.2 (A)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: now also C18.1
- net at C10.1, C11.1, D9.2 (A)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: now also C19.1
Changed lines of the file:
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@@
   (junction (at 412.75 132.08) (diameter 0) (color 0 0 0 0)
   )
+  (junction (at 461.01 85.09) (diameter 0) (color 0 0 0 0)
+  )
   (junction (at 238.76 92.71) (diameter 0) (color 0 0 0 0)
   )
@@
   (junction (at 459.74 280.67) (diameter 0) (color 0 0 0 0)
   )
+  (junction (at 459.74 196.85) (diameter 0) (color 0 0 0 0)
+  )
   (junction (at 518.16 144.78) (diameter 0) (color 0 0 0 0)
   )
@@
     (stroke (width 0) (type default))
   )
+  (wire (pts (xy 459.74 204.47) (xy 459.74 205.74))
+    (stroke (width 0) (type default))
+  )
   (wire (pts (xy 270.51 97.79) (xy 270.51 92.71))
     (stroke (width 0) (type default))
@@
     (stroke (width 0) (type default))
   )
+  (wire (pts (xy 461.01 85.09) (xy 449.58 85.09))
+    (stroke (width 0) (type default))
+  )
   (wire (pts (xy 222.25 101.6) (xy 224.79 101.6))
     (stroke (width 0) (type default))
@@
     (stroke (width 0) (type default))
   )
-  (wire (pts (xy 504.19 85.09) (xy 449.58 85.09))
+  (wire (pts (xy 504.19 85.09) (xy 461.01 85.09))
     (stroke (width 0) (type default))
   )
@@
     (stroke (width 0) (type default))
   )
-  (wire (pts (xy 504.19 196.85) (xy 449.58 196.85))
+  (wire (pts (xy 504.19 196.85) (xy 459.74 196.85))
     (stroke (width 0) (type default))
   )
@@
     (stroke (width 0) (type default))
   )
-  (wire (pts (xy 246.38 92.71) (xy 238.76 92.71))
-    (stroke (width 0) (type default))
-  )
   (wire (pts (xy 354.33 100.33) (xy 360.68 100.33))
     (stroke (width 0) (type default))
@@
     (stroke (width 0) (type default))
   )
+  (wire (pts (xy 459.74 196.85) (xy 449.58 196.85))
+    (stroke (width 0) (type default))
+  )
   (wire (pts (xy 506.73 243.84) (xy 506.73 259.08))
     (stroke (width 0) (type default))
@@
     (stroke (width 0) (type default))
   )
+  (wire (pts (xy 238.76 92.71) (xy 246.38 92.71))
+    (stroke (width 0) (type default))
+  )
   (wire (pts (xy 393.7 243.84) (xy 412.75 243.84))
     (stroke (width 0) (type default))
@@
     (stroke (width 0) (type default))
   )
+  (wire (pts (xy 461.01 92.71) (xy 461.01 93.98))
+    (stroke (width 0) (type default))
+  )
   (symbol (lib_id "Device:C") (at 378.46 124.46 0) (unit 1)
     (in_bom yes) (on_board yes) (dnp no) (fields_autoplaced)
@@
         (path "/68e09be7-3bbc-4443-a838-209ce20b2bef"
           (reference "C4") (unit 1)
+        )
+      )
+    )
+  )
+  (symbol (lib_id "power:GND2") (at 459.74 205.74 0) (unit 1)
+    (in_bom yes) (on_board yes) (dnp no) (fields_autoplaced)
+    (property "Reference" "#PWR023" (at 459.74 212.09 0)
+      (effects (font (size 1.27 1.27)) hide)
+    )
+    (property "Value" "GND2" (at 459.74 210.82 0)
+      (effects (font (size 1.27 1.27)))
+    )
+    (property "Footprint" "" (at 459.74 205.74 0)
+      (effects (font (size 1.27 1.27)) hide)
+    )
+    (property "Datasheet" "" (at 459.74 205.74 0)
+      (effects (font (size 1.27 1.27)) hide)
+    )
+    (pin "1")
+    (instances
+      (project "BANO_StepDown_LM5160_Total_Duplicate"
+        (path "/68e09be7-3bbc-4443-a838-209ce20b2bef"
+          (reference "#PWR023") (unit 1)
         )
       )
@@
         (path "/68e09be7-3bbc-4443-a838-209ce20b2bef"
           (reference "D6") (unit 1)
+        )
+      )
+    )
+  )
+  (symbol (lib_id "Device:C") (at 461.01 88.9 0) (unit 1)
+    (in_bom yes) (on_board yes) (dnp no) (fields_autoplaced)
+    (property "Reference" "C18" (at 464.82 87.63 0)
+      (effects (font (size 1.27 1.27)) (justify left))
+    )
+    (property "Value" "C" (at 464.82 90.17 0)
+      (effects (font (size 1.27 1.27)) (justify left))
+    )
+    (property "Footprint" "Capacitor_SMD:C_0805_2012Metric_Pad1.18x1.45mm_HandSolder" (at 461.9752 92.71 0)
+      (effects (font (size 1.27 1.27)) hide)
+    )
+    (property "Datasheet" "~" (at 461.01 88.9 0)
+      (effects (font (size 1.27 1.27)) hide)
+    )
+    (pin "1")
+    (pin "2")
+    (instances
+      (project "BANO_StepDown_LM5160_Total_Duplicate"
+        (path "/68e09be7-3bbc-4443-a838-209ce20b2bef"
+          (reference "C18") (unit 1)
         )
       )
@@
     )
   )
+  (symbol (lib_id "power:GND2") (at 461.01 93.98 0) (unit 1)
+    (in_bom yes) (on_board yes) (dnp no) (fields_autoplaced)
+    (property "Reference" "#PWR022" (at 461.01 100.33 0)
+      (effects (font (size 1.27 1.27)) hide)
+    )
+    (property "Value" "GND2" (at 461.01 99.06 0)
+      (effects (font (size 1.27 1.27)))
+    )
+    (property "Footprint" "" (at 461.01 93.98 0)
+      (effects (font (size 1.27 1.27)) hide)
+    )
+    (property "Datasheet" "" (at 461.01 93.98 0)
+      (effects (font (size 1.27 1.27)) hide)
+    )
+    (pin "1")
+    (instances
+      (project "BANO_StepDown_LM5160_Total_Duplicate"
+        (path "/68e09be7-3bbc-4443-a838-209ce20b2bef"
+          (reference "#PWR022") (unit 1)
+        )
+      )
+    )
+  )
   (symbol (lib_id "Device:R") (at 370.84 243.84 270) (unit 1)
     (in_bom yes) (on_board yes) (dnp no) (fields_autoplaced)
@@
       (effects (font (size 1.524 1.524)))
     )
-    (property "Footprint" "ul_SWPA3015S4R7MT:IND_SWPA3015S_SNL" (at 246.38 92.71 0)
+    (property "Footprint" "ul_SWPA4030S1R0NT:IND_SWPA4030S_SNL" (at 246.38 92.71 0)
       (effects (font (size 1.27 1.27) italic) hide)
     )
@@
       (effects (font (size 1.27 1.27)) (justify left))
     )
-    (property "Footprint" "Wire_holes:WireHole_0p8" (at 222.25 100.33 0)
+    (property "Footprint" "Wire_holes:WireHole_1p2" (at 222.25 100.33 0)
       (effects (font (size 1.27 1.27)) hide)
     )
@@
       (effects (font (size 1.27 1.27)) (justify left))
     )
-    (property "Footprint" "Wire_holes:WireHole_0p8" (at 222.25 116.84 0)
+    (property "Footprint" "Connector_Pin:Pin_D0.7mm_L6.5mm_W1.8mm_FlatFork" (at 222.25 116.84 0)
       (effects (font (size 1.27 1.27)) hide)
     )
@@
         (path "/68e09be7-3bbc-4443-a838-209ce20b2bef"
           (reference "D2") (unit 1)
+        )
+      )
+    )
+  )
+  (symbol (lib_id "Device:C") (at 459.74 200.66 0) (unit 1)
+    (in_bom yes) (on_board yes) (dnp no) (fields_autoplaced)
+    (property "Reference" "C19" (at 463.55 199.39 0)
+      (effects (font (size 1.27 1.27)) (justify left))
+    )
+    (property "Value" "C" (at 463.55 201.93 0)
+      (effects (font (size 1.27 1.27)) (justify left))
+    )
+    (property "Footprint" "Capacitor_SMD:C_0805_2012Metric_Pad1.18x1.45mm_HandSolder" (at 460.7052 204.47 0)
+      (effects (font (size 1.27 1.27)) hide)
+    )
+    (property "Datasheet" "~" (at 459.74 200.66 0)
+      (effects (font (size 1.27 1.27)) hide)
+    )
+    (pin "1")
+    (pin "2")
+    (instances
+      (project "BANO_StepDown_LM5160_Total_Duplicate"
+        (path "/68e09be7-3bbc-4443-a838-209ce20b2bef"
+          (reference "C19") (unit 1)
         )
       )
@@
       (effects (font (size 1.27 1.27)) (justify left))
     )
-    (property "Footprint" "Wire_holes:WireHole_0p8" (at 218.44 177.8 0)
+    (property "Footprint" "Wire_holes:WireHole_1p2" (at 218.44 177.8 0)
       (effects (font (size 1.27 1.27)) hide)
     )
@@
       (effects (font (size 1.27 1.27)))
     )
-    (property "Footprint" "Resistor_SMD:R_0402_1005Metric_Pad0.72x0.64mm_HandSolder" (at 279.4 211.328 90)
+    (property "Footprint" "Resistor_SMD:R_0603_1608Metric_Pad0.98x0.95mm_HandSolder" (at 279.4 211.328 90)
       (effects (font (size 1.27 1.27)) hide)
     )
@@
       (effects (font (size 1.524 1.524)))
     )
-    (property "Footprint" "ul_SWPA3015S4R7MT:IND_SWPA3015S_SNL" (at 246.38 204.47 0)
+    (property "Footprint" "ul_SWPA4030S1R0NT:IND_SWPA4030S_SNL" (at 246.38 204.47 0)
       (effects (font (size 1.27 1.27) italic) hide)
     )
@@
       (effects (font (size 1.27 1.27)) (justify left))
     )
-    (property "Footprint" "Wire_holes:WireHole_0p8" (at 222.25 91.44 0)
+    (property "Footprint" "Wire_holes:WireHole_1p2" (at 222.25 91.44 0)
       (effects (font (size 1.27 1.27)) hide)
     )
@@
       (effects (font (size 1.27 1.27)))
     )
-    (property "Footprint" "Resistor_SMD:R_0402_1005Metric_Pad0.72x0.64mm_HandSolder" (at 279.4 99.568 90)
-      (effects (font (size 1.27 1.27)) hide)
-    )
+    (property "Footprint" "Resistor_SMD:R_0603_1608Metric_Pad0.98x0.95mm_HandSolder" (at 279.4 99.568 90)
+      (effects (font (size 1.27 1.27)) hide)
+    )

Commit message: PCB work 6
Parts:
- C27, C9: footprint Capacitor_SMD:C_0402_1005Metric_Pad0.74x0.62mm_HandSolder -> Capacitor_SMD:C_0603_1608Metric_Pad1.08x0.95mm_HandSolder
Changed lines of the file:
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@@
       (effects (font (size 1.27 1.27)) (justify left))
     )
-    (property "Footprint" "Capacitor_SMD:C_0402_1005Metric_Pad0.74x0.62mm_HandSolder" (at 355.2952 212.09 0)
+    (property "Footprint" "Capacitor_SMD:C_0603_1608Metric_Pad1.08x0.95mm_HandSolder" (at 355.2952 212.09 0)
       (effects (font (size 1.27 1.27)) hide)
     )
@@
       (effects (font (size 1.27 1.27)) (justify left))
     )
-    (property "Footprint" "Capacitor_SMD:C_0402_1005Metric_Pad0.74x0.62mm_HandSolder" (at 355.2952 100.33 0)
+    (property "Footprint" "Capacitor_SMD:C_0603_1608Metric_Pad1.08x0.95mm_HandSolder" (at 355.2952 100.33 0)
       (effects (font (size 1.27 1.27)) hide)
     )
@@
   )
   (symbol (lib_id "Device:C") (at 262.89 217.17 0) (unit 1)
-    (in_bom yes) (on_board yes) (dnp no) (fields_autoplaced)
-    (property "Reference" "C14" (at 266.7 215.9 0)
-      (effects (font (size 1.27 1.27)) (justify left))
-    )
+    (in_bom yes) (on_board yes) (dnp no)
+    (property "Reference" "C14" (at 264.16 214.63 0)
+      (effects (font (size 1.27 1.27)) (justify left))
+    )
