File: MUZ_001/Main_PCB_002.kicad_sch (KiCad schematic)
At the start: 108 parts, among them Q1 DMT10H009LK3-13, Q2 DMT10H009LK3-13, Q3 DMT10H009LK3-13, Q4 DMT10H009LK3-13, Q5 DMT10H009LK3-13, Q6 BSS123, Q7 BSS123, Q8 BSS123, Q9 DMT10H009LK3-13, U1 TLV9061IDCKR, U2 LM5164DDA, U3 LM5164DDA, U4 SI7489DP-T1-E3, U6 STM32G031G8Ux

Commit message: PCB work 7
Parts:
- added C5: C, Capacitor_SMD:C_0402_1005Metric_Pad0.74x0.62mm_HandSolder, symbol Device:C
- added LED1, LED2, LED26, LED3: HSMW-C191-U0000, ul_HSMW-C191-U0000:LED_91-U0000, symbol HSMW-C191:HSMW-C191-U0000
- added R1, R24, R25, R26, R6: R, Resistor_SMD:R_0402_1005Metric_Pad0.72x0.64mm_HandSolder, symbol Device:R
- added R4: R, Resistor_SMD:R_0603_1608Metric_Pad0.98x0.95mm_HandSolder, symbol Device:R
- added U5: TLV9061IDCKR, ul_TLV9061IDCKR:DCK5_TEX, symbol DCK5_TEX:TLV9061IDCKR
Connections:
- net GND2: now also C5.2, LED1.1, R24.1, R4.2, U5.2 (V-)
- net at LED18.1, LED19.1, LED20.1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: now also LED3.1
- net at LED14.1, LED15.1, LED16.1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: now also LED2.1
- net at R17.1, R20.1, R22.1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: now also R1.1, R25.1, R26.1
- net at C10.1, C4.1, C9.1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: now also C5.1, U5.5 (V+)
- net at U6.28 (PB8): now also R6.2, U5.4 (OUT)
- net at LED22.1, LED23.1, LED24.1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: now also LED26.1
- new net: R24.2, R6.1, U5.3 (IN-)
- new net: LED3.2, R25.2
- new net: LED26.2, R26.2
- new net: LED1.2, R4.1, U5.1 (IN+)
- new net: LED2.2, R1.2
Other:
- moved on the sheet: LED14, LED15, LED16, LED17, LED22, LED23, LED24, LED25, Q6, Q8, R17, R20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
