File: MUZ_001/Main_PCB_002.kicad_sch (KiCad schematic)
At the start: 120 parts, among them Q1 DMT10H009LK3-13, Q2 DMT10H009LK3-13, Q3 DMT10H009LK3-13, Q4 DMT10H009LK3-13, Q5 DMT10H009LK3-13, Q6 BSS123, Q7 BSS123, Q8 BSS123, Q9 DMT10H009LK3-13, U1 TLV9061IDCKR, U2 LM5164DDA, U3 LM5164DDA, U4 SI7489DP-T1-E3, U5 TLV9061IDCKR, U6 STM32G031G8Ux

Commit message: MUZ 001
Parts:
- added C14: C, Capacitor_SMD:C_0603_1608Metric_Pad1.08x0.95mm_HandSolder, symbol Device:C
- added D19: BZT52Bxx, Diode_SMD:D_SOD-123F, symbol Diode:BZT52Bxx
- added D20, D22, D23: WireHole_1p5, Wire_holes:WireHole_1p2, symbol Connectors_for_Wire:WireHole_1p5
- added R31: R, Resistor_SMD:R_0402_1005Metric_Pad0.72x0.64mm_HandSolder, symbol Device:R
- CR1, CR2, CR3: footprint SO-8_STM -> ul_L6388ED:SO-8_STM
- Q1, Q2, Q3, Q4, Q5, Q9: footprint QPMOS1G2S3D_TO252_DIO -> ul_DMT10H009LK3-13:QPMOS1G2S3D_TO252_DIO
Connections:
- net GND2: now also C14.2, D19.2 (A)
- net at D24.1 (Conn), Q1.3 (D), Q3.3 (D)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: now also R31.2
- net at C13.1, L1.1, R15.2: now also D22.1 (Conn); no longer CR1.3 (VCC), CR2.3 (VCC), CR3.3 (VCC)
- new net: C14.1, D19.1 (K), D20.1 (Conn), R31.1
- new net: CR1.3 (VCC), CR2.3 (VCC), CR3.3 (VCC), D23.1 (Conn)
Other:
- moved on the sheet: C12, C13, L1, LED1, R15, R23, R9, U2

Commit message: MUZ 001 PCB 001
Parts:
- added C15: C, Capacitor_SMD:C_0402_1005Metric, symbol Device:C
- added C16: C, Capacitor_SMD:C_0402_1005Metric_Pad0.74x0.62mm_HandSolder, symbol Device:C
- added R39, R40: R, Resistor_SMD:R_0402_1005Metric_Pad0.72x0.64mm_HandSolder, symbol Device:R
Connections:
- net at R15.1, R23.2, U2.5 (FB): now also C15.2
- net at C10.1, C4.1, C5.1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: now also C16.1, R40.2; no longer C9.1
- net at R13.2, R14.1, U3.5 (FB): now also C16.2
- net at D22.1 (Conn), L1.1, R15.2: now also C15.1, R39.2; no longer C13.1
- new net: C9.1, R40.1
- new net: C13.1, R39.1
Other:
- moved on the sheet: C13, C9, R13, R14, R15, R23

Commit message: MUZ 001 PCB 001
Parts:
- removed Q5, Q9: DMT10H009LK3-13, ul_DMT10H009LK3-13:QPMOS1G2S3D_TO252_DIO, symbol DMT10H009LK3:DMT10H009LK3-13
- added Q10, Q11: BSS123, Package_TO_SOT_SMD:SOT-23, symbol Transistor_FET:BSS123
- R30, R4, R7: footprint Resistor_SMD:R_0603_1608Metric_Pad0.98x0.95mm_HandSolder -> Resistor_SMD:R_0402_1005Metric_Pad0.72x0.64mm_HandSolder
Connections:
- net GND2: now also Q11.2 (S)
- net at D24.1 (Conn), Q1.3 (D), Q3.3 (D)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: now also Q10.3 (D)
- net at CR2.5 (LVG): now also Q11.1 (G)
- net at C1.2, CR2.6 (OUT), D14.1 (Conn): now also Q10.2 (S), Q11.3 (D)
- net at CR2.7 (HVG): now also Q10.1 (G)
Changed lines of the file:
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@@
       (effects (font (size 1.27 1.27)) (justify left))
     )
-    (property "Footprint" "Resistor_SMD:R_0603_1608Metric_Pad0.98x0.95mm_HandSolder" (at 441.198 464.82 90)
+    (property "Footprint" "Resistor_SMD:R_0402_1005Metric_Pad0.72x0.64mm_HandSolder" (at 441.198 464.82 90)
       (effects (font (size 1.27 1.27)) hide)
     )
@@
         (path "/68e09be7-3bbc-4443-a838-209ce20b2bef"
           (reference "R34") (unit 1)
+        )
+      )
+    )
+  )
+  (symbol (lib_name "BSS123_1") (lib_id "Transistor_FET:BSS123") (at 344.17 97.79 0) (unit 1)
+    (in_bom yes) (on_board yes) (dnp no) (fields_autoplaced)
+    (property "Reference" "Q10" (at 350.52 96.52 0)
+      (effects (font (size 1.27 1.27)) (justify left))
+    )
+    (property "Value" "BSS123" (at 350.52 99.06 0)
+      (effects (font (size 1.27 1.27)) (justify left))
+    )
+    (property "Footprint" "Package_TO_SOT_SMD:SOT-23" (at 349.25 99.695 0)
+      (effects (font (size 1.27 1.27) italic) (justify left) hide)
+    )
+    (property "Datasheet" "http://www.diodes.com/assets/Datasheets/ds30366.pdf" (at 349.25 101.6 0)
+      (effects (font (size 1.27 1.27)) (justify left) hide)
+    )
+    (pin "2")
+    (pin "1")
+    (pin "3")
+    (instances
+      (project "Main_PCB_002"
+        (path "/68e09be7-3bbc-4443-a838-209ce20b2bef"
+          (reference "Q10") (unit 1)
         )
       )
@@
         (path "/68e09be7-3bbc-4443-a838-209ce20b2bef"
           (reference "#PWR013") (unit 1)
-        )
-      )
-    )
-  )
-  (symbol (lib_id "DMT10H009LK3:DMT10H009LK3-13") (at 339.09 110.49 0) (unit 1)
-    (in_bom yes) (on_board yes) (dnp no)
-    (property "Reference" "Q9" (at 350.52 109.22 0)
-      (effects (font (size 1.524 1.524)) (justify left))
-    )
-    (property "Value" "DMT10H009LK3-13" (at 350.52 110.49 0)
-      (effects (font (size 1.524 1.524)) (justify left))
-    )
-    (property "Footprint" "ul_DMT10H009LK3-13:QPMOS1G2S3D_TO252_DIO" (at 339.09 110.49 0)
-      (effects (font (size 1.27 1.27) italic) hide)
-    )
-    (property "Datasheet" "DMT10H009LK3-13" (at 339.09 110.49 0)
-      (effects (font (size 1.27 1.27) italic) hide)
-    )
-    (pin "1")
-    (pin "2")
-    (pin "3")
-    (instances
-      (project "Main_PCB_002"
-        (path "/68e09be7-3bbc-4443-a838-209ce20b2bef"
-          (reference "Q9") (unit 1)
         )
       )
@@
       (effects (font (size 1.27 1.27)) (justify left))
     )
-    (property "Footprint" "Resistor_SMD:R_0603_1608Metric_Pad0.98x0.95mm_HandSolder" (at 117.602 410.21 90)
+    (property "Footprint" "Resistor_SMD:R_0402_1005Metric_Pad0.72x0.64mm_HandSolder" (at 117.602 410.21 90)
       (effects (font (size 1.27 1.27)) hide)
     )
@@
       (effects (font (size 1.27 1.27)) (justify left))
     )
-    (property "Footprint" "Resistor_SMD:R_0603_1608Metric_Pad0.98x0.95mm_HandSolder" (at 117.602 430.53 90)
+    (property "Footprint" "Resistor_SMD:R_0402_1005Metric_Pad0.72x0.64mm_HandSolder" (at 117.602 430.53 90)
       (effects (font (size 1.27 1.27)) hide)
     )
@@
     )
   )
-  (symbol (lib_id "DMT10H009LK3:DMT10H009LK3-13") (at 339.09 97.79 0) (unit 1)
-    (in_bom yes) (on_board yes) (dnp no)
-    (property "Reference" "Q5" (at 350.52 96.52 0)
-      (effects (font (size 1.524 1.524)) (justify left))
-    )
-    (property "Value" "DMT10H009LK3-13" (at 350.52 97.79 0)
-      (effects (font (size 1.524 1.524)) (justify left))
-    )
-    (property "Footprint" "ul_DMT10H009LK3-13:QPMOS1G2S3D_TO252_DIO" (at 339.09 97.79 0)
-      (effects (font (size 1.27 1.27) italic) hide)
-    )
-    (property "Datasheet" "DMT10H009LK3-13" (at 339.09 97.79 0)
-      (effects (font (size 1.27 1.27) italic) hide)
-    )
-    (pin "1")
-    (pin "2")
-    (pin "3")
-    (instances
-      (project "Main_PCB_002"
-        (path "/68e09be7-3bbc-4443-a838-209ce20b2bef"
-          (reference "Q5") (unit 1)
-        )
-      )
-    )
-  )
   (symbol (lib_id "Device:C") (at 264.16 363.22 0) (unit 1)
     (in_bom yes) (on_board yes) (dnp no)
@@
         )
       )
+    )
+  )
+  (symbol (lib_name "BSS123_1") (lib_id "Transistor_FET:BSS123") (at 344.17 110.49 0) (unit 1)
+    (in_bom yes) (on_board yes) (dnp no) (fields_autoplaced)
+    (property "Reference" "Q11" (at 350.52 109.22 0)
+      (effects (font (size 1.27 1.27)) (justify left))
+    )
+    (property "Value" "BSS123" (at 350.52 111.76 0)
+      (effects (font (size 1.27 1.27)) (justify left))
+    )
+    (property "Footprint" "Package_TO_SOT_SMD:SOT-23" (at 349.25 112.395 0)
+      (effects (font (size 1.27 1.27) italic) (justify left) hide)
+    )
+    (property "Datasheet" "http://www.diodes.com/assets/Datasheets/ds30366.pdf" (at 349.25 114.3 0)
+      (effects (font (size 1.27 1.27)) (justify left) hide)
+    )
+    (pin "2")
+    (pin "1")
+    (pin "3")
+    (instances
+      (project "Main_PCB_002"
+        (path "/68e09be7-3bbc-4443-a838-209ce20b2bef"
+          (reference "Q11") (unit 1)
+        )
+      )
