File: MUZ_001/Main_PCB_002.kicad_pcb (KiCad board)
At the start: 2 copper layers, 88.9 x 22.2 mm, 87 parts, among them Q1 BSS123, U1 INA193, U3 LM5164DDA, U4 SI7489DP-T1-E3, U5 SI7489DP-T1-E3, U6 STM32G031G8Ux, U7 SI7489DP-T1-E3, U8 LM5164DDA

Commit message: MUZ 001
Parts:
- removed C15: C, Capacitor_SMD:C_0805_2012Metric_Pad1.18x1.45mm_HandSolder
- removed D29, D30: WireHole_1p5, Wire_holes:WireHole_1p2
- removed L3: SWPA4030S1R0NT, ul_VLS252012HBU-220M:IND_VLS252012_TDK
- removed U7: SI7489DP-T1-E3, ul_SI7852DP-T1:POWERPAK_SO-8_SINGLE_VIS
- removed U8: LM5164DDA, Package_SO:HSOP-8-1EP_3.9x4.9mm_P1.27mm_EP2.41x3.1mm_ThermalVias
- added C5: C, Capacitor_SMD:C_0402_1005Metric_Pad0.74x0.62mm_HandSolder, F.Cu at (115.0, 100.8)
- added C6: C, Capacitor_SMD:C_0805_2012Metric, F.Cu at (113.3, 115.9)
- added CR1: L6388ED, ul_L6388ED:SO-8_STM, F.Cu at (193.0, 158.1)
- added CR2: L6388ED, ul_L6388ED:SO-8_STM, F.Cu at (223.5, 88.9)
- added CR3: L6388ED, ul_L6388ED:SO-8_STM, F.Cu at (231.2, 127.6)
- added L1: SWPA4030S1R0NT, ul_VLS252012HBU-220M:IND_VLS252012_TDK, F.Cu at (52.1, 48.3)
- added LED10: HSMW-C191-U0000, ul_HSMW-C191-U0000:LED_91-U0000, F.Cu at (177.2, 79.1)
- added LED11: HSMW-C191-U0000, ul_HSMW-C191-U0000:LED_91-U0000, F.Cu at (177.2, 81.6)
- added LED12: HSMW-C191-U0000, ul_HSMW-C191-U0000:LED_91-U0000, F.Cu at (177.2, 84.1)
- added LED13: HSMW-C191-U0000, ul_HSMW-C191-U0000:LED_91-U0000, F.Cu at (177.2, 86.6)
- added LED14: HSMW-C191-U0000, ul_HSMW-C191-U0000:LED_91-U0000, F.Cu at (177.2, 89.0)
- added LED15: HSMW-C191-U0000, ul_HSMW-C191-U0000:LED_91-U0000, F.Cu at (177.2, 91.5)
- added LED16: HSMW-C191-U0000, ul_HSMW-C191-U0000:LED_91-U0000, F.Cu at (177.2, 94.0)
- added LED17: HSMW-C191-U0000, ul_HSMW-C191-U0000:LED_91-U0000, F.Cu at (177.2, 96.5)
- added LED18: HSMW-C191-U0000, ul_HSMW-C191-U0000:LED_91-U0000, F.Cu at (177.2, 98.9)
- added LED19: HSMW-C191-U0000, ul_HSMW-C191-U0000:LED_91-U0000, F.Cu at (182.5, 79.1)
- added LED20: HSMW-C191-U0000, ul_HSMW-C191-U0000:LED_91-U0000, F.Cu at (182.5, 81.6)
- added LED21: HSMW-C191-U0000, ul_HSMW-C191-U0000:LED_91-U0000, F.Cu at (182.5, 84.1)
- added LED22: HSMW-C191-U0000, ul_HSMW-C191-U0000:LED_91-U0000, F.Cu at (182.5, 86.6)
- added LED23: HSMW-C191-U0000, ul_HSMW-C191-U0000:LED_91-U0000, F.Cu at (182.5, 89.0)
- added LED24: HSMW-C191-U0000, ul_HSMW-C191-U0000:LED_91-U0000, F.Cu at (182.5, 91.5)
- added LED25: HSMW-C191-U0000, ul_HSMW-C191-U0000:LED_91-U0000, F.Cu at (182.5, 94.0)
- added LED26: HSMW-C191-U0000, ul_HSMW-C191-U0000:LED_91-U0000, F.Cu at (182.5, 96.5)
- added LED4: HSMW-C191-U0000, ul_HSMW-C191-U0000:LED_91-U0000, F.Cu at (171.9, 86.6)
- added LED5: HSMW-C191-U0000, ul_HSMW-C191-U0000:LED_91-U0000, F.Cu at (171.9, 89.0)
- added LED6: HSMW-C191-U0000, ul_HSMW-C191-U0000:LED_91-U0000, F.Cu at (171.9, 91.5)
- added LED7: HSMW-C191-U0000, ul_HSMW-C191-U0000:LED_91-U0000, F.Cu at (171.9, 94.0)
- added LED8: HSMW-C191-U0000, ul_HSMW-C191-U0000:LED_91-U0000, F.Cu at (171.9, 96.5)
- added LED9: HSMW-C191-U0000, ul_HSMW-C191-U0000:LED_91-U0000, F.Cu at (171.9, 98.9)
- added Q2: DMT10H009LK3-13, ul_DMT10H009LK3-13:QPMOS1G2S3D_TO252_DIO, F.Cu at (198.1, 147.3)
- added Q3: DMT10H009LK3-13, ul_DMT10H009LK3-13:QPMOS1G2S3D_TO252_DIO, F.Cu at (187.7, 147.2)
- added Q4: DMT10H009LK3-13, ul_DMT10H009LK3-13:QPMOS1G2S3D_TO252_DIO, F.Cu at (228.9, 116.8)
- added Q5: DMT10H009LK3-13, ul_DMT10H009LK3-13:QPMOS1G2S3D_TO252_DIO, F.Cu at (218.7, 78.7)
- added Q6: BSS123, Package_TO_SOT_SMD:SOT-23, F.Cu at (154.0, 45.7)
- added Q7: BSS123, Package_TO_SOT_SMD:SOT-23, F.Cu at (145.7, 44.8)
- added Q8: BSS123, Package_TO_SOT_SMD:SOT-23, F.Cu at (161.0, 44.1)
- added Q9: DMT10H009LK3-13, ul_DMT10H009LK3-13:QPMOS1G2S3D_TO252_DIO, F.Cu at (231.1, 78.0)
- added R32: R, Resistor_SMD:R_0402_1005Metric_Pad0.72x0.64mm_HandSolder, F.Cu at (109.5, 109.4)
- added R33: R, Resistor_SMD:R_0402_1005Metric_Pad0.72x0.64mm_HandSolder, F.Cu at (109.5, 111.4)
- added R34: R, Resistor_SMD:R_0402_1005Metric_Pad0.72x0.64mm_HandSolder, F.Cu at (109.5, 113.3)
- added R35: R, Resistor_SMD:R_0402_1005Metric_Pad0.72x0.64mm_HandSolder, F.Cu at (109.5, 115.3)
- added R36: R, Resistor_SMD:R_0402_1005Metric_Pad0.72x0.64mm_HandSolder, F.Cu at (109.5, 117.3)
- added R37: R, Resistor_SMD:R_0402_1005Metric_Pad0.72x0.64mm_HandSolder, F.Cu at (109.5, 119.3)
- added R38: R, Resistor_SMD:R_0402_1005Metric_Pad0.72x0.64mm_HandSolder, F.Cu at (109.5, 121.3)
- added U2: LM5164DDA, Package_SO:HSOP-8-1EP_3.9x4.9mm_P1.27mm_EP2.41x3.1mm_ThermalVias, F.Cu at (43.3, 45.1)
- C1, C3: footprint Capacitor_SMD:C_0805_2012Metric_Pad1.18x1.45mm_HandSolder -> Capacitor_SMD:C_0805_2012Metric
- C12: footprint Capacitor_SMD:C_0402_1005Metric_Pad0.74x0.62mm_HandSolder -> Capacitor_SMD:C_0603_1608Metric_Pad1.08x0.95mm_HandSolder
- C13: footprint Capacitor_SMD:C_0402_1005Metric_Pad0.74x0.62mm_HandSolder -> Capacitor_SMD:C_0805_2012Metric
- C4: footprint Capacitor_SMD:C_0603_1608Metric_Pad1.08x0.95mm_HandSolder -> Capacitor_SMD:C_0402_1005Metric_Pad0.74x0.62mm_HandSolder
- D14, D6: value MM5Zxx -> WireHole_1p5; footprint Diode_SMD:D_SOD-523 -> Wire_holes:WireHole_1p2
- D19: value WireHole_1p5 -> BZT52Bxx; footprint Wire_holes:WireHole_1p2 -> Diode_SMD:D_SOD-123F
- D20: value BAT54C -> WireHole_1p5; footprint Package_TO_SOT_SMD:SOT-23 -> Wire_holes:WireHole_1p2
- Q1: value BSS123 -> DMT10H009LK3-13; footprint Package_TO_SOT_SMD:SOT-23 -> ul_DMT10H009LK3-13:QPMOS1G2S3D_TO252_DIO
- R1: footprint Resistor_SMD:R_0603_1608Metric_Pad0.98x0.95mm_HandSolder -> Resistor_SMD:R_0402_1005Metric_Pad0.72x0.64mm_HandSolder
- R15, R23, R24, R25, R26, R27, R28, R6, R9: value BLM18KG102SH1D -> R; footprint ul_BLM18KG102SH1D:RES_0603_1P6XP8_MUR -> Resistor_SMD:R_0402_1005Metric_Pad0.72x0.64mm_HandSolder
- R30: footprint Resistor_SMD:R_0402_1005Metric_Pad0.72x0.64mm_HandSolder -> Resistor_SMD:R_0603_1608Metric_Pad0.98x0.95mm_HandSolder
- R4, R7: value BLM18KG102SH1D -> R; footprint ul_BLM18KG102SH1D:RES_0603_1P6XP8_MUR -> Resistor_SMD:R_0603_1608Metric_Pad0.98x0.95mm_HandSolder
- U1: value INA193 -> TLV9061IDCKR; footprint Package_TO_SOT_SMD:SOT-23-5 -> ul_TLV9061IDCKR:DCK5_TEX
- U5: value SI7489DP-T1-E3 -> TLV9061IDCKR; footprint ul_SI7852DP-T1:POWERPAK_SO-8_SINGLE_VIS -> ul_TLV9061IDCKR:DCK5_TEX
- moved R23 119.5 mm to (50.2, 50.8)
- moved Q1 117.9 mm to (238.8, 116.8), turned to 0 degrees
- moved R9 116.6 mm to (36.2, 50.8), turned to 0 degrees
- moved R31 108.4 mm to (43.7, 66.0), turned to 0 degrees
- moved C13 107.7 mm to (57.5, 48.3)
- moved R15 105.3 mm to (52.7, 50.8), turned to 0 degrees
- moved D19 92.9 mm to (49.4, 63.5)
- moved U6 83.1 mm to (57.4, 142.8)
- moved C12 80.7 mm to (50.8, 44.0), turned to 90 degrees
- moved D22 76.1 mm to (55.9, 53.3)
- moved C14 74.4 mm to (48.5, 66.0), turned to 0 degrees
- moved D23 72.6 mm to (61.0, 53.3)
- moved D4 71.2 mm to (15.2, 109.2)
- moved D3 62.1 mm to (15.2, 104.1), turned to 0 degrees
- moved D20 62.0 mm to (55.9, 63.5)
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Connections:
- C1 pad 1: Net-(C1-Pad1) -> Net-(CR1-VBOOT)
- C1 pad 2: GND2 -> Net-(CR2-OUT)
- C10 pad 1: Net-(D26-Conn) -> Net-(D16-Conn)
- C12 pad 1: Net-(D14-A) -> Net-(U2-BST)
- C12 pad 2: GND2 -> Net-(U2-SW)
- C13 pad 1: Net-(U6-PA4) -> Net-(D22-Conn)
- C14 pad 1: Net-(U8-BST) -> Net-(D19-K)
- C14 pad 2: Net-(U8-SW) -> GND2
- C3 pad 1: Net-(C3-Pad1) -> Net-(D6-Conn)
- C4 pad 1: Net-(D26-Conn) -> Net-(D16-Conn)
- C9 pad 1: Net-(D26-Conn) -> Net-(D16-Conn)
- D12 pad 1: Net-(D12-Conn) -> Net-(CR1-OUT)
- D14 pad 1: Net-(D14-K) -> Net-(CR2-OUT)
- D15 pad 1: Net-(D15-Conn) -> GND2
- D16 pad 1: Net-(D15-Conn) -> Net-(D16-Conn)
- D18 pad 1: GND2 -> Net-(D18-Conn)
- D19 pad 1: Net-(D19-Conn) -> Net-(D19-K)
- D2 pad 1: Net-(D2-Conn) -> Net-(CR3-OUT)
- D20 pad 1: Net-(D24-Conn) -> Net-(D19-K)
- D23 pad 1: Net-(D14-K) -> Net-(CR1-VCC)
- D26 pad 1: Net-(D26-Conn) -> Net-(D16-Conn)
- D27 pad 1: Net-(D26-Conn) -> Net-(D16-Conn)
- D28 pad 1: Net-(D26-Conn) -> Net-(D16-Conn)
- D6 pad 1: Net-(D24-Conn) -> Net-(D6-Conn)
- D7 pad 1: Net-(D7-Conn) -> Net-(D16-Conn)
- L2 pad 1: Net-(D26-Conn) -> Net-(D16-Conn)
- L2 pad 2: Net-(U3-BST) -> Net-(U3-SW)
- LED1 pad 1: unconnected-(LED1-Pad1) -> GND2
- LED1 pad 2: Net-(LED1-Pad2) -> Net-(U5-IN+)
- LED2 pad 1: unconnected-(LED2-Pad1) -> Net-(Q6-D)
- LED3 pad 1: unconnected-(LED3-Pad1) -> Net-(Q7-D)
- Q1 pad 1: Net-(Q1-G) -> Net-(CR3-HVG)
- Q1 pad 2: GND2 -> Net-(CR3-OUT)
- Q1 pad 3: Net-(Q1-D) -> Net-(D24-Conn)
- R1 pad 1: Net-(U1--) -> Net-(R1-Pad1)
- R1 pad 2: Net-(U1-+) -> Net-(LED2-Pad2)
- R11 pad 1: Net-(D6-A) -> Net-(LED12-Pad2)
- R11 pad 2: Net-(D24-Conn) -> Net-(U6-PA11/PA9)
- R14 pad 2: Net-(D26-Conn) -> Net-(D16-Conn)
- R15 pad 1: Net-(U6-PA3) -> Net-(U2-FB)
- R15 pad 2: Net-(D11-Conn) -> Net-(D22-Conn)
- R16 pad 1: Net-(U6-PA0) -> Net-(LED13-Pad2)
- R16 pad 2: Net-(U3-EN/UVLO) -> Net-(U6-PA12/PA10)
- R17 pad 1: GND2 -> Net-(R1-Pad1)
- R17 pad 2: Net-(U6-PA0) -> Net-(LED14-Pad2)
- R18 pad 2: Net-(D26-Conn) -> Net-(D16-Conn)
- R2 pad 1: Net-(U6-PB4) -> Net-(LED4-Pad2)
- R2 pad 2: Net-(D22-Conn) -> Net-(U6-PA6)
- R20 pad 1: GND2 -> Net-(R1-Pad1)
- R20 pad 2: Net-(D14-A) -> Net-(LED15-Pad2)
- R21 pad 1: Net-(U6-PA4) -> Net-(U1-IN-)
- R21 pad 2: Net-(R21-Pad2) -> Net-(U1-OUT)
- R22 pad 1: GND2 -> Net-(R1-Pad1)
- R23 pad 1: Net-(U6-PA13) -> GND2
- R23 pad 2: Net-(D8-Conn) -> Net-(U2-FB)
- R24 pad 1: Net-(U6-PA14) -> GND2
- R24 pad 2: Net-(D9-Conn) -> Net-(U5-IN-)
- R25 pad 1: Net-(U6-PB7) -> Net-(R1-Pad1)
- R25 pad 2: Net-(D1-Conn) -> Net-(LED3-Pad2)
- R26 pad 1: Net-(U6-PB6) -> Net-(R1-Pad1)
- R26 pad 2: Net-(D21-Conn) -> Net-(LED26-Pad2)
- R27 pad 1: Net-(C3-Pad1) -> Net-(R1-Pad1)
- R27 pad 2: Net-(D7-Conn) -> Net-(LED17-Pad2)
- R28 pad 1: Net-(D26-Conn) -> Net-(R1-Pad1)
- R28 pad 2: Net-(D19-Conn) -> Net-(LED18-Pad2)
- R29 pad 1: Net-(LED1-Pad2) -> GND2
- R29 pad 2: Net-(U6-PC6) -> Net-(U1-IN-)
- R3 pad 1: Net-(U6-PB5) -> Net-(LED10-Pad2)
- R3 pad 2: Net-(D24-Conn) -> Net-(U6-PA7)
- R30 pad 1: Net-(LED2-Pad2) -> Net-(D18-Conn)
- R30 pad 2: Net-(U6-PB1) -> Net-(U1-IN+)
- R31 pad 1: Net-(LED3-Pad2) -> Net-(D19-K)
- R31 pad 2: Net-(U6-PB0) -> Net-(D24-Conn)
- R4 pad 1: Net-(D12-Conn) -> Net-(U5-IN+)
- R4 pad 2: Net-(C1-Pad1) -> GND2
- R6 pad 1: Net-(U1--) -> Net-(U5-IN-)
- R6 pad 2: Net-(D2-Conn) -> Net-(U5-OUT)
- R7 pad 1: Net-(D13-Conn) -> Net-(U1-IN+)
- R7 pad 2: Net-(R21-Pad2) -> GND2
- R8 pad 1: Net-(Q1-D) -> Net-(LED11-Pad2)
- R8 pad 2: Net-(D6-A) -> Net-(U6-PA8)
- R9 pad 1: Net-(U6-PA2) -> GND2
- R9 pad 2: Net-(D10-Conn) -> Net-(U2-RON)
- U1 pad 1: Net-(U8-FB) -> Net-(U1-IN+)
- U1 pad 3: Net-(U1-+) -> Net-(U1-IN-)
- U1 pad 4: Net-(U1--) -> Net-(U1-OUT)
- U1 pad 5: Net-(D26-Conn) -> Net-(D16-Conn)
- U3 pad 2: Net-(U3-EN/UVLO) -> Net-(D24-Conn)
- U3 pad 3: Net-(U3-EN/UVLO) -> Net-(D24-Conn)
- U5 pad 1: Net-(D24-Conn) -> Net-(U5-IN+)
- U5 pad 2: Net-(D24-Conn) -> GND2
- U5 pad 3: Net-(D24-Conn) -> Net-(U5-IN-)
- U5 pad 4: Net-(D6-A) -> Net-(U5-OUT)
- U5 pad 5: Net-(C3-Pad1) -> Net-(D16-Conn)
- U6 pad 1: unconnected-(U6-PC14-Pad1) -> Net-(CR1-HIN)
- U6 pad 10: Net-(U6-PA4) -> Net-(D13-Conn)
- U6 pad 11: unconnected-(U6-PA5-Pad11) -> Net-(D6-Conn)
- U6 pad 12: unconnected-(U6-PA6-Pad12) -> Net-(U6-PA6)
- U6 pad 13: unconnected-(U6-PA7-Pad13) -> Net-(U6-PA7)
- U6 pad 14: Net-(U6-PB0) -> Net-(U1-OUT)
- U6 pad 15: Net-(U6-PB1) -> Net-(CR3-HIN)
- U6 pad 16: unconnected-(U6-PA8-Pad16) -> Net-(U6-PA8)
- U6 pad 17: Net-(U6-PC6) -> Net-(CR2-LIN)
- U6 pad 18: unconnected-(U6-PA11/PA9-Pad18) -> Net-(U6-PA11/PA9)
- U6 pad 19: unconnected-(U6-PA12/PA10-Pad19) -> Net-(U6-PA12/PA10)
- U6 pad 2: unconnected-(U6-PC15-Pad2) -> Net-(CR1-LIN)
- U6 pad 20: Net-(U6-PA13) -> Net-(D8-Conn)
- U6 pad 21: Net-(U6-PA14) -> Net-(D9-Conn)
- U6 pad 22: Net-(Q1-G) -> Net-(U6-PA15)
- U6 pad 23: unconnected-(U6-PB3-Pad23) -> Net-(U6-PB3)
- U6 pad 24: Net-(U6-PB4) -> Net-(CR3-LIN)
- U6 pad 25: Net-(U6-PB5) -> Net-(CR2-HIN)
- U6 pad 26: Net-(U6-PB6) -> Net-(D21-Conn)
- U6 pad 27: Net-(U6-PB7) -> Net-(D1-Conn)
- U6 pad 28: unconnected-(U6-PB8-Pad28) -> Net-(U5-OUT)
- U6 pad 3: Net-(D26-Conn) -> Net-(D16-Conn)
- U6 pad 6: Net-(U6-PA0) -> Net-(Q6-G)
- U6 pad 8: Net-(U6-PA2) -> Net-(D10-Conn)
- U6 pad 9: Net-(U6-PA3) -> Net-(D11-Conn)
Routing:
- net Net-(D26-Conn): track 85.5 -> 0.00 mm, vias 3 -> 0
- net Net-(D24-Conn): track 70.5 -> 0.00 mm, vias 2 -> 0
- net Net-(D22-Conn): track 69.5 -> 0.00 mm, vias 2 -> 0
- net Net-(U6-PA0): track 48.9 -> 0.00 mm
- net Net-(U6-PA1): track 28.9 -> 0.00 mm
- net Net-(Q1-G): track 24.7 -> 0.00 mm, vias 2 -> 0
- net Net-(U8-FB): track 23.6 -> 0.00 mm
- net Net-(C1-Pad1): track 17.8 -> 0.00 mm
- net Net-(C2-Pad1): track 16.6 -> 0.00 mm
- net Net-(U3-FB): track 15.3 -> 0.00 mm
- net Net-(D25-Conn): track 14.5 -> 0.00 mm
- net Net-(D14-K): track 14.2 -> 0.00 mm
- net Net-(U6-PA13): track 14.1 -> 0.00 mm
- net Net-(U6-PA14): track 13.2 -> 0.00 mm
- net Net-(U6-PB7): track 12.6 -> 0.00 mm, vias 2 -> 0
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- removed copper zone on B.Cu, net GND2
- removed copper zone on F.Cu, net GND2
Other:
- board outline removed
- board text removed: "3.3B"
- board text removed: "CLK"
- board text removed: "GND"
- board text removed: "IO"
- board text removed: "RX"
- board text removed: "TX"
- board text removed: "UART1"
- board text removed: "UART2"
- board text removed: "НАВ"
- board text removed: "СТРОБ"
- board text removed: "Синхро"

Commit message: MUZ 001
Parts:
- moved D12 155.1 mm to (244.5, 160.7)
- moved D2 142.0 mm to (237.7, 126.3)
- moved D14 137.0 mm to (238.5, 92.1)
- moved R4 126.5 mm to (191.2, 31.8)
- moved R6 125.4 mm to (194.4, 33.0)
- moved C1 122.9 mm to (231.1, 74.9)
- moved R24 121.2 mm to (196.9, 33.0)
- moved U1 110.0 mm to (40.3, 172.1)
- moved Q8 109.7 mm to (167.0, 153.7)
- moved Q7 109.5 mm to (157.4, 153.7)
- moved Q6 108.2 mm to (146.6, 153.7)
- moved D18 105.1 mm to (32.7, 173.3)
- moved C5 105.0 mm to (191.8, 29.2)
- moved U5 103.4 mm to (195.3, 29.8)
- moved C4 102.9 mm to (40.3, 169.5)
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
Commit message: MUZ 001 PCB 001
Parts:
- added C15: C, Capacitor_SMD:C_0402_1005Metric, F.Cu at (48.1, 46.8)
- added C16: C, Capacitor_SMD:C_0402_1005Metric_Pad0.74x0.62mm_HandSolder, F.Cu at (52.2, 86.7)
- added R39: R, Resistor_SMD:R_0402_1005Metric_Pad0.72x0.64mm_HandSolder, F.Cu at (47.9, 48.5)
- added R40: R, Resistor_SMD:R_0402_1005Metric_Pad0.72x0.64mm_HandSolder, F.Cu at (42.8, 101.2)
- moved R15 7.59 mm to (45.5, 48.5)
- moved R23 7.49 mm to (43.1, 48.5)
- moved C13 6.63 mm to (50.9, 48.0)
- moved R9 5.11 mm to (40.7, 48.5), turned to 180 degrees
- moved L1 4.21 mm to (50.7, 44.3), turned to 90 degrees
- moved C12 2.84 mm to (48.0, 44.0)
- moved R12 2.77 mm to (38.3, 96.0)
- moved R13 1.88 mm to (40.6, 96.0)
Connections:
- C13 pad 1: Net-(D22-Conn) -> Net-(C13-Pad1)
- C9 pad 1: Net-(D16-Conn) -> Net-(C9-Pad1)
Routing:
- net Net-(D22-Conn): track 0.00 -> 5.60 mm
- net Net-(U2-FB): track 0.00 -> 5.48 mm
- net Net-(U2-SW): track 0.00 -> 4.60 mm
- net Net-(U2-BST): track 0.00 -> 2.20 mm
- net Net-(U2-RON): track 0.00 -> 1.75 mm
- net Net-(C13-Pad1): track 0.00 -> 1.54 mm
- net Net-(D24-Conn): track 0.00 -> 1.27 mm

Commit message: MUZ 001 PCB 001
Parts:
- removed Q5, Q9: DMT10H009LK3-13, ul_DMT10H009LK3-13:QPMOS1G2S3D_TO252_DIO
- added Q10: BSS123, Package_TO_SOT_SMD:SOT-23, F.Cu at (229.5, 95.7)
- added Q11: BSS123, Package_TO_SOT_SMD:SOT-23, F.Cu at (229.4, 99.7)
- R30, R4, R7: footprint Resistor_SMD:R_0603_1608Metric_Pad0.98x0.95mm_HandSolder -> Resistor_SMD:R_0402_1005Metric_Pad0.72x0.64mm_HandSolder
- moved R14 64.3 mm to (49.0, 36.1), turned to -90 degrees
- moved R40 63.6 mm to (49.0, 37.9), turned to 180 degrees
- moved C9 62.1 mm to (52.0, 37.4)
- moved U3 58.5 mm to (44.3, 34.2)
- moved C8 58.3 mm to (49.2, 33.1), turned to 90 degrees
- moved R13 58.2 mm to (44.2, 37.9)
- moved R12 58.2 mm to (41.8, 37.9), turned to 180 degrees
- moved L2 54.9 mm to (52.1, 33.5), turned to 90 degrees
- moved C16 49.1 mm to (46.6, 37.9), turned to 180 degrees
- moved CR1 42.2 mm to (225.4, 118.3)
- moved D12 31.4 mm to (229.5, 133.0), turned to 180 degrees
- moved D2 24.7 mm to (235.9, 101.7)
- moved Q2 23.6 mm to (225.5, 128.5), turned to 180 degrees
- moved Q3 21.9 mm to (234.0, 128.6), turned to 180 degrees
- moved C1 19.7 mm to (225.4, 93.7), turned to 180 degrees
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Routing:
- net Net-(D24-Conn): track 1.27 -> 57.8 mm
- net Net-(CR1-VCC): track 0.00 -> 25.6 mm
- net Net-(CR3-OUT): track 0.00 -> 22.5 mm
- net Net-(CR1-OUT): track 0.00 -> 21.2 mm
- net GND2: track 0.00 -> 17.6 mm
- net Net-(CR2-OUT): track 0.00 -> 15.5 mm
- net Net-(CR3-HVG): track 0.00 -> 11.3 mm
- net Net-(CR1-HVG): track 0.00 -> 10.9 mm
- net Net-(D16-Conn): track 0.00 -> 9.51 mm
- net Net-(U3-FB): track 0.00 -> 5.68 mm
- net Net-(U3-SW): track 0.00 -> 5.13 mm
- net Net-(U5-IN-): track 0.00 -> 3.86 mm
- net Net-(CR2-HVG): track 0.00 -> 3.77 mm
- net Net-(CR3-LVG): track 0.00 -> 3.72 mm
- net Net-(CR1-LVG): track 0.00 -> 3.42 mm
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
Commit message: MUZ 001 PCB 001
Parts:
- moved D25 15.5 mm to (34.5, 102.3)
- moved R10 11.4 mm to (33.1, 99.6), turned to 180 degrees
- moved C7 11.2 mm to (33.1, 98.4)
- moved D3 6.79 mm to (20.8, 100.6)
- moved R5 5.96 mm to (22.5, 98.7)
- moved D5 5.74 mm to (32.7, 101.7), turned to 90 degrees
- moved C2 5.68 mm to (23.0, 101.8), turned to -90 degrees
- moved U4 4.05 mm to (28.0, 100.4), turned to 180 degrees
- moved R31 2.75 mm to (46.4, 65.3), turned to 90 degrees
- moved C14 0.40 mm to (48.7, 65.7)
- turned R11 to 180 degrees
- turned R16 to 180 degrees
- turned R2 to 180 degrees
- turned R3 to 180 degrees
- turned R8 to 180 degrees
Routing:
- net Net-(LED10-Pad2): track 0.00 -> 16.9 mm, vias 0 -> 2
- net Net-(LED4-Pad2): track 0.00 -> 15.0 mm, vias 0 -> 2
- net Net-(C2-Pad1): track 0.00 -> 7.88 mm
- net Net-(D25-Conn): track 0.00 -> 6.13 mm
- net Net-(D5-A): track 0.00 -> 4.27 mm
- net Net-(D19-K): track 0.00 -> 4.25 mm
- net GND2: track 17.6 -> 20.7 mm
